File: CM4IOv5.kicad_sch (KiCad schematic)
At the start: 8 parts

Commit message: board
Other:
- added sheet Sensors1 (Sensors.kicad_sch)
Changed lines of the file:
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@@
+	)
+	(sheet
+		(at 243.84 64.77)
+		(size 31.75 34.29)
+		(fields_autoplaced yes)
+		(stroke
+			(width 0.1524)
+			(type solid)
+		)
+		(fill
+			(color 0 0 0 0.0000)
+		)
+		(property "Sheetname" "Sensors1"
+			(at 243.84 64.0584 0)
+			(effects
+				(font
+					(size 1.27 1.27)
+				)
+				(justify left bottom)
+			)
+		)
+		(property "Sheetfile" "Sensors.kicad_sch"
+			(at 243.84 99.6446 0)
+			(effects
+				(font
+					(size 1.27 1.27)
+				)
+				(justify left top)
+			)
+		)
+		(instances
+			(project "CM4IOv5"
+				(path "/e63e39d7-6ac0-4ffd-8aa3-1841a4541b55"
+					(page "3")
+				)
+			)
+		)
 	)
 	(sheet

Commit message: changes stuff
Other:
- removed sheet Sensors1
- sheet Sensors ports: added Boot, IMU_Rst, Int, SCL, SDA; removed none
Changed lines of the file:
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@@
-	)
-	(sheet
-		(at 243.84 64.77)
-		(size 31.75 34.29)
-		(fields_autoplaced yes)
-		(stroke
-			(width 0.1524)
-			(type solid)
-		)
-		(fill
-			(color 0 0 0 0.0000)
-		)
-		(property "Sheetname" "Sensors1"
-			(at 243.84 64.0584 0)
-			(effects
-				(font
-					(size 1.27 1.27)
-				)
-				(justify left bottom)
-			)
-		)
-		(property "Sheetfile" "Sensors.kicad_sch"
-			(at 243.84 99.6446 0)
-			(effects
-				(font
-					(size 1.27 1.27)
-				)
-				(justify left top)
-			)
-		)
-		(instances
-			(project "CM4IOv5"
-				(path "/e63e39d7-6ac0-4ffd-8aa3-1841a4541b55"
-					(page "3")
-				)
-			)
-		)
 	)
 	(sheet
@@
 			)
 		)
+		(pin "SCL" input
+			(at 63.5 115.57 0)
+			(effects
+				(font
+					(size 1.27 1.27)
+				)
+				(justify right)
+			)
+		)
+		(pin "SDA" input
+			(at 63.5 119.38 0)
+			(effects
+				(font
+					(size 1.27 1.27)
+				)
+				(justify right)
+			)
+		)
+		(pin "Boot" input
+			(at 63.5 123.19 0)
+			(effects
+				(font
+					(size 1.27 1.27)
+				)
+				(justify right)
+			)
+		)
+		(pin "Int" input
+			(at 63.5 127 0)
+			(effects
+				(font
+					(size 1.27 1.27)
+				)
+				(justify right)
+			)
+		)
+		(pin "IMU_Rst" input
+			(at 63.5 130.81 0)
+			(effects
+				(font
+					(size 1.27 1.27)
+				)
+				(justify right)
+			)
+		)

Commit message: stuff
Other:
- sheet CM4_GPIO ( Ethernet, GPIO, SDCARD) ports: added Boot, Int, RX, Rst, TX; removed none
- sheet CM4_HighSpeed ports: added none; removed SCL0, SDA0
- sheet Sensors ports: added 3.3v; removed none
- note added: "-------"
- note added: "Envionmental Sensor"
- note added: "IMU"
- note added: "Sensor Stuff"
Changed lines of the file:
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@@
+	(wire
+		(pts
+			(xy 63.5 130.81) (xy 68.58 130.81)
+		)
+		(stroke
+			(width 0)
+			(type default)
+		)
+	)
 	(wire
 		(pts
@@
 	(wire
 		(pts
-			(xy 137.16 101.6) (xy 137.16 116.84)
-		)
-		(stroke
-			(width 0)
-			(type solid)
-		)
-	)
-	(wire
-		(pts
 			(xy 162.56 116.84) (xy 162.56 101.6)
 		)
@@
 	(wire
 		(pts
+			(xy 63.5 119.38) (xy 68.58 119.38)
+		)
+		(stroke
+			(width 0)
+			(type default)
+		)
+	)
+	(wire
+		(pts
 			(xy 147.32 101.6) (xy 147.32 116.84)
 		)
@@
 	(wire
 		(pts
+			(xy 63.5 134.62) (xy 71.12 134.62)
+		)
+		(stroke
+			(width 0)
+			(type default)
+		)
+	)
+	(wire
+		(pts
 			(xy 168.91 135.89) (xy 179.07 135.89)
 		)
@@
 	(wire
 		(pts
+			(xy 140.97 113.03) (xy 140.97 116.84)
+		)
+		(stroke
+			(width 0)
+			(type default)
+		)
+	)
+	(wire
+		(pts
 			(xy 168.91 58.42) (xy 190.5 58.42)
 		)
@@
 	(wire
 		(pts
+			(xy 63.5 123.19) (xy 68.58 123.19)
+		)
+		(stroke
+			(width 0)
+			(type default)
+		)
+	)
+	(wire
+		(pts
 			(xy 218.44 62.23) (xy 226.06 62.23)
 		)
@@
 	(wire
 		(pts
+			(xy 63.5 127) (xy 68.58 127)
+		)
+		(stroke
+			(width 0)
+			(type default)
+		)
+	)
+	(wire
+		(pts
 			(xy 105.41 60.96) (xy 132.08 60.96)
 		)
@@
 	(wire
 		(pts
+			(xy 63.5 115.57) (xy 68.58 115.57)
+		)
+		(stroke
+			(width 0)
+			(type default)
+		)
+	)
+	(wire
+		(pts
+			(xy 137.16 113.03) (xy 137.16 116.84)
+		)
+		(stroke
+			(width 0)
+			(type default)
+		)
+	)
+	(wire
+		(pts
 			(xy 168.91 62.23) (xy 190.5 62.23)
 		)
@@
 		(pts
 			(xy 168.91 48.26) (xy 190.5 48.26)
-		)
-		(stroke
-			(width 0)
-			(type solid)
-		)
-	)
-	(wire
-		(pts
-			(xy 140.97 101.6) (xy 140.97 116.84)
 		)
 		(stroke
@@
 		)
 	)
+	(text "Envionmental Sensor"
+		(exclude_from_sim no)
+		(at 44.45 119.888 0)
+		(effects
+			(font
+				(size 1.27 1.27)
+			)
+		)
+	)
 	(text "Connectors\n-------\nDual USB\nmicroUSB"
 		(exclude_from_sim no)
@@
 		)
 	)
+	(text "IMU"
+		(exclude_from_sim no)
+		(at 36.322 116.586 0)
+		(effects
+			(font
+				(size 1.27 1.27)
+			)
+		)
+	)
+	(text "Sensor Stuff"
+		(exclude_from_sim no)
+		(at 39.878 113.284 0)
+		(effects
+			(font
+				(size 1.27 1.27)
+			)
+		)
+	)
+	(text "-------"
+		(exclude_from_sim no)
+		(at 39.624 114.554 0)
+		(effects
+			(font
+				(size 1.27 1.27)
+			)
+		)
+	)
 	(text "Connectors\n-------\nEthernet\nSDCARD\n40way RPI\nJumpers"
 		(exclude_from_sim no)
@@
 		)
 	)
+	(label "SDA"
+		(at 68.58 119.38 0)
+		(fields_autoplaced yes)
+		(effects
+			(font
+				(size 1.27 1.27)
+			)
+			(justify left bottom)
+		)
+	)
+	(label "SCL"
+		(at 68.58 115.57 0)
+		(fields_autoplaced yes)
+		(effects
+			(font
+				(size 1.27 1.27)
+			)
+			(justify left bottom)
+		)
+	)
 	(label "+5v"
 		(at 170.18 130.81 0)
@@
 		)
 	)
+	(label "+3.3v"
+		(at 71.12 134.62 0)
+		(fields_autoplaced yes)
+		(effects
+			(font
+				(size 1.27 1.27)
+			)
+			(justify left bottom)
+		)
+	)
 	(label "+5v"
 		(at 73.66 52.07 0)
@@
 		)
 	)
+	(label "SCL"
+		(at 140.97 113.03 90)
+		(fields_autoplaced yes)
+		(effects
+			(font
+				(size 1.27 1.27)
+			)
+			(justify left bottom)
+		)
+	)
 	(label "+12v"
 		(at 219.71 62.23 0)
+		(fields_autoplaced yes)
+		(effects
+			(font
+				(size 1.27 1.27)
+			)
+			(justify left bottom)
+		)
+	)
+	(label "SDA"
+		(at 137.16 113.03 90)
 		(fields_autoplaced yes)
 		(effects
@@
 			)
 		)
+		(pin "Rst" output
+			(at 132.08 140.97 180)
+			(effects
+				(font
+					(size 1.27 1.27)
+				)
+				(justify left)
+			)
+		)
+		(pin "Boot" output
+			(at 132.08 144.78 180)
+			(effects
+				(font
+					(size 1.27 1.27)
+				)
+				(justify left)
+			)
+		)
+		(pin "Int" output
+			(at 168.91 140.97 0)
+			(effects
+				(font
+					(size 1.27 1.27)
+				)
+				(justify right)
+			)
+		)
+		(pin "TX" output
+			(at 168.91 143.51 0)
+			(effects
+				(font
+					(size 1.27 1.27)
+				)
+				(justify right)
+			)
+		)
+		(pin "RX" output
+			(at 168.91 146.05 0)
+			(effects
+				(font
+					(size 1.27 1.27)
+				)
+				(justify right)
+			)
+		)
 		(instances
 			(project "CM4IOv5"
@@
 			)
 		)
-		(pin "SCL0" input
-			(at 140.97 101.6 270)
-			(effects
-				(font
-					(size 1.27 1.27)
-				)
-				(justify left)
-			)
-		)
-		(pin "SDA0" input
-			(at 137.16 101.6 270)
-			(effects
-				(font
-					(size 1.27 1.27)
-				)
-				(justify left)
-			)
-		)
 		(pin "+5v" input
 			(at 132.08 77.47 180)
@@
 			(effects
 				(font
+					(size 1.27 1.27)
+				)
+				(justify right)
+			)
+		)
+		(pin "3.3v" input
+			(at 63.5 134.62 0)
+			(effects
+				(font

Commit message: stuff
Parts:
- added J15: HTST-110-X-X-D-RA, HTST-110-X-X-D-RA:SAMTEC_HTST-110-X-X-D-RA, symbol HTST-110-X-X-D-RA:HTST-110-X-X-D-RA
Connections:
- net SCL: now also J15.03
- net SDA: now also J15.05
- new net 5v_EXT_Stack: J15.01
Other:
- sheet CM4_GPIO ( Ethernet, GPIO, SDCARD) ports: added Alert, Leak; removed none
- sheet Power Stuff ports: added 5v, 5v_EXT_Stack, 5v_Ext_Barrel, Alert, SCL, SDA; removed none
- sheet Sensors ports: added Signal; removed none
- sheet USBhub ports: added 3.3v, 5v, USB2_N, USB2_P; removed none

Commit message: stuff
Other:
- added sheet Connectors (Connectors.kicad_sch)
- sheet CM4_GPIO ( Ethernet, GPIO, SDCARD) ports: added DE, RE; removed none
- sheet PSUs ports: added none; removed +5v
- sheet Power Stuff ports: added none; removed 5v_Ext_Barrel
- sheet RS485 ports: added 3.3v, DE, RE, RX, TX; removed none

Commit message: stuff
Parts:
- added SW1: 1301.9314.24, 1301.9314.24_SCH, symbol 1301_9314_24:1301.9314.24
Connections:
- net nEXTRST: now also SW1.2, SW1.4
- net n_reset: now reaches J15.07
- new net GND: SW1.1, SW1.3
Other:
- added sheet PWM_Generatrion (PWM_Generatrion.kicad_sch)
- added sheet ethernet (ethernet.kicad_sch)
- sheet CM4_GPIO ( Ethernet, GPIO, SDCARD) ports: added OE_PWM, n_reset; removed none
- sheet Connectors ports: added A, B; removed none
- sheet RS485 ports: added A, B; removed none
- note added: "Reset"

Commit message: stuff
Changed lines of the file:
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@@
 		)
 	)
-	(label "5v"
+	(label "+5v"
 		(at 170.18 130.81 0)
 		(fields_autoplaced yes)
@@
 		)
 	)
-	(label "5v"
+	(label "+5v"
 		(at 118.11 166.37 0)
 		(fields_autoplaced yes)

Commit message: stuff
Other:
- added sheet Sensors1 (Sensors1.kicad_sch)
- sheet CM4_GPIO ( Ethernet, GPIO, SDCARD) ports: added Boot1, IMU_Rst1, Int1; removed none
- company: © 2020-2022 Raspberry Pi Ltd (formerly Raspberry Pi (Trading) Ltd.) -> Sahil Mitra
- moved on the sheet: J15
