File: CM4IOv5.kicad_sch (KiCad schematic)
At the start: 10 parts, among them J15 HTST-110-X-X-D-RA, SW1 1301.9314.24

Commit message: stuff
Other:
- removed sheet PSUs
- removed sheet USB2-HUB
- note removed: "Connectors ------- DC Barrel Jack 4 pin power"
- note removed: "Connectors ------- Dual USB microUSB"

Commit message: stuff
Parts:
- added C2: .1u, symbol Device:C
- added R8: 10k, symbol Device:R
Connections:
- net nEXTRST: now also C2.1, R8.1; no longer SW1.2, SW1.4
- new net: C2.2, R8.2, SW1.2, SW1.4
Other:
- moved on the sheet: SW1

Commit message: stuff
Other:
- removed sheet Sensors1

Commit message: stuff
Connections:
- net n_reset: no longer J15.07
- net nEXTRST renamed CM4_GPIO ( Ethernet, GPIO, SDCARD)/nEXTRST
Other:
- sheet CM4_GPIO ( Ethernet, GPIO, SDCARD) ports: added IMU1_PS0, IMU_PS0; removed none
- sheet CM4_HighSpeed ports: added none; removed USBOTG_ID
- sheet Sensors ports: added Boot1, IMU1_PS0, IMU_PS0, IMU_Rst1, Int1; removed none
- note added: "-----------"
- note added: "Backplane Connector (PWM)"
- note added: "Linear Regulator"
- note added: "PWM Generation"
- note added: "PWM Generator"
- note added: "Power Components"
- note added: "Power Monitor"
- note added: "Power Mux"
- note added: "USBC Pwr Only"
- note removed: "Reset"
- moved on the sheet: H1, H2, H3, H4, H5, H6, H7, H8, J15, R8, SW1

Commit message: stuff
Other:
- removed sheet PCIe-connector
- removed sheet ethernet
- sheet CM4_HighSpeed ports: added none; removed PCIE_CLK_N, PCIE_CLK_P, PCIE_CLK_nREQ, PCIE_RX_N, PCIE_RX_P, PCIE_TX_N, PCIE_TX_P, PCIE_nRST
- note removed: "Connector ------ PCIe x1"

Commit message: stuff
Other:
- sheet CM4_GPIO ( Ethernet, GPIO, SDCARD) ports: added XRSTJ; removed CAM_GPIO
- sheet CM4_HighSpeed ports: added none; removed +3.3v, CAM_GPIO
- sheet PWM_Generatrion ports: added 5v, A, B, CS, ConRst, NISO, NOSI, SCLK, Telemetry; removed none
- sheet USBhub ports: added XRSTJ; removed none
- note added: "Backplane Connector(PWM)"
- note removed: "Backplane Connector (PWM)"
Changed lines of the file:
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@@
 	(wire
 		(pts
+			(xy 113.03 49.53) (xy 121.92 49.53)
+		)
+		(stroke
+			(width 0)
+			(type default)
+		)
+	)
+	(wire
+		(pts
 			(xy 193.04 124.46) (xy 193.04 130.81)
 		)
@@
 	(wire
 		(pts
+			(xy 168.91 146.05) (xy 193.04 146.05)
+		)
+		(stroke
+			(width 0)
+			(type default)
+		)
+	)
+	(wire
+		(pts
 			(xy 83.82 111.76) (xy 77.47 111.76)
 		)
@@
 	(wire
 		(pts
-			(xy 113.03 49.53) (xy 132.08 49.53)
+			(xy 218.44 154.94) (xy 224.79 154.94)
+		)
+		(stroke
+			(width 0)
+			(type default)
+		)
+	)
+	(wire
+		(pts
+			(xy 113.03 58.42) (xy 119.38 58.42)
 		)
 		(stroke
@@
 	(wire
 		(pts
-			(xy 168.91 148.59) (xy 179.07 148.59)
+			(xy 220.98 127) (xy 220.98 124.46)
 		)
 		(stroke
@@
 	(wire
 		(pts
-			(xy 220.98 127) (xy 220.98 124.46)
+			(xy 114.3 97.79) (xy 119.38 97.79)
 		)
 		(stroke
@@
 	(wire
 		(pts
-			(xy 114.3 97.79) (xy 119.38 97.79)
+			(xy 114.3 128.27) (xy 132.08 128.27)
 		)
 		(stroke
@@
 	(wire
 		(pts
-			(xy 114.3 128.27) (xy 132.08 128.27)
+			(xy 218.44 147.32) (xy 224.79 147.32)
 		)
 		(stroke
@@
 	(wire
 		(pts
-			(xy 151.13 86.36) (xy 151.13 92.71)
+			(xy 162.56 86.36) (xy 162.56 92.71)
 		)
 		(stroke
@@
 	(wire
 		(pts
-			(xy 218.44 147.32) (xy 224.79 147.32)
+			(xy 114.3 100.33) (xy 132.08 100.33)
 		)
 		(stroke
@@
 	(wire
 		(pts
-			(xy 162.56 86.36) (xy 162.56 92.71)
+			(xy 114.3 138.43) (xy 132.08 138.43)
 		)
 		(stroke
@@
 	(wire
 		(pts
-			(xy 114.3 100.33) (xy 132.08 100.33)
+			(xy 114.3 135.89) (xy 132.08 135.89)
 		)
 		(stroke
@@
 	(wire
 		(pts
-			(xy 114.3 138.43) (xy 132.08 138.43)
+			(xy 168.91 143.51) (xy 193.04 143.51)
 		)
 		(stroke
@@
 	(wire
 		(pts
-			(xy 114.3 135.89) (xy 132.08 135.89)
+			(xy 218.44 152.4) (xy 224.79 152.4)
 		)
 		(stroke
@@
 	(wire
 		(pts
-			(xy 168.91 143.51) (xy 193.04 143.51)
+			(xy 125.73 113.03) (xy 132.08 113.03)
 		)
 		(stroke
@@
 	(wire
 		(pts
+			(xy 218.44 149.86) (xy 224.79 149.86)
+		)
+		(stroke
+			(width 0)
+			(type default)
+		)
+	)
+	(wire
+		(pts
 			(xy 83.82 101.6) (xy 77.47 101.6)
 		)
@@
 	(text "PWM Generation\n"
 		(exclude_from_sim no)
-		(at 202.438 147.066 0)
+		(at 207.264 148.336 0)
 		(effects
 			(font
@@
 	(text "-------"
 		(exclude_from_sim no)
-		(at 200.152 148.336 0)
+		(at 204.978 149.606 0)
 		(effects
 			(font
@@
 		)
 	)
-	(text "Backplane Connector\n(PWM)"
+	(text "Backplane \nConnector(PWM)"
 		(exclude_from_sim no)
-		(at 204.978 153.416 0)
+		(at 207.518 154.432 0)
 		(effects
 			(font
@@
 	(text "PWM Generator\n"
 		(exclude_from_sim no)
-		(at 202.184 150.368 0)
+		(at 207.01 151.638 0)
 		(effects
 			(font
@@
 		)
 	)
-	(label "n_reset"
-		(at 179.07 148.59 0)
-		(fields_autoplaced yes)
-		(effects
-			(font
-				(size 1.27 1.27)
-			)
-			(justify left bottom)
-		)
-	)
 	(label "DE"
 		(at 119.38 102.87 0)
@@
 		)
 	)
+	(label "A"
+		(at 224.79 152.4 180)
+		(fields_autoplaced yes)
+		(effects
+			(font
+				(size 1.27 1.27)
+			)
+			(justify right bottom)
+		)
+	)
 	(label "B"
 		(at 83.82 96.52 180)
@@
 		)
 	)
+	(label "+5v"
+		(at 224.79 149.86 180)
+		(fields_autoplaced yes)
+		(effects
+			(font
+				(size 1.27 1.27)
+			)
+			(justify right bottom)
+		)
+	)
 	(label "SCL"
 		(at 83.82 104.14 180)
@@
 		)
 	)
+	(label "B"
+		(at 224.79 154.94 180)
+		(fields_autoplaced yes)
+		(effects
+			(font
+				(size 1.27 1.27)
+			)
+			(justify right bottom)
+		)
+	)
+	(label "XRSTJ"
+		(at 119.38 58.42 180)
+		(fields_autoplaced yes)
+		(effects
+			(font
+				(size 1.27 1.27)
+			)
+			(justify right bottom)
+		)
+	)
 	(label "SCL"
 		(at 125.73 123.19 0)
@@
 		)
 	)
+	(label "XRSTJ"
+		(at 125.73 113.03 0)
+		(fields_autoplaced yes)
+		(effects
+			(font
+				(size 1.27 1.27)
+			)
+			(justify left bottom)
+		)
+	)
 	(label "SDA"
 		(at 129.54 120.65 180)
@@
 			)
 		)
-		(pin "CAM_GPIO" output
-			(at 151.13 92.71 90)
-			(effects
-				(font
-					(size 1.27 1.27)
-				)
-				(justify right)
-			)
-		)
 		(pin "SCL0" output
 			(at 132.08 123.19 180)
@@
 		)
 		(pin "n_reset" output
-			(at 168.91 148.59 0)
+			(at 168.91 146.05 0)
 			(effects
 				(font
@@
 			)
 		)
+		(pin "XRSTJ" output
+			(at 132.08 113.03 180)
+			(effects
+				(font
+					(size 1.27 1.27)
+				)
+				(justify left)
+			)
+		)
 		(instances
 			(project "CM4IOv5"
@@
 			)
 		)
-		(pin "CAM_GPIO" input
-			(at 151.13 86.36 270)
-			(effects
-				(font
-					(size 1.27 1.27)
-				)
-				(justify left)
-			)
-		)
 		(pin "+5v" input
 			(at 132.08 45.72 180)
@@
 			)
 		)
-		(pin "+3.3v" input
-			(at 132.08 49.53 180)
-			(effects
-				(font
-					(size 1.27 1.27)
-				)
-				(justify left)
-			)
-		)
 		(pin "GPIO_VREF" input
 			(at 147.32 86.36 270)
@@
 			)
 		)
+		(pin "XRSTJ" input
+			(at 113.03 58.42 0)
+			(effects
+				(font
+					(size 1.27 1.27)
+				)
+				(justify right)
+			)
+		)
 		(instances
 			(project "CM4IOv5"
@@
 			)
 		)
+		(pin "5v" input
+			(at 218.44 149.86 0)
+			(effects
+				(font
+					(size 1.27 1.27)
+				)
+				(justify right)
+			)
+		)
+		(pin "A" input
+			(at 218.44 152.4 0)
+			(effects
+				(font
+					(size 1.27 1.27)
+				)
+				(justify right)
+			)
+		)
+		(pin "SCLK" input
+			(at 193.04 156.21 180)
+			(effects
+				(font
+					(size 1.27 1.27)
+				)
+				(justify left)
+			)
+		)
+		(pin "B" input
+			(at 218.44 154.94 0)
+			(effects
+				(font
+					(size 1.27 1.27)
+				)
+				(justify right)
+			)
+		)
+		(pin "NOSI" input
+			(at 193.04 153.67 180)
+			(effects
+				(font
+					(size 1.27 1.27)
+				)
+				(justify left)
+			)
+		)
+		(pin "Telemetry" input
+			(at 193.04 140.97 180)
+			(effects
+				(font
+					(size 1.27 1.27)
+				)
+				(justify left)
+			)
+		)
+		(pin "CS" input
+			(at 193.04 151.13 180)
+			(effects
+				(font
+					(size 1.27 1.27)
+				)
+				(justify left)
+			)
+		)
+		(pin "ConRst" input
+			(at 193.04 146.05 180)
+			(effects
+				(font
+					(size 1.27 1.27)
+				)
+				(justify left)
+			)
+		)
+		(pin "NISO" input
+			(at 193.04 148.59 180)
+			(effects
+				(font
+					(size 1.27 1.27)
+				)
+				(justify left)
+			)
+		)

Commit message: stuff
Connections:
- no-connect marks 0 -> 17
Other:
- sheet Connectors ports: added Leak; removed LEAK
- sheet Power Stuff ports: added 3.3v; removed none

Commit message: stuff
Other:
- sheet RS485 ports: added TB_EN; removed none
Changed lines of the file:
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@@
+			)
+		)
+		(pin "TB_EN" input
+			(at 114.3 110.49 0)
+			(effects
+				(font
+					(size 1.27 1.27)
+				)
+				(justify right)
 			)
 		)
