File: Sensors.kicad_sch (KiCad schematic)
At the start: 15 parts, among them U17 BNO085, U19 BME280

Commit message: board
Parts:
- renumbered C22 to C13, C23 to C53, JP1 to JP3, JP2 to JP4, R21 to R37, R19 to R38, U17 to U12, XTAL1 to XTAL2
Changed lines of the file:
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@@
 		(dnp no)
 		(fields_autoplaced yes)
-		(property "Reference" "U17"
+		(property "Reference" "U12"
 			(at 91.44 46.99 0)
 			(effects
@@
 		)
 		(instances
-			(project ""
-				(path "/e63e39d7-6ac0-4ffd-8aa3-1841a4541b55/d818c5c4-22e1-4750-8cc8-fe8a67dac1ec"
-					(reference "U17")
+			(project "CM4IOv5"
+				(path "/e63e39d7-6ac0-4ffd-8aa3-1841a4541b55/be571de0-64ad-4b5b-adc2-f7cb405f0103"
+					(reference "U12")
 					(unit 1)
 				)
@@
 		(instances
 			(project "CM4IOv5"
+				(path "/e63e39d7-6ac0-4ffd-8aa3-1841a4541b55/be571de0-64ad-4b5b-adc2-f7cb405f0103"
+					(reference "R39")
+					(unit 1)
+				)
 				(path "/e63e39d7-6ac0-4ffd-8aa3-1841a4541b55/d818c5c4-22e1-4750-8cc8-fe8a67dac1ec"
 					(reference "R20")
@@
 		(dnp no)
 		(fields_autoplaced yes)
-		(property "Reference" "R21"
+		(property "Reference" "R37"
 			(at 48.26 48.2599 0)
 			(effects
@@
 		)
 		(instances
-			(project ""
-				(path "/e63e39d7-6ac0-4ffd-8aa3-1841a4541b55/d818c5c4-22e1-4750-8cc8-fe8a67dac1ec"
-					(reference "R21")
+			(project "CM4IOv5"
+				(path "/e63e39d7-6ac0-4ffd-8aa3-1841a4541b55/be571de0-64ad-4b5b-adc2-f7cb405f0103"
+					(reference "R37")
 					(unit 1)
 				)
@@
 		(dnp no)
 		(fields_autoplaced yes)
-		(property "Reference" "#PWR032"
+		(property "Reference" "#PWR058"
 			(at 220.98 93.98 0)
 			(effects
@@
 		)
 		(instances
-			(project ""
-				(path "/e63e39d7-6ac0-4ffd-8aa3-1841a4541b55/d818c5c4-22e1-4750-8cc8-fe8a67dac1ec"
-					(reference "#PWR032")
+			(project "CM4IOv5"
+				(path "/e63e39d7-6ac0-4ffd-8aa3-1841a4541b55/be571de0-64ad-4b5b-adc2-f7cb405f0103"
+					(reference "#PWR058")
 					(unit 1)
 				)
@@
 		(instances
 			(project "CM4IOv5"
+				(path "/e63e39d7-6ac0-4ffd-8aa3-1841a4541b55/be571de0-64ad-4b5b-adc2-f7cb405f0103"
+					(reference "R7")
+					(unit 1)
+				)
 				(path "/e63e39d7-6ac0-4ffd-8aa3-1841a4541b55/d818c5c4-22e1-4750-8cc8-fe8a67dac1ec"
 					(reference "R32")
@@
 		(dnp no)
 		(fields_autoplaced yes)
-		(property "Reference" "#PWR035"
+		(property "Reference" "#PWR053"
 			(at 77.47 33.02 0)
 			(effects
@@
 		)
 		(instances
-			(project ""
-				(path "/e63e39d7-6ac0-4ffd-8aa3-1841a4541b55/d818c5c4-22e1-4750-8cc8-fe8a67dac1ec"
-					(reference "#PWR035")
+			(project "CM4IOv5"
+				(path "/e63e39d7-6ac0-4ffd-8aa3-1841a4541b55/be571de0-64ad-4b5b-adc2-f7cb405f0103"
+					(reference "#PWR053")
 					(unit 1)
 				)
@@
 		(dnp no)
 		(fields_autoplaced yes)
-		(property "Reference" "JP2"
+		(property "Reference" "JP4"
 			(at 64.77 25.4 0)
 			(effects
@@
 		)
 		(instances
-			(project ""
-				(path "/e63e39d7-6ac0-4ffd-8aa3-1841a4541b55/d818c5c4-22e1-4750-8cc8-fe8a67dac1ec"
-					(reference "JP2")
+			(project "CM4IOv5"
+				(path "/e63e39d7-6ac0-4ffd-8aa3-1841a4541b55/be571de0-64ad-4b5b-adc2-f7cb405f0103"
+					(reference "JP4")
 					(unit 1)
 				)
@@
 		(dnp no)
 		(fields_autoplaced yes)
-		(property "Reference" "R19"
+		(property "Reference" "R38"
 			(at 181.61 88.8999 0)
 			(effects
@@
 		)
 		(instances
-			(project ""
-				(path "/e63e39d7-6ac0-4ffd-8aa3-1841a4541b55/d818c5c4-22e1-4750-8cc8-fe8a67dac1ec"
-					(reference "R19")
+			(project "CM4IOv5"
+				(path "/e63e39d7-6ac0-4ffd-8aa3-1841a4541b55/be571de0-64ad-4b5b-adc2-f7cb405f0103"
+					(reference "R38")
 					(unit 1)
 				)
@@
 		(dnp no)
 		(fields_autoplaced yes)
-		(property "Reference" "#PWR03"
+		(property "Reference" "#PWR056"
 			(at 144.78 55.88 0)
 			(effects
@@
 		)
 		(instances
-			(project ""
-				(path "/e63e39d7-6ac0-4ffd-8aa3-1841a4541b55/d818c5c4-22e1-4750-8cc8-fe8a67dac1ec"
-					(reference "#PWR03")
+			(project "CM4IOv5"
+				(path "/e63e39d7-6ac0-4ffd-8aa3-1841a4541b55/be571de0-64ad-4b5b-adc2-f7cb405f0103"
+					(reference "#PWR056")
 					(unit 1)
 				)
@@
 		(dnp no)
 		(fields_autoplaced yes)
-		(property "Reference" "#PWR028"
+		(property "Reference" "#PWR055"
 			(at 139.7 99.06 0)
 			(effects
@@
 		)
 		(instances
-			(project ""
-				(path "/e63e39d7-6ac0-4ffd-8aa3-1841a4541b55/d818c5c4-22e1-4750-8cc8-fe8a67dac1ec"
-					(reference "#PWR028")
+			(project "CM4IOv5"
+				(path "/e63e39d7-6ac0-4ffd-8aa3-1841a4541b55/be571de0-64ad-4b5b-adc2-f7cb405f0103"
+					(reference "#PWR055")
 					(unit 1)
 				)
@@
 		(instances
 			(project "CM4IOv5"
+				(path "/e63e39d7-6ac0-4ffd-8aa3-1841a4541b55/be571de0-64ad-4b5b-adc2-f7cb405f0103"
+					(reference "U21")
+					(unit 1)
+				)
 				(path "/e63e39d7-6ac0-4ffd-8aa3-1841a4541b55/d818c5c4-22e1-4750-8cc8-fe8a67dac1ec"
 					(reference "U19")
@@
 		(dnp no)
 		(fields_autoplaced yes)
-		(property "Reference" "#PWR034"
+		(property "Reference" "#PWR052"
 			(at 45.72 40.64 0)
 			(effects
@@
 		)
 		(instances
-			(project ""
-				(path "/e63e39d7-6ac0-4ffd-8aa3-1841a4541b55/d818c5c4-22e1-4750-8cc8-fe8a67dac1ec"
-					(reference "#PWR034")
+			(project "CM4IOv5"
+				(path "/e63e39d7-6ac0-4ffd-8aa3-1841a4541b55/be571de0-64ad-4b5b-adc2-f7cb405f0103"
+					(reference "#PWR052")
 					(unit 1)
 				)
@@
 		(dnp no)
 		(fields_autoplaced yes)
-		(property "Reference" "#PWR033"
+		(property "Reference" "#PWR059"
 			(at 237.49 127 0)
 			(effects
@@
 		)
 		(instances
-			(project ""
-				(path "/e63e39d7-6ac0-4ffd-8aa3-1841a4541b55/d818c5c4-22e1-4750-8cc8-fe8a67dac1ec"
-					(reference "#PWR033")
+			(project "CM4IOv5"
+				(path "/e63e39d7-6ac0-4ffd-8aa3-1841a4541b55/be571de0-64ad-4b5b-adc2-f7cb405f0103"
+					(reference "#PWR059")
 					(unit 1)
 				)
@@
 		(dnp no)
 		(fields_autoplaced yes)
-		(property "Reference" "JP1"
+		(property "Reference" "JP3"
 			(at 64.77 20.32 0)
 			(effects
@@
 		)
 		(instances
-			(project ""
-				(path "/e63e39d7-6ac0-4ffd-8aa3-1841a4541b55/d818c5c4-22e1-4750-8cc8-fe8a67dac1ec"
-					(reference "JP1")
+			(project "CM4IOv5"
+				(path "/e63e39d7-6ac0-4ffd-8aa3-1841a4541b55/be571de0-64ad-4b5b-adc2-f7cb405f0103"
+					(reference "JP3")
 					(unit 1)
 				)
@@
 		(instances
 			(project "CM4IOv5"
+				(path "/e63e39d7-6ac0-4ffd-8aa3-1841a4541b55/be571de0-64ad-4b5b-adc2-f7cb405f0103"
+					(reference "C55")
+					(unit 1)
+				)
 				(path "/e63e39d7-6ac0-4ffd-8aa3-1841a4541b55/d818c5c4-22e1-4750-8cc8-fe8a67dac1ec"
 					(reference "C48")
@@
 		(dnp no)
 		(fields_autoplaced yes)
-		(property "Reference" "C22"
+		(property "Reference" "C13"
 			(at 148.59 39.3699 0)
 			(effects
@@
 		)
 		(instances
-			(project ""
-				(path "/e63e39d7-6ac0-4ffd-8aa3-1841a4541b55/d818c5c4-22e1-4750-8cc8-fe8a67dac1ec"
-					(reference "C22")
+			(project "CM4IOv5"
+				(path "/e63e39d7-6ac0-4ffd-8aa3-1841a4541b55/be571de0-64ad-4b5b-adc2-f7cb405f0103"
+					(reference "C13")
 					(unit 1)
 				)
@@
 		(dnp no)
 		(fields_autoplaced yes)
-		(property "Reference" "XTAL1"
+		(property "Reference" "XTAL2"
 			(at 203.2 44.45 0)
 			(effects
@@
 		)
 		(instances
-			(project ""
-				(path "/e63e39d7-6ac0-4ffd-8aa3-1841a4541b55/d818c5c4-22e1-4750-8cc8-fe8a67dac1ec"
-					(reference "XTAL1")
+			(project "CM4IOv5"
+				(path "/e63e39d7-6ac0-4ffd-8aa3-1841a4541b55/be571de0-64ad-4b5b-adc2-f7cb405f0103"
+					(reference "XTAL2")
 					(unit 1)
 				)
@@
 		(instances
 			(project "CM4IOv5"
+				(path "/e63e39d7-6ac0-4ffd-8aa3-1841a4541b55/be571de0-64ad-4b5b-adc2-f7cb405f0103"
+					(reference "C12")
+					(unit 1)
+				)
 				(path "/e63e39d7-6ac0-4ffd-8aa3-1841a4541b55/d818c5c4-22e1-4750-8cc8-fe8a67dac1ec"
 					(reference "C24")
@@
 		(dnp no)
 		(fields_autoplaced yes)
-		(property "Reference" "#PWR031"
+		(property "Reference" "#PWR057"
 			(at 201.93 72.39 0)
 			(effects
@@
 		)
 		(instances
-			(project ""
-				(path "/e63e39d7-6ac0-4ffd-8aa3-1841a4541b55/d818c5c4-22e1-4750-8cc8-fe8a67dac1ec"
-					(reference "#PWR031")
+			(project "CM4IOv5"
+				(path "/e63e39d7-6ac0-4ffd-8aa3-1841a4541b55/be571de0-64ad-4b5b-adc2-f7cb405f0103"
+					(reference "#PWR057")
 					(unit 1)
 				)
@@
 		(instances
 			(project "CM4IOv5"
+				(path "/e63e39d7-6ac0-4ffd-8aa3-1841a4541b55/be571de0-64ad-4b5b-adc2-f7cb405f0103"
+					(reference "R6")
+					(unit 1)
+				)
 				(path "/e63e39d7-6ac0-4ffd-8aa3-1841a4541b55/d818c5c4-22e1-4750-8cc8-fe8a67dac1ec"
 					(reference "R31")
@@
 		(instances
 			(project "CM4IOv5"
+				(path "/e63e39d7-6ac0-4ffd-8aa3-1841a4541b55/be571de0-64ad-4b5b-adc2-f7cb405f0103"
+					(reference "C54")
+					(unit 1)
+				)
 				(path "/e63e39d7-6ac0-4ffd-8aa3-1841a4541b55/d818c5c4-22e1-4750-8cc8-fe8a67dac1ec"
 					(reference "C46")
@@
 		(dnp no)
 		(fields_autoplaced yes)
-		(property "Reference" "#PWR030"
+		(property "Reference" "#PWR054"
 			(at 138.43 36.83 0)
 			(effects
@@
 		)
 		(instances
-			(project ""
-				(path "/e63e39d7-6ac0-4ffd-8aa3-1841a4541b55/d818c5c4-22e1-4750-8cc8-fe8a67dac1ec"
-					(reference "#PWR030")
+			(project "CM4IOv5"
+				(path "/e63e39d7-6ac0-4ffd-8aa3-1841a4541b55/be571de0-64ad-4b5b-adc2-f7cb405f0103"
+					(reference "#PWR054")
 					(unit 1)
 				)
@@
 		(dnp no)
 		(fields_autoplaced yes)
-		(property "Reference" "C23"
+		(property "Reference" "C53"
 			(at 161.29 39.3699 0)
 			(effects
@@
 		)
 		(instances
-			(project ""
-				(path "/e63e39d7-6ac0-4ffd-8aa3-1841a4541b55/d818c5c4-22e1-4750-8cc8-fe8a67dac1ec"
-					(reference "C23")
-					(unit 1)
-				)
+			(project "CM4IOv5"
+				(path "/e63e39d7-6ac0-4ffd-8aa3-1841a4541b55/be571de0-64ad-4b5b-adc2-f7cb405f0103"
+					(reference "C53")
+					(unit 1)
+				)

Commit message: changes stuff
Parts:
- renumbered C24 to C12, C46 to C54, C48 to C55, R20 to R39, R31 to R6, R32 to R7, U19 to U21
Connections:
- net Rst renamed IMU_Rst

Commit message: stuff
Parts:
- renumbered C12 to C24, C54 to C46, C55 to C48, C13 to C?, C53 to C?, JP4 to JP?, JP3 to JP?, R39 to R20, R6 to R31, R7 to R32, R37 to R?, R38 to R?, U21 to U19, U12 to U?, XTAL2 to XTAL?
Connections:
- net +3.3V renamed 3.3v

Commit message: stuff
Parts:
- added D9: 1N4148, digikey-footprints:Diode_DO-35_P10mm, symbol dk_Diodes-Rectifiers-Single:1N4148
- added Q2: 2N7002, digikey-footprints:SOT-23-3, symbol dk_Transistors-FETs-MOSFETs-Single:2N7002
- added R19, R6: 1k, symbol Device:R
- added R21: 240, symbol Device:R
- added R7: 27k, symbol Device:R
Connections:
- net 3.3v: now also Q2.3 (D), R7.1
- net GND: now also D9.1, R19.2
- new net: Q2.1 (G), R6.2, R7.2
- new net: D9.2, R21.2
- new net Probe: R6.1
- new net Signal: Q2.2 (S), R19.1, R21.1

Commit message: stuff
Parts:
- added J16, J17, J18, J21: SM02B-GHS-TB, CONN_SM02B-GHS_JST, symbol SM02B_GHS_TB:SM02B-GHS-TB
Connections:
- net GND: now also U?.10 (CLKSEL0), J16.2, J17.2, J18.2, J21.2
- net Probe: now also J16.1, J17.1, J18.1, J21.1

Commit message: stuff
Parts:
- R31, R32: value 2.2k -> 10k
Other:
- note added: "LEAK Sensor"
Changed lines of the file:
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@@
+		)
+	)
+	(text "LEAK Sensor\n"
+		(exclude_from_sim no)
+		(at 90.424 142.748 0)
+		(effects
+			(font
+				(size 1.27 1.27)
+			)
 		)
 	)
@@
 			)
 		)
-		(property "Value" "2.2k"
+		(property "Value" "10k"
 			(at 26.67 45.7199 0)
 			(effects
@@
 			)
 		)
-		(property "Value" "2.2k"
+		(property "Value" "10k"
 			(at 21.59 45.7199 0)
 			(effects

Commit message: stuff
Parts:
- gave numbers to parts that had none: 8
- renumbered D9 to D17, J16 to J27, J17 to J28, J18 to J29, J21 to J30, Q2 to Q3, R6 to R50, R7 to R51, R19 to R52, R21 to R53

Commit message: stuff
Parts:
- renumbered C83 to C?, C84 to C?, D17 to D?, J29 to J?, J28 to J?, J30 to J?, J27 to J?, JP5 to JP?, JP4 to JP?, Q3 to Q?, R51 to R?, R49 to R?, R50 to R?, R54 to R?, R52 to R?, R53 to R?, U26 to U?, XTAL1 to XTAL?
