File: Sensors.kicad_sch (KiCad schematic)
At the start: 25 parts, among them U19 BME280

Commit message: stuff
Connections:
- net GND: now also U?.2 (GND), U?.25 (GNDIO)
- new net PS0: U?.6 (PS0/WAKE)
Changed lines of the file:
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@@
 	)
 	(junction
+		(at 121.92 92.71)
+		(diameter 0)
+		(color 0 0 0 0)
+	)
+	(junction
 		(at 71.12 180.34)
 		(diameter 0)
@@
 	)
 	(junction
-		(at 121.92 92.71)
-		(diameter 0)
-		(color 0 0 0 0)
-	)
-	(junction
 		(at 184.15 105.41)
 		(diameter 0)
@@
 	(wire
 		(pts
-			(xy 52.07 77.47) (xy 52.07 111.76)
-		)
-		(stroke
-			(width 0)
-			(type default)
-		)
-	)
-	(wire
-		(pts
 			(xy 78.74 156.21) (xy 82.55 156.21)
 		)
@@
 	(wire
 		(pts
-			(xy 121.92 92.71) (xy 121.92 111.76)
-		)
-		(stroke
-			(width 0)
-			(type default)
-		)
-	)
-	(wire
-		(pts
 			(xy 29.21 72.39) (xy 29.21 115.57)
 		)
@@
 	(wire
 		(pts
-			(xy 52.07 111.76) (xy 121.92 111.76)
-		)
-		(stroke
-			(width 0)
-			(type default)
-		)
-	)
-	(wire
-		(pts
 			(xy 165.1 102.87) (xy 179.07 102.87)
 		)
@@
 		)
 	)
+	(label "PS0"
+		(at 52.07 77.47 0)
+		(fields_autoplaced yes)
+		(effects
+			(font
+				(size 1.27 1.27)
+			)
+			(justify left bottom)
+		)
+	)
 	(label "SDA"
 		(at 27.94 64.77 0)
@@
 					(unit 1)
 				)
+			)
+		)
+	)
+	(symbol
+		(lib_id "power:GND")
+		(at 121.92 92.71 0)
+		(unit 1)
+		(exclude_from_sim no)
+		(in_bom yes)
+		(on_board yes)
+		(dnp no)
+		(fields_autoplaced yes)
+		(property "Reference" "#PWR012"
+			(at 121.92 99.06 0)
+			(effects
+				(font
+					(size 1.27 1.27)
+				)
+				(hide yes)
+			)
+		)
+		(property "Value" "GND"
+			(at 121.92 97.79 0)
+			(effects
+				(font
+					(size 1.27 1.27)
+				)
+			)
+		)
+		(property "Footprint" ""
+			(at 121.92 92.71 0)
+			(effects
+				(font
+					(size 1.27 1.27)
+				)
+				(hide yes)
+			)
+		)
+		(property "Datasheet" ""
+			(at 121.92 92.71 0)
+			(effects
+				(font
+					(size 1.27 1.27)
+				)
+				(hide yes)
+			)
+		)
+		(property "Description" "Power symbol creates a global label with name \"GND\" , ground"
+			(at 121.92 92.71 0)
+			(effects
+				(font
+					(size 1.27 1.27)
+				)
+				(hide yes)
+			)
+		)
+		(pin "1"
+		)
+		(instances
+			(project ""
+				(path "/e63e39d7-6ac0-4ffd-8aa3-1841a4541b55/d818c5c4-22e1-4750-8cc8-fe8a67dac1ec"
+					(reference "#PWR012")
+					(unit 1)
+				)

Commit message: stuff
Parts:
- removed C24, C? (x2): .1u, symbol Device:C
- removed C46, C48: 22p, symbol Device:C
- removed JP? (x2): Jumper_2_Open, symbol Jumper:Jumper_2_Open
- removed R?: 10k, symbol Device:R
- removed R?: 2.2k, symbol Device:R
- removed U?: BNO085, BNO085:IC_BNO085, symbol BNO085:BNO085
- removed XTAL?: ECS-_327-12_5-34B-TR, digikey-footprints:SMD-2_3.2x1.5mm, symbol dk_Crystals:ECS-_327-12_5-34B-TR
- added C13, C14, C15, C16, C17, C18: .1u, symbol Device:C
- added JP10, JP7, JP8, JP9: Jumper_2_Open, symbol Jumper:Jumper_2_Open
- added R27, R36, R47: 2.2k, symbol Device:R
- added R28, R48: 10k, symbol Device:R
- added U13: BME280, digikey-footprints:Pressure_Sensor_LGA-8_2.5x2.5mm_BME280, symbol dk_Humidity-Moisture-Sensors:BME280
- added U16, U7: BNO085, BNO085:IC_BNO085, symbol BNO085:BNO085
Connections:
- net 3.3v: now also C14.1, C15.1, C17.1, C18.1, JP7.1 (A), JP9.1 (A), R27.1, R28.1, R36.1, R47.1, R48.1, U13.2 (CSB), U13.6 (VDDIO), U13.8 (VDD), U16.10 (CLKSEL0), U16.28 (VDDIO), U16.3 (VDD), U16.5 (PS1), U7.10 (CLKSEL0), U7.28 (VDDIO), U7.3 (VDD), U7.5 (PS1)
- net Boot: now also R28.2, U7.4 (~{BOOT})
- net GND: now also C13.2, C14.2, C15.2, C16.2, C17.2, C18.2, JP10.1 (A), JP8.1 (A), U13.1 (GND), U13.7 (GND), U16.2 (GND), U16.25 (GNDIO), U16.26 (XOUT32/CLKSEL1), U7.2 (GND), U7.25 (GNDIO), U7.26 (XOUT32/CLKSEL1)
- net IMU_Rst: now also U7.11 (~{RST})
- net Int: now also U7.14 (~{H_INT})
- net SCL: now also U16.19 (H_SCL/SCK/RX), U7.19 (H_SCL/SCK/RX)
- net SDA: now also U16.20 (H_SDA/H_MISO/TX), U7.20 (H_SDA/H_MISO/TX)
- net ENV_SCL: now reaches U19.4 (SCK)
- net ENV_SCL: now also R20.2, U7.15 (ENV_SCL)
- net ENV_SDA: now reaches U19.3 (SDI)
- net ENV_SDA: now also R27.2, U7.16 (ENV_SDA); no longer R20.2
- new net: C13.1, U7.9 (CAP)
- new net: U7.1 (RESV_NC), U7.12 (RESV_NC), U7.13 (RESV_NC), U7.21 (RESV_NC), U7.22 (RESV_NC), U7.23 (RESV_NC), U7.24 (RESV_NC), U7.7 (RESV_NC), U7.8 (RESV_NC)
- new net: U16.1 (RESV_NC), U16.12 (RESV_NC), U16.13 (RESV_NC), U16.21 (RESV_NC), U16.22 (RESV_NC), U16.23 (RESV_NC), U16.24 (RESV_NC), U16.7 (RESV_NC), U16.8 (RESV_NC)
- new net: C16.1, U16.9 (CAP)
- new net Boot1: R48.2, U16.4 (~{BOOT})
- new net ENV_SCL1: R36.2, U13.4 (SCK), U16.15 (ENV_SCL)
- new net ENV_SDA1: R47.2, U13.3 (SDI), U16.16 (ENV_SDA)
- new net IMU1_PS0: U16.6 (PS0/WAKE)
- new net IMU_PS0: U7.6 (PS0/WAKE)
- new net IMU_Rst1: U16.11 (~{RST})
- new net Int1: U16.14 (~{H_INT})
- new net SA0: JP7.2 (B), JP8.2 (B), U7.17 (SA0/H_MOSI)
- new net SA0_1: JP10.2 (B), JP9.2 (B), U16.17 (SA0/H_MOSI)
- no-connect marks 0 -> 6
Other:
- note added: "Address Select Jumpers"
- note added: "Enviornmental Sensors"
- note added: "IMUs"
- note added: "Pull Up Resistors"
- note removed: "Clock"
- note removed: "IMU"
- note removed: "SENSOR PRESSURE HUMIDITY TEMP"
- moved on the sheet: D?, J?, Q?, R?
