File: ethernet.kicad_sch (KiCad schematic)
At the start: 4 parts, among them U17 KSZ9897RTXC, Y2 25 MHz

Commit message: stuff
Parts:
- added IC1: PD69104B1ILQ-TR, QFN50P800X800X100-49N-D, symbol PD69104B1ILQ-TR:PD69104B1ILQ-TR
- added U23, U24, U25, U26: 0816-1X1T-23-F, 0816-1X1T_BEL, symbol 0816_1X1T_23_F:0816-1X1T-23-F

Commit message: stuff
Parts:
- removed U23, U24, U25, U26: 0816-1X1T-23-F, 0816-1X1T_BEL, symbol 0816_1X1T_23_F:0816-1X1T-23-F
- added J24: 0826-1X1T-GH-F, 0826-1X1T-GH-F:BEL_0826-1X1T-GH-F, symbol 0826-1X1T-GH-F:0826-1X1T-GH-F
Connections:
- net GND: now also J24.S1 (SHIELD), J24.S2 (SHIELD)
- net 1Tx+: now reaches U17.1 (TXRX1P_A)
- net 1Tx+: now also J24.11 (TRD1+)
- net 2Tx+: now reaches U17.12 (TXRX2P_A)
- net 2Tx-: now reaches U17.13 (TXRX2M_A)
- net 2Rx+: now reaches U17.15 (TXRX2P_B)
- net 2Rx-: now reaches U17.16 (TXRX2M_B)
- net 2Tx2+: now reaches U17.17 (TXRX2P_C)
- net 2Tx2-: now reaches U17.18 (TXRX2M_C)
- net 1Tx-: now reaches U17.2 (TXRX1M_A)
- net 1Tx-: now also J24.10 (TRD1-)
- net 2Rx2+: now reaches U17.20 (TXRX2P_D)
- net 2Rx2-: now reaches U17.21 (TXRX2M_D)
- net 3Tx+: now reaches U17.24 (TXRX3P_A)
- net 3Tx-: now reaches U17.25 (TXRX3M_A)
- net 3Rx+: now reaches U17.26 (TXRX3P_B)
- net 3Rx-: now reaches U17.27 (TXRX3M_B)
- net 3Tx2+: now reaches U17.28 (TXRX3P_C)
- net 3Tx2-: now reaches U17.29 (TXRX3M_C)
- net 3Rx2+: now reaches U17.31 (TXRX3P_D)
- net 3Rx2-: now reaches U17.32 (TXRX3M_D)
- net 4Tx+: now reaches U17.34 (TXRX4P_A)
- net 4Tx-: now reaches U17.35 (TXRX4M_A)
- net 4Rx+: now reaches U17.37 (TXRX4P_B)
- net 4Rx-: now reaches U17.38 (TXRX4M_B)
- net 4Tx2+: now reaches U17.39 (TXRX4P_C)
- net 1Rx+: now reaches U17.4 (TXRX1P_B)
- net 1Rx+: now also J24.4 (TRD2+)
- net 4Tx2-: now reaches U17.40 (TXRX4M_C)
- net 4Rx2+: now reaches U17.42 (TXRX4P_D)
- net 4Rx2-: now reaches U17.43 (TXRX4M_D)
- net 1Rx-: now reaches U17.5 (TXRXIM_B)
- net 1Rx-: now also J24.5 (TRD2-)
- net 1Tx2+: now reaches U17.6 (TXRX1P_C)
- net 1Tx2+: now also J24.3 (TRD3+)
- net 1Tx2-: now reaches U17.7 (TXRX1M_C)
- net 1Tx2-: now also J24.2 (TRD3-)
- net 1Rx2+: now reaches U17.8 (TXRX1P_D)
- net 1Rx2+: now also J24.8 (TRD4+)
- net 1Rx2-: now reaches U17.9 (TXRX1M_D)
- net 1Rx2-: now also J24.9 (TRD4-)

Commit message: stuff
Parts:
- added C66: .7uf, symbol Device:C
- added C67, C69, C71: 22uf, symbol Device:C
- added C68: .9uf, symbol Device:C
- added C70: .8uf, symbol Device:C
- added C72: .3uf, symbol Device:C
- added C73: 10uf, symbol Device:C
- added L2, L4: L, symbol Device:L
Connections:
- net 1.2v: now also C70.1, C71.1, L4.2; no longer U17.10 (AVDDH), U17.111 (AVDDH__4), U17.122 (AVDDH__5), U17.128 (AVDDH__6), U17.22 (AVDDH__1), U17.33 (AVDDH__2), U17.44 (AVDDH__3)
- net 3.3v: now also C72.1, C73.1; no longer U17.114 (AVDDL__6), U17.119 (AVDDL__7), U17.124 (AVDDL__8), U17.14 (AVDDL__1), U17.19 (AVDDL__2), U17.3 (AVDDL), U17.30 (AVDDL__3), U17.36 (AVDDL__4), U17.41 (AVDDL__5)
- net GND: now also C66.2, C67.2, C68.2, C69.2, C70.2, C71.2, C72.2, C73.2
- net Xin: now also U17.95 (CLKO_25_125)
- new net: C68.1, C69.1, L4.1, U17.114 (AVDDL__6), U17.119 (AVDDL__7), U17.124 (AVDDL__8), U17.14 (AVDDL__1), U17.19 (AVDDL__2), U17.3 (AVDDL), U17.30 (AVDDL__3), U17.36 (AVDDL__4), U17.41 (AVDDL__5)
- new net: C66.1, C67.1, L2.1, U17.10 (AVDDH), U17.111 (AVDDH__4), U17.122 (AVDDH__5), U17.128 (AVDDH__6), U17.22 (AVDDH__1), U17.33 (AVDDH__2), U17.44 (AVDDH__3)
- new net 2.5v: L2.2

Commit message: stuff
Parts:
- added R44: 6.04k, symbol Device:R
- C55, C56: value 22p -> 15p
Connections:
- net GND: now also R44.1
- net SCL: now reaches U17.101 (SCL/MDC)
- net at U17.127 (ISET): now also R44.2
- net SDA: now reaches U17.98 (SDI/SDA/MDIO)
Changed lines of the file:
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@@
+	(wire
+		(pts
+			(xy 133.35 102.87) (xy 137.16 102.87)
+		)
+		(stroke
+			(width 0)
+			(type default)
+		)
+	)
 	(wire
 		(pts
@@
 	(wire
 		(pts
+			(xy 128.27 166.37) (xy 137.16 166.37)
+		)
+		(stroke
+			(width 0)
+			(type default)
+		)
+	)
+	(wire
+		(pts
 			(xy 213.36 189.23) (xy 222.25 189.23)
 		)
@@
 	(wire
 		(pts
+			(xy 125.73 102.87) (xy 125.73 106.68)
+		)
+		(stroke
+			(width 0)
+			(type default)
+		)
+	)
+	(wire
+		(pts
 			(xy 50.8 45.72) (xy 50.8 46.99)
 		)
@@
 		(pts
 			(xy 227.33 80.01) (xy 229.87 80.01)
+		)
+		(stroke
+			(width 0)
+			(type default)
+		)
+	)
+	(wire
+		(pts
+			(xy 132.08 44.45) (xy 137.16 44.45)
 		)
 		(stroke
@@
 		)
 	)
+	(label "SCL"
+		(at 132.08 44.45 0)
+		(fields_autoplaced yes)
+		(effects
+			(font
+				(size 1.27 1.27)
+			)
+			(justify left bottom)
+		)
+	)
 	(label "2Rx-"
 		(at 222.25 135.89 0)
@@
 	(label "1Tx2+"
 		(at 222.25 128.27 0)
+		(fields_autoplaced yes)
+		(effects
+			(font
+				(size 1.27 1.27)
+			)
+			(justify left bottom)
+		)
+	)
+	(label "SDA"
+		(at 128.27 166.37 0)
 		(fields_autoplaced yes)
 		(effects
@@
 			)
 		)
-		(property "Value" "22p"
+		(property "Value" "15p"
 			(at 71.12 55.8799 0)
 			(effects
@@
 			)
 		)
-		(property "Value" "22p"
+		(property "Value" "15p"
 			(at 54.61 55.8799 0)
 			(effects
@@
 	)
 	(symbol
+		(lib_id "Device:R")
+		(at 129.54 102.87 90)
+		(unit 1)
+		(exclude_from_sim no)
+		(in_bom yes)
+		(on_board yes)
+		(dnp no)
+		(fields_autoplaced yes)
+		(property "Reference" "R44"
+			(at 129.54 96.52 90)
+			(effects
+				(font
+					(size 1.27 1.27)
+				)
+			)
+		)
+		(property "Value" "6.04k"
+			(at 129.54 99.06 90)
+			(effects
+				(font
+					(size 1.27 1.27)
+				)
+			)
+		)
+		(property "Footprint" ""
+			(at 129.54 104.648 90)
+			(effects
+				(font
+					(size 1.27 1.27)
+				)
+				(hide yes)
+			)
+		)
+		(property "Datasheet" "~"
+			(at 129.54 102.87 0)
+			(effects
+				(font
+					(size 1.27 1.27)
+				)
+				(hide yes)
+			)
+		)
+		(property "Description" "Resistor"
+			(at 129.54 102.87 0)
+			(effects
+				(font
+					(size 1.27 1.27)
+				)
+				(hide yes)
+			)
+		)
+		(pin "1"
+		)
+		(pin "2"
+		)
+		(instances
+			(project ""
+				(path "/e63e39d7-6ac0-4ffd-8aa3-1841a4541b55/34e173dc-63e8-46a7-a290-a6dacd790c17"
+					(reference "R44")
+					(unit 1)
+				)
+			)
+		)
+	)
+	(symbol
 		(lib_id "Device:L")
 		(at 233.68 50.8 90)
@@
 					(unit 1)
 				)
+			)
+		)
+	)
+	(symbol
+		(lib_id "power:GND")
+		(at 125.73 106.68 0)
+		(unit 1)
+		(exclude_from_sim no)
+		(in_bom yes)
+		(on_board yes)
+		(dnp no)
+		(fields_autoplaced yes)
+		(property "Reference" "#PWR060"
+			(at 125.73 113.03 0)
+			(effects
+				(font
+					(size 1.27 1.27)
+				)
+				(hide yes)
+			)
+		)
+		(property "Value" "GND"
+			(at 125.73 111.76 0)
+			(effects
+				(font
+					(size 1.27 1.27)
+				)
+			)
+		)
+		(property "Footprint" ""
+			(at 125.73 106.68 0)
+			(effects
+				(font
+					(size 1.27 1.27)
+				)
+				(hide yes)
+			)
+		)
+		(property "Datasheet" ""
+			(at 125.73 106.68 0)
+			(effects
+				(font
+					(size 1.27 1.27)
+				)
+				(hide yes)
+			)
+		)
+		(property "Description" "Power symbol creates a global label with name \"GND\" , ground"
+			(at 125.73 106.68 0)
+			(effects
+				(font
+					(size 1.27 1.27)
+				)
+				(hide yes)
+			)
+		)
+		(pin "1"
+		)
+		(instances
+			(project ""
+				(path "/e63e39d7-6ac0-4ffd-8aa3-1841a4541b55/34e173dc-63e8-46a7-a290-a6dacd790c17"
+					(reference "#PWR060")
+					(unit 1)
+				)

Commit message: stuff
Parts:
- added C74: 1000p, symbol Device:C
- added C75, C76, C77, C78: .1u, symbol Device:C
- added C79: 1u, symbol Device:C
- added R45, R46: 100, symbol Device:R
- added U24: MIC5219-2.5YMM-TR, MSOP-8_MM_MCH, symbol MIC5219-2.5YMM-TR:MIC5219-2.5YMM-TR
Connections:
- net 2.5v: now also C79.1, U24.3 (OUT)
- net 3.3v: now also U24.1 (EN), U24.2 (IN)
- net GND: now also C74.2, C75.2, C76.1, C77.1, C78.1, C79.2, U24.5 (GND), U24.6 (GND), U24.7 (GND), U24.8 (GND); no longer J24.S1 (SHIELD), J24.S2 (SHIELD)
- net at J24.1 (TRCT3): now also C77.2
- net at J24.12 (TRCT1): now also C75.1
- net at J24.13 (VC1): now also J24.14 (VC2), J24.15 (VC3), J24.16 (VC4)
- net Led1_0: now reaches J24.17
- net at J24.18: now also R45.1
- net Led1_1: now reaches J24.19
- net Led1_1: now also U17.106 (LED1_1)
- net at J24.20: now also R46.2
- net at J24.6 (TRCT2): now also C76.2
- net at J24.7 (TRCT4): now also C78.2
- net LED1_0: now reaches U17.105 (LED1_0)
- net Led4_0: now reaches U17.85 (LED4_0)
- net Led4_1: now reaches U17.86 (LED4_1)
- net Led3_0: now reaches U17.88 (LED3_0)
- net Led3_1: now reaches U17.89 (LED3_1)
- net Led2_0: now reaches U17.91 (LED2_0)
- net Led2_1: now reaches U17.92 (LED2_1)
- new net: C74.1, J24.S1 (SHIELD), J24.S2 (SHIELD)
