File: Sensors1.kicad_sch (KiCad schematic)
At the start: 12 parts, among them U26 BNO085

Commit message: stuff
Parts:
- renumbered C24 to C82, C46 to C85, C48 to C86, R31 to R47, R32 to R48
Changed lines of the file:
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@@
 		(dnp no)
 		(fields_autoplaced yes)
-		(property "Reference" "U?"
+		(property "Reference" "U26"
 			(at 91.44 46.99 0)
 			(effects
@@
 					(unit 1)
 				)
-				(path "/e63e39d7-6ac0-4ffd-8aa3-1841a4541b55/d818c5c4-22e1-4750-8cc8-fe8a67dac1ec"
-					(reference "U?")
-					(unit 1)
-				)
 			)
 		)
@@
 		(dnp no)
 		(fields_autoplaced yes)
-		(property "Reference" "R?"
+		(property "Reference" "R49"
 			(at 48.26 48.2599 0)
 			(effects
@@
 					(unit 1)
 				)
-				(path "/e63e39d7-6ac0-4ffd-8aa3-1841a4541b55/d818c5c4-22e1-4750-8cc8-fe8a67dac1ec"
-					(reference "R?")
-					(unit 1)
-				)
 			)
 		)
@@
 		(dnp no)
 		(fields_autoplaced yes)
-		(property "Reference" "R32"
+		(property "Reference" "R48"
 			(at 26.67 43.1799 0)
 			(effects
@@
 					(unit 1)
 				)
-				(path "/e63e39d7-6ac0-4ffd-8aa3-1841a4541b55/d818c5c4-22e1-4750-8cc8-fe8a67dac1ec"
-					(reference "R32")
-					(unit 1)
-				)
 			)
 		)
@@
 		(dnp no)
 		(fields_autoplaced yes)
-		(property "Reference" "#PWR?"
+		(property "Reference" "#PWR082"
 			(at 77.47 33.02 0)
 			(effects
@@
 					(unit 1)
 				)
-				(path "/e63e39d7-6ac0-4ffd-8aa3-1841a4541b55/d818c5c4-22e1-4750-8cc8-fe8a67dac1ec"
-					(reference "#PWR?")
-					(unit 1)
-				)
 			)
 		)
@@
 		(dnp no)
 		(fields_autoplaced yes)
-		(property "Reference" "JP?"
+		(property "Reference" "JP5"
 			(at 64.77 25.4 0)
 			(effects
@@
 					(unit 1)
 				)
-				(path "/e63e39d7-6ac0-4ffd-8aa3-1841a4541b55/d818c5c4-22e1-4750-8cc8-fe8a67dac1ec"
-					(reference "JP?")
-					(unit 1)
-				)
 			)
 		)
@@
 		(dnp no)
 		(fields_autoplaced yes)
-		(property "Reference" "#PWR?"
+		(property "Reference" "#PWR088"
 			(at 144.78 55.88 0)
 			(effects
@@
 					(unit 1)
 				)
-				(path "/e63e39d7-6ac0-4ffd-8aa3-1841a4541b55/d818c5c4-22e1-4750-8cc8-fe8a67dac1ec"
-					(reference "#PWR?")
-					(unit 1)
-				)
 			)
 		)
@@
 		(dnp no)
 		(fields_autoplaced yes)
-		(property "Reference" "#PWR?"
+		(property "Reference" "#PWR087"
 			(at 139.7 99.06 0)
 			(effects
@@
 					(unit 1)
 				)
-				(path "/e63e39d7-6ac0-4ffd-8aa3-1841a4541b55/d818c5c4-22e1-4750-8cc8-fe8a67dac1ec"
-					(reference "#PWR?")
-					(unit 1)
-				)
 			)
 		)
@@
 		(dnp no)
 		(fields_autoplaced yes)
-		(property "Reference" "JP?"
+		(property "Reference" "JP4"
 			(at 64.77 20.32 0)
 			(effects
@@
 					(unit 1)
 				)
-				(path "/e63e39d7-6ac0-4ffd-8aa3-1841a4541b55/d818c5c4-22e1-4750-8cc8-fe8a67dac1ec"
-					(reference "JP?")
-					(unit 1)
-				)
 			)
 		)
@@
 		(dnp no)
 		(fields_autoplaced yes)
-		(property "Reference" "C48"
+		(property "Reference" "C86"
 			(at 214.63 57.1499 0)
 			(effects
@@
 					(unit 1)
 				)
-				(path "/e63e39d7-6ac0-4ffd-8aa3-1841a4541b55/d818c5c4-22e1-4750-8cc8-fe8a67dac1ec"
-					(reference "C48")
-					(unit 1)
-				)
 			)
 		)
@@
 		(dnp no)
 		(fields_autoplaced yes)
-		(property "Reference" "C?"
+		(property "Reference" "C83"
 			(at 148.59 39.3699 0)
 			(effects
@@
 					(unit 1)
 				)
-				(path "/e63e39d7-6ac0-4ffd-8aa3-1841a4541b55/d818c5c4-22e1-4750-8cc8-fe8a67dac1ec"
-					(reference "C?")
-					(unit 1)
-				)
 			)
 		)
@@
 		(dnp no)
 		(fields_autoplaced yes)
-		(property "Reference" "XTAL?"
+		(property "Reference" "XTAL1"
 			(at 203.2 44.45 0)
 			(effects
@@
 					(unit 1)
 				)
-				(path "/e63e39d7-6ac0-4ffd-8aa3-1841a4541b55/d818c5c4-22e1-4750-8cc8-fe8a67dac1ec"
-					(reference "XTAL?")
-					(unit 1)
-				)
 			)
 		)
@@
 		(dnp no)
 		(fields_autoplaced yes)
-		(property "Reference" "C24"
+		(property "Reference" "C82"
 			(at 143.51 82.5499 0)
 			(effects
@@
 					(unit 1)
 				)
-				(path "/e63e39d7-6ac0-4ffd-8aa3-1841a4541b55/d818c5c4-22e1-4750-8cc8-fe8a67dac1ec"
-					(reference "C24")
-					(unit 1)
-				)
 			)
 		)
@@
 		(dnp no)
 		(fields_autoplaced yes)
-		(property "Reference" "#PWR?"
+		(property "Reference" "#PWR089"
 			(at 201.93 72.39 0)
 			(effects
@@
 					(unit 1)
 				)
-				(path "/e63e39d7-6ac0-4ffd-8aa3-1841a4541b55/d818c5c4-22e1-4750-8cc8-fe8a67dac1ec"
-					(reference "#PWR?")
-					(unit 1)
-				)
 			)
 		)
@@
 		(dnp no)
 		(fields_autoplaced yes)
-		(property "Reference" "R31"
+		(property "Reference" "R47"
 			(at 21.59 43.1799 0)
 			(effects
@@
 					(unit 1)
 				)
-				(path "/e63e39d7-6ac0-4ffd-8aa3-1841a4541b55/d818c5c4-22e1-4750-8cc8-fe8a67dac1ec"
-					(reference "R31")
-					(unit 1)
-				)
 			)
 		)
@@
 		(dnp no)
 		(fields_autoplaced yes)
-		(property "Reference" "C46"
+		(property "Reference" "C85"
 			(at 198.12 57.1499 0)
 			(effects
@@
 					(unit 1)
 				)
-				(path "/e63e39d7-6ac0-4ffd-8aa3-1841a4541b55/d818c5c4-22e1-4750-8cc8-fe8a67dac1ec"
-					(reference "C46")
-					(unit 1)
-				)
 			)
 		)
@@
 		(dnp no)
 		(fields_autoplaced yes)
-		(property "Reference" "C?"
+		(property "Reference" "C84"
 			(at 161.29 39.3699 0)
 			(effects
@@
 					(unit 1)
 				)
-				(path "/e63e39d7-6ac0-4ffd-8aa3-1841a4541b55/d818c5c4-22e1-4750-8cc8-fe8a67dac1ec"
-					(reference "C?")
-					(unit 1)
-				)

Commit message: stuff
Parts:
- added R6, R7: 2.2k, symbol Device:R
- added U4: BME280, digikey-footprints:Pressure_Sensor_LGA-8_2.5x2.5mm_BME280, symbol dk_Humidity-Moisture-Sensors:BME280
Connections:
- net 3.3v: now also R6.1, R7.1, U4.2 (CSB), U4.6 (VDDIO), U4.8 (VDD)
- net GND: now also U4.1 (GND), U4.7 (GND)
- net at U26.15 (ENV_SCL): now also R6.2, U4.4 (SCK)
- net at U26.16 (ENV_SDA): now also R7.2, U4.3 (SDI)
Other:
- note added: "SENSOR PRESSURE HUMIDITY TEMP"
