File: PowerStuff.kicad_sch (KiCad schematic)
At the start: 2 parts, among them U14 INA260AIPW, U20 AZ1117IH-3.3TRG1

Commit message: stuff
Parts:
- added JP1, JP2: Jumper_2_Open, symbol Jumper:Jumper_2_Open
Connections:
- net GND: now also U14.11 (GND__1), U14.6 (GND)
- net Vs: now reaches U14.10 (VS), U20.2 (OUTPUT), U20.4 (VOUT)
- net Vs: now also JP1.1 (A), JP2.1 (A)
- net 5v: now reaches U14.14 (IN-), U14.15 (IN-__1), U14.16 (IN-__2)
- net at U14.4 (A1): now also JP1.2 (B)
- net at U14.5 (AO): now also JP2.2 (B)
- net Alert: now reaches U14.7 (ALERT)
- net SDA: now reaches U14.8 (SDA)
- net SCL: now reaches U14.9 (SCL)
- net +5V renamed 5v_EXT_Stack
- net 5v_EXT_Stack: now also U14.1 (IN+)
- new net 5v_Ext_Barrel: U14.2 (IN+__1)
- now unconnected: U14.3 (IN+__2)
Other:
- note added: "Linear Regulator"
- note added: "Power Monitor"

Commit message: stuff
Parts:
- added C12: 150u, symbol Device:C
- added D10, D11, D12, D13, D14, D15, D16, D17: LED, symbol Device:LED
- added J23: UJC-HP-L-G-5-MSMT-TR, UJC-HP-L-G-5-MSMT-TR:CUI_UJC-HP-L-G-5-MSMT-TR, symbol UJC-HP-L-G-5-MSMT-TR:UJC-HP-L-G-5-MSMT-TR
- added JP3: Jumper_2_Open, symbol Jumper:Jumper_2_Open
- added R37, R38, R39, R40, R41, R42, R43, R44: 240, symbol Device:R
- added TP7, TP8, TP9: TestPoint, symbol Connector:TestPoint
- added U12: TPS2117DRLR, TPS2117DRLR:SOTFL50P160X60-8N, symbol TPS2117DRLR:TPS2117DRLR
- added U17: LM3480IM3-5.0, LM3480IM3-5.0:SOT95P263X110-3N, symbol LM3480IM3-5.0:LM3480IM3-5.0
Connections:
- net 5v_Ext_Barrel is gone; now on net 5v_EXT_Total: U14.2 (IN+__1)
- net 5v: now also C12.1, JP3.2 (B), R42.1, R44.1, TP7.1
- net 5v_EXT_Stack: now also R41.1, U12.3 (VIN1), U12.4 (PR1), U12.5 (MODE); no longer U14.1 (IN+), U20.3 (INPUT)
- net GND: now also C12.2, D10.1 (K), D11.1 (K), D12.1 (K), D13.1 (K), D14.1 (K), D15.1 (K), D16.1 (K), D17.1 (K), J23.A12 (GND), J23.B12 (GND__1), J23.SH1 (SHIELD), J23.SH2 (SHIELD__1), J23.SH3 (SHIELD__2), J23.SH4 (SHIELD__3), TP9.1, U12.1 (GND), U17.3 (GND)
- net 5v_EXT_Total: now reaches U14.3 (IN+__2)
- net 5v_EXT_Total: now also U14.1 (IN+), U20.3 (INPUT), JP3.1 (A), R40.1, U12.2 (VOUT)
- new net: D10.2 (A), R37.2
- new net: D13.2 (A), R40.2
- new net: D12.2 (A), R39.2
- new net: D16.2 (A), R43.2
- new net: D14.2 (A), R41.2
- new net: D15.2 (A), R42.2
- new net: D17.2 (A), R44.2
- new net: R37.1, U12.8 (ST)
- new net: D11.2 (A), R38.2
- new net 3.3v: R43.1, TP8.1
- new net C_IN: J23.A9 (VBUS), J23.B9 (VBUS__1), R38.1, U17.2 (IN)
- new net C_OUT: R39.1, U12.6 (VIN2), U17.1 (OUT)
Other:
- note added: "12v to 5v"
- note added: "Power MUX"
- note added: "Power Monitor Bypass"
- note added: "USB C Power Only"

Commit message: stuff
Parts:
- removed U17: LM3480IM3-5.0, LM3480IM3-5.0:SOT95P263X110-3N, symbol LM3480IM3-5.0:LM3480IM3-5.0
- added C13, C53, C54: 22uf, symbol Device:C
- added L1: 2.2uH, symbol Device:L
- added U21: TPS63061DSCT, TPS63061DSCT:CONV_TPS63061DSCT, symbol TPS63061DSCT:TPS63061DSCT
Connections:
- net C_IN: now also C13.1, U21.2 (VIN), U21.3 (EN)
- net C_OUT: now also C54.1, U21.9 (VOUT)
- net GND: now also C13.2, C53.2, C54.2, U21.11 (PGND), U21.11_1 (PGND__1), U21.11_10 (PGND__10), U21.11_11 (PGND__11), U21.11_12 (PGND__12), U21.11_13 (PGND__13), U21.11_2 (PGND__2), U21.11_3 (PGND__3), U21.11_4 (PGND__4), U21.11_5 (PGND__5), U21.11_6 (PGND__6), U21.11_7 (PGND__7), U21.11_8 (PGND__8), U21.11_9 (PGND__9), U21.7 (GND)
- new net: L1.1, U21.1 (L1)
- new net: L1.2, U21.10 (L2)
- new net: C53.1, U21.6 (VAUX)
Other:
- note removed: "12v to 5v"
- moved on the sheet: C12, D10, D17, J23, JP3, R37, R44, U12, U20

Commit message: stuff
Parts:
- removed D17: LED, symbol Device:LED
- removed R44: 240, symbol Device:R
Connections:
- net 5v_EXT_Total: now also U12.7 (VOUT__1), U14.12 (VBUS)
Changed lines of the file:
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@@
 	)
 	(junction
+		(at 144.78 139.7)
+		(diameter 0)
+		(color 0 0 0 0)
+	)
+	(junction
 		(at 88.9 66.04)
 		(diameter 0)
@@
 	)
 	(junction
-		(at 53.34 146.05)
-		(diameter 0)
-		(color 0 0 0 0)
-	)
-	(junction
 		(at 237.49 125.73)
 		(diameter 0)
@@
 	(wire
 		(pts
-			(xy 93.98 146.05) (xy 93.98 148.59)
+			(xy 237.49 115.57) (xy 237.49 118.11)
 		)
 		(stroke
@@
 	(wire
 		(pts
-			(xy 237.49 115.57) (xy 237.49 118.11)
+			(xy 88.9 106.68) (xy 96.52 106.68)
 		)
 		(stroke
@@
 	(wire
 		(pts
-			(xy 53.34 146.05) (xy 69.85 146.05)
-		)
-		(stroke
-			(width 0)
-			(type default)
-		)
-	)
-	(wire
-		(pts
 			(xy 175.26 149.86) (xy 175.26 143.51)
 		)
@@
 	(wire
 		(pts
-			(xy 191.77 80.01) (xy 199.39 80.01)
+			(xy 144.78 142.24) (xy 144.78 139.7)
 		)
 		(stroke
@@
 	(wire
 		(pts
-			(xy 88.9 63.5) (xy 96.52 63.5)
+			(xy 191.77 80.01) (xy 199.39 80.01)
 		)
 		(stroke
@@
 	(wire
 		(pts
-			(xy 88.9 66.04) (xy 96.52 66.04)
+			(xy 88.9 63.5) (xy 96.52 63.5)
 		)
 		(stroke
@@
 	(wire
 		(pts
-			(xy 191.77 21.59) (xy 191.77 29.21)
+			(xy 88.9 66.04) (xy 96.52 66.04)
 		)
 		(stroke
@@
 	(wire
 		(pts
-			(xy 25.4 69.85) (xy 33.02 69.85)
+			(xy 191.77 21.59) (xy 191.77 29.21)
 		)
 		(stroke
@@
 	(wire
 		(pts
-			(xy 113.03 149.86) (xy 111.76 149.86)
+			(xy 25.4 69.85) (xy 33.02 69.85)
 		)
 		(stroke
@@
 	(wire
 		(pts
-			(xy 165.1 22.86) (xy 168.91 22.86)
+			(xy 113.03 149.86) (xy 111.76 149.86)
 		)
 		(stroke
@@
 	(wire
 		(pts
-			(xy 191.77 92.71) (xy 191.77 96.52)
+			(xy 165.1 22.86) (xy 168.91 22.86)
 		)
 		(stroke
@@
 	(wire
 		(pts
-			(xy 88.9 146.05) (xy 93.98 146.05)
+			(xy 191.77 92.71) (xy 191.77 96.52)
 		)
 		(stroke
@@
 	(wire
 		(pts
-			(xy 143.51 139.7) (xy 151.13 139.7)
+			(xy 143.51 139.7) (xy 144.78 139.7)
 		)
 		(stroke
@@
 	(wire
 		(pts
-			(xy 77.47 146.05) (xy 81.28 146.05)
-		)
-		(stroke
-			(width 0)
-			(type default)
-		)
-	)
-	(wire
-		(pts
 			(xy 165.1 48.26) (xy 165.1 50.8)
 		)
@@
 	(wire
 		(pts
+			(xy 143.51 142.24) (xy 144.78 142.24)
+		)
+		(stroke
+			(width 0)
+			(type default)
+		)
+	)
+	(wire
+		(pts
 			(xy 237.49 102.87) (xy 237.49 105.41)
 		)
@@
 	(wire
 		(pts
+			(xy 144.78 139.7) (xy 151.13 139.7)
+		)
+		(stroke
+			(width 0)
+			(type default)
+		)
+	)
+	(wire
+		(pts
 			(xy 237.49 105.41) (xy 237.49 107.95)
 		)
@@
 		)
 	)
+	(label "5v_EXT_Total"
+		(at 88.9 106.68 0)
+		(fields_autoplaced yes)
+		(effects
+			(font
+				(size 1.27 1.27)
+			)
+			(justify left bottom)
+		)
+	)
 	(label "Vs"
 		(at 69.85 81.28 0)
@@
 		)
 	)
+	(label "Activity LED"
+		(at 161.29 153.67 0)
+		(fields_autoplaced yes)
+		(effects
+			(font
+				(size 1.27 1.27)
+			)
+			(justify left bottom)
+		)
+	)
 	(label "Vs"
 		(at 69.85 91.44 0)
@@
 	)
 	(symbol
-		(lib_id "Device:LED")
-		(at 85.09 146.05 180)
-		(unit 1)
-		(exclude_from_sim no)
-		(in_bom yes)
-		(on_board yes)
-		(dnp no)
-		(fields_autoplaced yes)
-		(property "Reference" "D17"
-			(at 86.6775 138.43 0)
-			(effects
-				(font
-					(size 1.27 1.27)
-				)
-			)
-		)
-		(property "Value" "LED"
-			(at 86.6775 140.97 0)
-			(effects
-				(font
-					(size 1.27 1.27)
-				)
-			)
-		)
-		(property "Footprint" ""
-			(at 85.09 146.05 0)
-			(effects
-				(font
-					(size 1.27 1.27)
-				)
-				(hide yes)
-			)
-		)
-		(property "Datasheet" "~"
-			(at 85.09 146.05 0)
-			(effects
-				(font
-					(size 1.27 1.27)
-				)
-				(hide yes)
-			)
-		)
-		(property "Description" "Light emitting diode"
-			(at 85.09 146.05 0)
-			(effects
-				(font
-					(size 1.27 1.27)
-				)
-				(hide yes)
-			)
-		)
-		(pin "2"
-		)
-		(pin "1"
-		)
-		(instances
-			(project "CM4IOv5"
-				(path "/e63e39d7-6ac0-4ffd-8aa3-1841a4541b55/acb84883-a282-458c-b6f6-5a3e93f97765"
-					(reference "D17")
-					(unit 1)
-				)
-			)
-		)
-	)
-	(symbol
 		(lib_id "power:GND")
 		(at 180.34 147.32 0)
@@
 	(symbol
 		(lib_id "power:GND")
-		(at 93.98 148.59 0)
-		(unit 1)
-		(exclude_from_sim no)
-		(in_bom yes)
-		(on_board yes)
-		(dnp no)
-		(fields_autoplaced yes)
-		(property "Reference" "#PWR060"
-			(at 93.98 154.94 0)
-			(effects
-				(font
-					(size 1.27 1.27)
-				)
-				(hide yes)
-			)
-		)
-		(property "Value" "GND"
-			(at 93.98 153.67 0)
-			(effects
-				(font
-					(size 1.27 1.27)
-				)
-			)
-		)
-		(property "Footprint" ""
-			(at 93.98 148.59 0)
-			(effects
-				(font
-					(size 1.27 1.27)
-				)
-				(hide yes)
-			)
-		)
-		(property "Datasheet" ""
-			(at 93.98 148.59 0)
-			(effects
-				(font
-					(size 1.27 1.27)
-				)
-				(hide yes)
-			)
-		)
-		(property "Description" "Power symbol creates a global label with name \"GND\" , ground"
-			(at 93.98 148.59 0)
-			(effects
-				(font
-					(size 1.27 1.27)
-				)
-				(hide yes)
-			)
-		)
-		(pin "1"
-		)
-		(instances
-			(project "CM4IOv5"
-				(path "/e63e39d7-6ac0-4ffd-8aa3-1841a4541b55/acb84883-a282-458c-b6f6-5a3e93f97765"
-					(reference "#PWR060")
-					(unit 1)
-				)
-			)
-		)
-	)
-	(symbol
-		(lib_id "power:GND")
 		(at 57.15 59.69 0)
 		(unit 1)
@@
 					(unit 1)
 				)
-			)
-		)
-	)
-	(symbol
-		(lib_id "Device:R")
-		(at 73.66 146.05 90)
-		(unit 1)
-		(exclude_from_sim no)
-		(in_bom yes)
-		(on_board yes)
-		(dnp no)
-		(fields_autoplaced yes)
-		(property "Reference" "R44"
-			(at 73.66 139.7 90)
-			(effects
-				(font
-					(size 1.27 1.27)
-				)
-			)
-		)
-		(property "Value" "240"
-			(at 73.66 142.24 90)
-			(effects
-				(font
-					(size 1.27 1.27)
-				)
-			)
-		)
-		(property "Footprint" ""
-			(at 73.66 147.828 90)
-			(effects
-				(font
-					(size 1.27 1.27)
-				)
-				(hide yes)
-			)
-		)
-		(property "Datasheet" "~"
-			(at 73.66 146.05 0)
-			(effects
-				(font
-					(size 1.27 1.27)
-				)
-				(hide yes)
-			)
-		)
-		(property "Description" "Resistor"
-			(at 73.66 146.05 0)
-			(effects
-				(font
-					(size 1.27 1.27)
-				)
-				(hide yes)
-			)
-		)
-		(pin "1"
-		)
-		(pin "2"
-		)
-		(instances
-			(project "CM4IOv5"
-				(path "/e63e39d7-6ac0-4ffd-8aa3-1841a4541b55/acb84883-a282-458c-b6f6-5a3e93f97765"
-					(reference "R44")
-					(unit 1)
-				)

Commit message: stuff
Other:
- note added: "Buck/Boost Converter"
Changed lines of the file:
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@@
 		)
 	)
+	(text "Buck/Boost Converter\n"
+		(exclude_from_sim no)
+		(at 206.248 61.976 0)
+		(effects
+			(font
+				(size 1.27 1.27)
+			)
+		)
+	)
 	(text "Power Monitor Bypass"
 		(exclude_from_sim no)
@@
 			)
 		)
-		(property "Datasheet" ""
+		(property "Datasheet" "https://www.ti.com/lit/ds/symlink/ina260.pdf?HQS=dis-dk-null-digikeymode-dsf-pf-null-wwe&ts=1729222745324&ref_url=https%253A%252F%252Fwww.ti.com%252Fgeneral%252Fdocs%252Fsuppproductinfo.tsp%253FdistId%253D10%2526gotoUrl%253Dhttps%253A%252F%252Fwww.ti.com%252Flit%252Fgpn%252Fina260"
 			(at 114.3 86.36 0)
 			(effects
@@
 			)
 		)
-		(property "Datasheet" ""
+		(property "Datasheet" "https://www.sameskydevices.com/product/resource/ujc-hp-l-g-5-msmt-tr.pdf"
 			(at 152.4 30.48 0)
 			(effects
@@
 			)
 		)
-		(property "Datasheet" ""
+		(property "Datasheet" "https://www.ti.com/lit/ds/symlink/tps2117.pdf?ts=1701351126648&ref_url=https%253A%252F%252Fwww.google.com%252F"
 			(at 128.27 147.32 0)
 			(effects
@@
 			)
 		)
-		(property "Datasheet" ""
+		(property "Datasheet" "https://www.ti.com/general/docs/suppproductinfo.tsp?distId=10&gotoUrl=http%253A%252F%252Fwww.ti.com%252Flit%252Fgpn%252Ftps63061"
 			(at 219.71 85.09 0)
 			(effects
@@
 			)
 		)
-		(property "Datasheet" ""
+		(property "Datasheet" "https://www.diodes.com/assets/Datasheets/AZ1117I.pdf"
 			(at 215.9 34.29 0)
 			(effects

Commit message: stuff
Parts:
- removed C13, C53, C54: 22uf, symbol Device:C
- removed L1: 2.2uH, symbol Device:L
- removed U21: TPS63061DSCT, TPS63061DSCT:CONV_TPS63061DSCT, symbol TPS63061DSCT:TPS63061DSCT
- added C3: 10u, symbol Device:C
- added C4: 22u, symbol Device:C
- added C6: .1u, symbol Device:C
- added JP4: Jumper_2_Open, symbol Jumper:Jumper_2_Open
- added R11, R12, R13, R14, R9: 1k, symbol Device:R
- added R15, R16: 5.1k, symbol Device:R
Connections:
- net 5v_EXT_Stack: now also JP4.1 (A), R11.1, R12.1, R9.1; no longer U12.4 (PR1), U12.5 (MODE)
- net 5v_EXT_Total: now also C3.1, JP4.2 (B)
- net C_IN: now also U12.6 (VIN2)
- net C_OUT: no longer U12.6 (VIN2)
- net GND: now also C3.2, C4.2, C6.2, R13.1, R14.1, R15.2, R16.2
- net Vs: now also C4.1, C6.1
- net at JP1.2 (B), U14.4 (A1): now also R13.2
- net at JP2.2 (B), U14.5 (AO): now also R14.2
- net at J23.A5 (CC1): now also R16.1
- net at J23.B5 (CC2): now also R15.1
- net at R37.1, U12.8 (ST): now also R9.2
- new net: R11.2, U12.5 (MODE)
- new net: R12.2, U12.4 (PR1)
Other:
- note added: "BYPASS Jumper for Power Mux (in case it not working)"
- note removed: "Buck/Boost Converter"
- moved on the sheet: JP1, JP2

Commit message: stuff
Parts:
- removed D12: LED, symbol Device:LED
- removed R39: 240, symbol Device:R
- added TP2, TP4, TP6: TestPoint, symbol Connector:TestPoint
Connections:
- net 5v_EXT_Stack: now also R12.2, TP6.1; no longer R12.1
- net 5v_EXT_Total: now also TP4.1
- net C_IN: now also TP2.1
- net A1: now reaches R13.2, U14.4 (A1)
- net A1: now also JP2.2 (B); no longer JP1.2 (B)
- net A0: now reaches R14.2, U14.5 (AO)
- net A0: now also JP1.2 (B); no longer JP2.2 (B)
- net at U12.4 (PR1): now also R12.1; no longer R12.2
Other:
- note added: "Bypasses"
- note added: "Jumpers"
- note added: "Monitor Address"
- note added: "Points"
- note added: "Power Leds"
- note added: "Power Mux Bypass"
- note added: "Test"
- note removed: "BYPASS Jumper for Power Mux (in case it not working)"
- moved on the sheet: C12, C3, C4, C6, D10, D11, D13, D14, D15, D16, J23, JP1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
