File: RS485.kicad_sch (KiCad schematic)
At the start: 1 part, among them U8 MAX485CSA_T

Commit message: stuff
Parts:
- added J22: 430450212, CON_430450212_MOL, symbol 2024-10-13_01-19-49:430450212
Connections:
- net RX: now reaches U8.1 (RO)
- net RE: now reaches U8.2 (~{RE})
- net DE: now reaches U8.3 (DE)
- net TX: now reaches U8.4 (DI)
- net GND: now reaches U8.5 (GND)
- net at U8.6 (A): now also J22.2
- net at U8.7 (B): now also J22.1
- net 3.3v: now reaches U8.8 (VCC)

Commit message: stuff
Connections:
- net B: now reaches J22.1, U8.7 (B)
- net A: now reaches J22.2, U8.6 (A)
Changed lines of the file:
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@@
+		)
+	)
+	(hierarchical_label "B"
+		(shape input)
+		(at 110.49 92.71 270)
+		(fields_autoplaced yes)
+		(effects
+			(font
+				(size 1.27 1.27)
+			)
+			(justify right)
+		)
+	)
+	(hierarchical_label "A"
+		(shape input)
+		(at 110.49 90.17 90)
+		(fields_autoplaced yes)
+		(effects
+			(font
+				(size 1.27 1.27)
+			)
+			(justify left)
 		)
 	)

Commit message: stuff
Parts:
- added U23: ISO1410DWR, ISO1410DWR:SOIC127P1030X265-16N, symbol ISO1410DWR:ISO1410DWR
Connections:
- new net: U23.15 (GND2), U23.9 (GND2)
- new net: U23.2 (GND1), U23.8 (GND1)
Changed lines of the file:
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@@
+	)
+	(symbol
+		(lib_id "ISO1410DWR:ISO1410DWR")
+		(at 219.71 95.25 0)
+		(unit 1)
+		(exclude_from_sim no)
+		(in_bom yes)
+		(on_board yes)
+		(dnp no)
+		(fields_autoplaced yes)
+		(property "Reference" "U23"
+			(at 219.71 72.39 0)
+			(effects
+				(font
+					(size 1.27 1.27)
+				)
+			)
+		)
+		(property "Value" "ISO1410DWR"
+			(at 219.71 74.93 0)
+			(effects
+				(font
+					(size 1.27 1.27)
+				)
+			)
+		)
+		(property "Footprint" "ISO1410DWR:SOIC127P1030X265-16N"
+			(at 219.71 95.25 0)
+			(effects
+				(font
+					(size 1.27 1.27)
+				)
+				(justify bottom)
+				(hide yes)
+			)
+		)
+		(property "Datasheet" ""
+			(at 219.71 95.25 0)
+			(effects
+				(font
+					(size 1.27 1.27)
+				)
+				(hide yes)
+			)
+		)
+		(property "Description" ""
+			(at 219.71 95.25 0)
+			(effects
+				(font
+					(size 1.27 1.27)
+				)
+				(hide yes)
+			)
+		)
+		(property "MF" "Texas Instruments"
+			(at 219.71 95.25 0)
+			(effects
+				(font
+					(size 1.27 1.27)
+				)
+				(justify bottom)
+				(hide yes)
+			)
+		)
+		(property "Description_1" "\nEMC protected, 500-Kbps, half-duplex, 5-kVrms isolated RS-485 & RS-422 transceiver\n"
+			(at 219.71 95.25 0)
+			(effects
+				(font
+					(size 1.27 1.27)
+				)
+				(justify bottom)
+				(hide yes)
+			)
+		)
+		(property "Package" "SOIC-16 Texas Instruments"
+			(at 219.71 95.25 0)
+			(effects
+				(font
+					(size 1.27 1.27)
+				)
+				(justify bottom)
+				(hide yes)
+			)
+		)
+		(property "Price" "None"
+			(at 219.71 95.25 0)
+			(effects
+				(font
+					(size 1.27 1.27)
+				)
+				(justify bottom)
+				(hide yes)
+			)
+		)
+		(property "SnapEDA_Link" "https://www.snapeda.com/parts/ISO1410DWR/Texas+Instruments/view-part/?ref=snap"
+			(at 219.71 95.25 0)
+			(effects
+				(font
+					(size 1.27 1.27)
+				)
+				(justify bottom)
+				(hide yes)
+			)
+		)
+		(property "MP" "ISO1410DWR"
+			(at 219.71 95.25 0)
+			(effects
+				(font
+					(size 1.27 1.27)
+				)
+				(justify bottom)
+				(hide yes)
+			)
+		)
+		(property "Availability" "In Stock"
+			(at 219.71 95.25 0)
+			(effects
+				(font
+					(size 1.27 1.27)
+				)
+				(justify bottom)
+				(hide yes)
+			)
+		)
+		(property "Check_prices" "https://www.snapeda.com/parts/ISO1410DWR/Texas+Instruments/view-part/?ref=eda"
+			(at 219.71 95.25 0)
+			(effects
+				(font
+					(size 1.27 1.27)
+				)
+				(justify bottom)
+				(hide yes)
+			)
+		)
+		(pin "3"
+		)
+		(pin "9"
+		)
+		(pin "4"
+		)
+		(pin "1"
+		)
+		(pin "5"
+		)
+		(pin "6"
+		)
+		(pin "12"
+		)
+		(pin "16"
+		)
+		(pin "15"
+		)
+		(pin "2"
+		)
+		(pin "13"
+		)
+		(pin "8"
+		)
+		(instances
+			(project ""
+				(path "/e63e39d7-6ac0-4ffd-8aa3-1841a4541b55/92056ffc-70e5-4b84-9d1d-3f511482facd"
+					(reference "U23")
+					(unit 1)
+				)
+			)
+		)
 	)
 	(symbol

Commit message: stuff
Parts:
- added C7: .1u, symbol Device:C
Connections:
- net 3.3v: now also C7.1
- net GND: now also C7.2
Changed lines of the file:
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@@
 	(generator_version "8.0")
 	(paper "A4")
+	(junction
+		(at 181.61 78.74)
+		(diameter 0)
+		(color 0 0 0 0)
+	)
 	(wire
 		(pts
@@
 	(wire
 		(pts
-			(xy 166.37 78.74) (xy 171.45 78.74)
+			(xy 166.37 78.74) (xy 181.61 78.74)
 		)
 		(stroke
@@
 	(wire
 		(pts
-			(xy 171.45 74.93) (xy 171.45 78.74)
+			(xy 181.61 76.2) (xy 181.61 78.74)
 		)
 		(stroke
@@
 	(hierarchical_label "3.3v"
 		(shape input)
-		(at 171.45 74.93 0)
+		(at 181.61 76.2 0)
 		(fields_autoplaced yes)
 		(effects
@@
 	(symbol
 		(lib_id "power:GND")
+		(at 181.61 86.36 0)
+		(unit 1)
+		(exclude_from_sim no)
+		(in_bom yes)
+		(on_board yes)
+		(dnp no)
+		(fields_autoplaced yes)
+		(property "Reference" "#PWR011"
+			(at 181.61 92.71 0)
+			(effects
+				(font
+					(size 1.27 1.27)
+				)
+				(hide yes)
+			)
+		)
+		(property "Value" "GND"
+			(at 181.61 91.44 0)
+			(effects
+				(font
+					(size 1.27 1.27)
+				)
+			)
+		)
+		(property "Footprint" ""
+			(at 181.61 86.36 0)
+			(effects
+				(font
+					(size 1.27 1.27)
+				)
+				(hide yes)
+			)
+		)
+		(property "Datasheet" ""
+			(at 181.61 86.36 0)
+			(effects
+				(font
+					(size 1.27 1.27)
+				)
+				(hide yes)
+			)
+		)
+		(property "Description" "Power symbol creates a global label with name \"GND\" , ground"
+			(at 181.61 86.36 0)
+			(effects
+				(font
+					(size 1.27 1.27)
+				)
+				(hide yes)
+			)
+		)
+		(pin "1"
+		)
+		(instances
+			(project ""
+				(path "/e63e39d7-6ac0-4ffd-8aa3-1841a4541b55/92056ffc-70e5-4b84-9d1d-3f511482facd"
+					(reference "#PWR011")
+					(unit 1)
+				)
+			)
+		)
+	)
+	(symbol
+		(lib_id "power:GND")
 		(at 172.72 111.76 0)
 		(unit 1)
@@
 					(unit 1)
 				)
+			)
+		)
+	)
+	(symbol
+		(lib_id "Device:C")
+		(at 181.61 82.55 0)
+		(unit 1)
+		(exclude_from_sim no)
+		(in_bom yes)
+		(on_board yes)
+		(dnp no)
+		(fields_autoplaced yes)
+		(property "Reference" "C7"
+			(at 185.42 81.2799 0)
+			(effects
+				(font
+					(size 1.27 1.27)
+				)
+				(justify left)
+			)
+		)
+		(property "Value" ".1u"
+			(at 185.42 83.8199 0)
+			(effects
+				(font
+					(size 1.27 1.27)
+				)
+				(justify left)
+			)
+		)
+		(property "Footprint" ""
+			(at 182.5752 86.36 0)
+			(effects
+				(font
+					(size 1.27 1.27)
+				)
+				(hide yes)
+			)
+		)
+		(property "Datasheet" "~"
+			(at 181.61 82.55 0)
+			(effects
+				(font
+					(size 1.27 1.27)
+				)
+				(hide yes)
+			)
+		)
+		(property "Description" "Unpolarized capacitor"
+			(at 181.61 82.55 0)
+			(effects
+				(font
+					(size 1.27 1.27)
+				)
+				(hide yes)
+			)
+		)
+		(pin "2"
+		)
+		(pin "1"
+		)
+		(instances
+			(project ""
+				(path "/e63e39d7-6ac0-4ffd-8aa3-1841a4541b55/92056ffc-70e5-4b84-9d1d-3f511482facd"
+					(reference "C7")
+					(unit 1)
+				)

Commit message: stuff
Other:
- note added: "Galvanicly Isolated RS485 Transceiver"
- note added: "RS485 Header"
- note added: "RS485 Transceiver"
- moved on the sheet: C7, J22, U23, U8

Commit message: stuff
Parts:
- added T1: DA2304-ALD, DA2304-ALD:XFMR_DA2304-ALD, symbol DA2304-ALD:DA2304-ALD
- added U4: LP2985A-50DBVR, LP2985A-50DBVR:SOT95P280X145-5N, symbol LP2985A-50DBVR:LP2985A-50DBVR
Other:
- moved on the sheet: U23

Commit message: stuff
Parts:
- removed U23: ISO1410DWR, ISO1410DWR:SOIC127P1030X265-16N, symbol ISO1410DWR:ISO1410DWR
- added C10, C11: C, symbol Device:C
- added C19: .1u, symbol Device:C
- added C20: 10n, symbol Device:C
- added C21: 4.7u, symbol Device:C
- added C9: 10u, symbol Device:C
- added D12, D17: MBR0520LT, Diode_SMD:D_SOD-123, symbol Diode:MBR0520LT
- added J11: 430450212, CON_430450212_MOL, symbol 2024-10-13_01-19-49:430450212
- added U6: ISO3086TDW, DW16, symbol ISO3086T:ISO3086TDW
Connections:
- net RE is gone; now on net DE: U8.2 (~{RE})
- net DE: now also U6.6 (*RE), U6.7 (DE)
- net GND: now also C9.1
- net RX: now also U6.5 (R)
- net TX: now also U6.8 (D)
- net D1: now reaches T1.1
- net D1: now also U6.1 (D1)
- net VCC1: now reaches T1.2
- net VCC1: now also T1.3, C9.2, U6.4 (VCC1)
- net D2: now reaches T1.4
- net D2: now also U6.2 (D2)
- net at T1.5: now also D17.2 (A)
- net GND2: now reaches T1.6
- net GND2: now also T1.7, U4.2 (GND), C10.2, C11.2, C19.1, C20.2, C21.1, U6.15 (GND2), U6.9 (GND2)
- net at T1.8: now also D12.2 (A)
- net Vin: now reaches U4.1 (VIN)
- net Vin: now also U4.3 (ON/~{OFF}), C10.1, C11.1, D12.1 (K), D17.1 (K)
- net at U4.4 (BYPASS): now also C20.1
- net VCC2: now reaches U4.5 (VOUT)
- net VCC2: now also C19.2, C21.2, U6.16 (VCC2)
- new net GND1: U6.3 (GND1)
- new net TB_A: J11.2, U6.11 (Y), U6.14 (A)
- new net TB_B: J11.1, U6.12 (Z), U6.13 (B)
Other:
- note added: "Transformer"
- note added: "Voltage Regulator"
- moved on the sheet: J22, T1, U4
