File: RS485.kicad_sch (KiCad schematic)
At the start: 15 parts, among them J11 430450212, J22 430450212, T1 DA2304-ALD, U4 LP2985A-50DBVR, U6 ISO3086TDW, U8 MAX485CSA_T

Commit message: stuff
Connections:
- net DE: no longer U6.6 (*RE), U6.7 (DE), U8.2 (~{RE})
- new net RE: U8.2 (~{RE})
- new net TB_EN: U6.6 (*RE), U6.7 (DE)
Changed lines of the file:
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@@
-		)
-	)
-	(label "RE"
-		(at 133.35 55.88 0)
-		(fields_autoplaced yes)
-		(effects
-			(font
-				(size 1.27 1.27)
-			)
-			(justify left bottom)
 		)
 	)
@@
 		(fields_autoplaced yes)
 		(effects
-			(font
-				(size 1.27 1.27)
-			)
-			(justify left bottom)
-		)
-	)
-	(label "DE"
-		(at 133.35 58.42 0)
-		(fields_autoplaced yes)
-		(effects

Commit message: stuff
Parts:
- added R30, R39, R44, R45: 10k, symbol Device:R
Connections:
- net GND1 is gone; now on net GND: U6.3 (GND1)
- net A: now also R30.1
- net B: now also R39.1
- net GND: now also R39.2, R45.2
- net TB_A: now also R44.1
- net TB_B: now also R45.1
- new net +5V: R30.2, R44.2
- no-connect marks 0 -> 1

Commit message: stuff
Changed lines of the file:
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@@
+	)
+	(label "TB_B"
+		(at 203.2 52.07 0)
+		(fields_autoplaced yes)
+		(effects
+			(font
+				(size 1.27 1.27)
+			)
+			(justify left bottom)
+		)
 	)
 	(label "TB_B"
@@
 		)
 	)
-	(label "D"
-		(at 133.35 60.96 0)
-		(fields_autoplaced yes)
-		(effects
-			(font
-				(size 1.27 1.27)
-			)
-			(justify left bottom)
-		)
-	)
-	(label "R"
-		(at 133.35 53.34 0)
-		(fields_autoplaced yes)
-		(effects
-			(font
-				(size 1.27 1.27)
-			)
-			(justify left bottom)
-		)
-	)
 	(label "GND2"
 		(at 203.2 60.96 180)
@@
 		)
 	)
+	(label "TB_A"
+		(at 203.2 49.53 0)
+		(fields_autoplaced yes)
+		(effects
+			(font
+				(size 1.27 1.27)
+			)
+			(justify left bottom)
+		)
+	)
 	(label "D2"
 		(at 41.91 101.6 0)
@@
 		)
 	)
-	(hierarchical_label "TB_A"
-		(shape input)
-		(at 203.2 49.53 0)
-		(fields_autoplaced yes)
-		(effects
-			(font
-				(size 1.27 1.27)
-			)
-			(justify left)
-		)
-	)
-	(hierarchical_label "TB_B"
-		(shape input)
-		(at 203.2 52.07 0)
-		(fields_autoplaced yes)
-		(effects
-			(font
-				(size 1.27 1.27)
-			)
-			(justify left)
-		)
-	)

Commit message: stuff
Connections:
- net 3.3v renamed +3.3V
Changed lines of the file:
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@@
 		)
 	)
-	(hierarchical_label "3.3v"
+	(hierarchical_label "TB_EN"
 		(shape input)
-		(at 92.71 34.29 0)
+		(at 133.35 57.15 180)
 		(fields_autoplaced yes)
 		(effects
@@
 				(size 1.27 1.27)
 			)
-			(justify left)
-		)
-	)
-	(hierarchical_label "TB_EN"
+			(justify right)
+		)
+	)
+	(hierarchical_label "RX"
 		(shape input)
-		(at 133.35 57.15 180)
+		(at 82.55 46.99 0)
 		(fields_autoplaced yes)
 		(effects
@@
 				(size 1.27 1.27)
 			)
-			(justify right)
-		)
-	)
-	(hierarchical_label "RX"
+			(justify left)
+		)
+	)
+	(hierarchical_label "TX"
 		(shape input)
-		(at 82.55 46.99 0)
+		(at 36.83 41.91 180)
 		(fields_autoplaced yes)
 		(effects
@@
 				(size 1.27 1.27)
 			)
-			(justify left)
-		)
-	)
-	(hierarchical_label "TX"
+			(justify right)
+		)
+	)
+	(hierarchical_label "B"
 		(shape input)
-		(at 36.83 41.91 180)
+		(at 36.83 57.15 180)
 		(fields_autoplaced yes)
 		(effects
@@
 		)
 	)
-	(hierarchical_label "B"
+	(hierarchical_label "A"
 		(shape input)
-		(at 36.83 57.15 180)
+		(at 36.83 52.07 180)
 		(fields_autoplaced yes)
 		(effects
@@
 		)
 	)
-	(hierarchical_label "A"
+	(hierarchical_label "RE"
 		(shape input)
-		(at 36.83 52.07 180)
+		(at 82.55 41.91 0)
 		(fields_autoplaced yes)
 		(effects
@@
 				(size 1.27 1.27)
 			)
-			(justify right)
-		)
-	)
-	(hierarchical_label "RE"
+			(justify left)
+		)
+	)
+	(hierarchical_label "DE"
 		(shape input)
-		(at 82.55 41.91 0)
+		(at 82.55 44.45 0)
 		(fields_autoplaced yes)
 		(effects
@@
 		)
 	)
-	(hierarchical_label "DE"
-		(shape input)
-		(at 82.55 44.45 0)
-		(fields_autoplaced yes)
-		(effects
-			(font
-				(size 1.27 1.27)
-			)
-			(justify left)
-		)
-	)
 	(symbol
 		(lib_id "2024-10-13_01-19-49:430450212")
@@
 					(unit 1)
 				)
+			)
+		)
+	)
+	(symbol
+		(lib_id "power:+3.3V")
+		(at 92.71 34.29 0)
+		(unit 1)
+		(exclude_from_sim no)
+		(in_bom yes)
+		(on_board yes)
+		(dnp no)
+		(fields_autoplaced yes)
+		(property "Reference" "#PWR0133"
+			(at 92.71 38.1 0)
+			(effects
+				(font
+					(size 1.27 1.27)
+				)
+				(hide yes)
+			)
+		)
+		(property "Value" "+3.3V"
+			(at 92.71 29.21 0)
+			(effects
+				(font
+					(size 1.27 1.27)
+				)
+			)
+		)
+		(property "Footprint" ""
+			(at 92.71 34.29 0)
+			(effects
+				(font
+					(size 1.27 1.27)
+				)
+				(hide yes)
+			)
+		)
+		(property "Datasheet" ""
+			(at 92.71 34.29 0)
+			(effects
+				(font
+					(size 1.27 1.27)
+				)
+				(hide yes)
+			)
+		)
+		(property "Description" "Power symbol creates a global label with name \"+3.3V\""
+			(at 92.71 34.29 0)
+			(effects
+				(font
+					(size 1.27 1.27)
+				)
+				(hide yes)
+			)
+		)
+		(pin "1"
+		)
+		(instances
+			(project ""
+				(path "/e63e39d7-6ac0-4ffd-8aa3-1841a4541b55/92056ffc-70e5-4b84-9d1d-3f511482facd"
+					(reference "#PWR0133")
+					(unit 1)
+				)

Commit message: stuff
Changed lines of the file:
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@@
-		)
-	)
-	(label "GND1"
-		(at 133.35 48.26 0)
-		(fields_autoplaced yes)
-		(effects
-			(font
-				(size 1.27 1.27)
-			)
-			(justify left bottom)
 		)
 	)

Commit message: stuff
Parts:
- C10, C11: value C -> 1u
Connections:
- net VCC1 is gone; now on net +3.3V: C9.2, T1.2, T1.3, U6.4 (VCC1)

Commit message: assigned footprints
Parts:
- C10, C11, C19, C20, C21, C7, C9: footprint (none) -> Capacitor_SMD:C_0805_2012Metric
- J11, J22: footprint CON_430450212_MOL -> RS485-Header:CON_430450212_MOL
- R30, R39, R44, R45: footprint (none) -> Resistor_SMD:R_0805_2012Metric
- U4: footprint LP2985A-50DBVR:SOT95P280X145-5N -> LP2985A_50DBVR:SOT95P280X145-5N
- U6: footprint DW16 -> ISO3086TDW:DW16
Changed lines of the file:
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@@
 			)
 		)
-		(property "Footprint" "CON_430450212_MOL"
+		(property "Footprint" "RS485-Header:CON_430450212_MOL"
 			(at 259.08 41.91 0)
 			(effects
@@
 			)
 		)
-		(property "Footprint" ""
+		(property "Footprint" "Capacitor_SMD:C_0805_2012Metric"
 			(at 89.8652 110.49 0)
 			(effects
@@
 			)
 		)
-		(property "Footprint" ""
+		(property "Footprint" "Resistor_SMD:R_0805_2012Metric"
 			(at 215.9 98.298 90)
 			(effects
@@
 			)
 		)
-		(property "Footprint" ""
+		(property "Footprint" "Resistor_SMD:R_0805_2012Metric"
 			(at 214.63 118.618 90)
 			(effects
@@
 			)
 		)
-		(property "Footprint" ""
+		(property "Footprint" "Resistor_SMD:R_0805_2012Metric"
 			(at 215.9 94.488 90)
 			(effects
@@
 			)
 		)
-		(property "Footprint" ""
+		(property "Footprint" "Resistor_SMD:R_0805_2012Metric"
 			(at 214.63 122.428 90)
 			(effects
@@
 			)
 		)
-		(property "Footprint" "DW16"
+		(property "Footprint" "ISO3086TDW:DW16"
 			(at 138.43 43.18 0)
 			(effects
@@
 			)
 		)
-		(property "Footprint" ""
+		(property "Footprint" "Capacitor_SMD:C_0805_2012Metric"
 			(at 204.1652 43.18 0)
 			(effects
@@
 			)
 		)
-		(property "Footprint" ""
+		(property "Footprint" "Capacitor_SMD:C_0805_2012Metric"
 			(at 41.91 108.2548 0)
 			(effects
@@
 			)
 		)
-		(property "Footprint" ""
+		(property "Footprint" "Capacitor_SMD:C_0805_2012Metric"
 			(at 214.3252 43.18 0)
 			(effects
@@
 			)
 		)
-		(property "Footprint" "CON_430450212_MOL"
+		(property "Footprint" "RS485-Header:CON_430450212_MOL"
 			(at 259.08 58.42 0)
 			(effects
@@
 			)
 		)
-		(property "Footprint" "LP2985A-50DBVR:SOT95P280X145-5N"
+		(property "Footprint" "LP2985A_50DBVR:SOT95P280X145-5N"
 			(at 149.86 110.49 0)
 			(effects
@@
 			)
 		)
-		(property "Footprint" ""
+		(property "Footprint" "Capacitor_SMD:C_0805_2012Metric"
 			(at 129.2352 119.38 0)
 			(effects
@@
 			)
 		)
-		(property "Footprint" ""
+		(property "Footprint" "Capacitor_SMD:C_0805_2012Metric"
 			(at 79.7052 110.49 0)
 			(effects
@@
 			)
 		)
-		(property "Footprint" ""
+		(property "Footprint" "Capacitor_SMD:C_0805_2012Metric"
 			(at 93.6752 44.45 0)
 			(effects

Commit message: stuff
Parts:
- removed C10, C11: 1u, Capacitor_SMD:C_0805_2012Metric, symbol Device:C
- removed C19: .1u, Capacitor_SMD:C_0805_2012Metric, symbol Device:C
- removed C21: 4.7u, Capacitor_SMD:C_0805_2012Metric, symbol Device:C
- removed C9: 10u, Capacitor_SMD:C_0805_2012Metric, symbol Device:C
- removed D12, D17: MBR0520LT, Diode_SMD:D_SOD-123, symbol Diode:MBR0520LT
- removed T1: DA2304-ALD, DA2304-ALD:XFMR_DA2304-ALD, symbol DA2304-ALD:DA2304-ALD
- removed U6: ISO3086TDW, ISO3086TDW:DW16, symbol ISO3086T:ISO3086TDW
- added U6: ISOW1432BDFMR, ISOW1432BDFMR:SOIC127P1030X355-20N, symbol ISOW1432BDFMR:ISOW1432BDFMR
Connections:
- no-connect marks 1 -> 0
Other:
- note added: "Pull Up Resistors"
- note removed: "Galvanicly Isolated RS485 Transceiver"
- note removed: "Transformer"
- moved on the sheet: C20, R30, R39, R44, R45, U4
