File: RS485.kicad_sch (KiCad schematic)
At the start: 11 parts, among them J11 430450212, J22 430450212, U4 LP2985A-50DBVR, U6 ISOW1432BDFMR, U8 MAX485CSA_T

Commit message: stuff
Parts:
- added C10, C25: 10n, symbol Device:C
- added C11, C26: 1u, symbol Device:C
- added C19, C24, C27: 10u, symbol Device:C
- added C21, C9: .1u, symbol Device:C
- added FB1, FB2, FB3, FB4, FB5: FerriteBead, symbol Device:FerriteBead
- added R46: 5k, symbol Device:R
- added R49: 120, symbol Device:R
Connections:
- net +3.3V: now also FB1.1
- net +5V: now also FB2.1; no longer R44.2
- net GND: now also U6.6 (GNDIO), C9.2, FB3.2; no longer R45.2
- net GND2: now also R45.2, U6.15 (GISOIN), C21.2, C24.2, FB5.2
- net TB_A: now also U6.17 (Y), U6.20 (A), R49.2
- net TB_B: now also U6.18 (Z), U6.19 (B), R49.1
- net VCC2: now also R44.2, U6.16 (VISOIN), C21.1, C24.1, FB4.2
- net at U6.1 (VIO): now also C9.1, FB1.2, R46.1
- net at U6.10 (GND1): now also C10.2, C11.2, C19.2, FB3.1
- net at U6.11 (GND2): now also U6.13 (MODE), C25.2, C26.2, C27.2, FB5.1
- net at U6.12 (VISOOUT): now also C25.1, C26.1, C27.1, FB4.1
- net TX_TB: now reaches U6.2 (D)
- net TB_EN: now reaches U6.3 (DE)
- net TB_EN: now also U6.5 (~{RE})
- net RX_TB: now reaches U6.4 (R)
- net ISO_FLT: now reaches U6.8 (EN/FLT)
- net ISO_FLT: now also R46.2
- net at U6.9 (VDD): now also C10.1, C11.1, C19.1, FB2.2
- no-connect marks 0 -> 2
Other:
- note added: "Isolated RS485 Transceiver"
- moved on the sheet: U6

Commit message: stuff
Parts:
- removed FB5: FerriteBead, symbol Device:FerriteBead
- added FB6: FerriteBead, CM4IO:L_Bourns_SRN6045TA, symbol Device:FerriteBead
- C10, C11, C19, C21, C24, C25, C26, C27, C9: footprint (none) -> Capacitor_SMD:C_0805_2012Metric
- FB1, FB2, FB3, FB4: footprint (none) -> CM4IO:L_Bourns_SRN6045TA
- R46, R49: footprint (none) -> Resistor_SMD:R_0805_2012Metric
Connections:
- net +3.3V: now also FB6.1; no longer FB1.1
- net +5V: now also FB1.1; no longer FB2.1
- net GND: now also FB2.1; no longer FB3.2
- net GND2: now also FB4.2
- net VCC2: now also FB3.2; no longer FB4.2
- net at C10.1, C11.1, C19.1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: now also FB1.2; no longer FB2.2
- net at C10.2, C11.2, C19.2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: now also FB2.2; no longer FB3.1
- net at C25.2, C26.2, C27.2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: now also FB4.1
- net at C9.1, R46.1, U6.1 (VIO): now also FB6.2; no longer FB1.2
- net at C25.1, C26.1, C27.1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: now also FB3.1; no longer FB4.1

Commit message: STUFF
Connections:
- net A renamed A+
- net B renamed A-
- net TB_A renamed TB+
- net TB_B renamed TB-
Changed lines of the file:
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@@
+	(wire
+		(pts
+			(xy 57.15 91.44) (xy 57.15 99.06)
+		)
+		(stroke
+			(width 0)
+			(type default)
+		)
+	)
+	(wire
+		(pts
+			(xy 153.67 149.86) (xy 153.67 152.4)
+		)
+		(stroke
+			(width 0)
+			(type default)
+		)
+	)
+	(wire
+		(pts
+			(xy 106.68 119.38) (xy 106.68 121.92)
+		)
+		(stroke
+			(width 0)
+			(type default)
+		)
+	)
 	(wire
 		(pts
 			(xy 36.83 57.15) (xy 41.91 57.15)
-		)
-		(stroke
-			(width 0)
-			(type default)
-		)
-	)
-	(wire
-		(pts
-			(xy 57.15 91.44) (xy 57.15 99.06)
-		)
-		(stroke
-			(width 0)
-			(type default)
-		)
-	)
-	(wire
-		(pts
-			(xy 153.67 149.86) (xy 153.67 152.4)
-		)
-		(stroke
-			(width 0)
-			(type default)
-		)
-	)
-	(wire
-		(pts
-			(xy 106.68 119.38) (xy 106.68 121.92)
 		)
 		(stroke
@@
 		)
 	)
-	(label "TB_A"
-		(at 193.04 62.23 0)
-		(fields_autoplaced yes)
-		(effects
-			(font
-				(size 1.27 1.27)
-			)
-			(justify left bottom)
-		)
-	)
-	(label "TB_B"
-		(at 193.04 66.04 0)
-		(fields_autoplaced yes)
-		(effects
-			(font
-				(size 1.27 1.27)
-			)
-			(justify left bottom)
-		)
-	)
-	(label "TB_B"
+	(label "A-"
+		(at 194.31 41.91 0)
+		(fields_autoplaced yes)
+		(effects
+			(font
+				(size 1.27 1.27)
+			)
+			(justify left bottom)
+		)
+	)
+	(label "TB-"
 		(at 260.35 58.42 0)
 		(fields_autoplaced yes)
@@
 		)
 	)
-	(label "B"
-		(at 260.35 41.91 0)
+	(label "TB+"
+		(at 119.38 121.92 0)
 		(fields_autoplaced yes)
 		(effects
@@
 		)
 	)
-	(label "A"
+	(label "A+"
 		(at 36.83 52.07 0)
 		(fields_autoplaced yes)
@@
 		)
 	)
-	(label "TB_A"
-		(at 119.38 121.92 0)
-		(fields_autoplaced yes)
-		(effects
-			(font
-				(size 1.27 1.27)
-			)
-			(justify left bottom)
-		)
-	)
-	(label "A"
+	(label "A-"
+		(at 260.35 41.91 0)
+		(fields_autoplaced yes)
+		(effects
+			(font
+				(size 1.27 1.27)
+			)
+			(justify left bottom)
+		)
+	)
+	(label "TB+"
+		(at 260.35 55.88 0)
+		(fields_autoplaced yes)
+		(effects
+			(font
+				(size 1.27 1.27)
+			)
+			(justify left bottom)
+		)
+	)
+	(label "TB+"
+		(at 193.04 62.23 0)
+		(fields_autoplaced yes)
+		(effects
+			(font
+				(size 1.27 1.27)
+			)
+			(justify left bottom)
+		)
+	)
+	(label "A+"
 		(at 260.35 39.37 0)
 		(fields_autoplaced yes)
@@
 		)
 	)
-	(label "A"
+	(label "A+"
 		(at 194.31 38.1 0)
-		(fields_autoplaced yes)
-		(effects
-			(font
-				(size 1.27 1.27)
-			)
-			(justify left bottom)
-		)
-	)
-	(label "B"
-		(at 36.83 57.15 0)
 		(fields_autoplaced yes)
 		(effects
@@
 		)
 	)
-	(label "TB_B"
+	(label "TB-"
 		(at 119.38 114.3 0)
 		(fields_autoplaced yes)
@@
 		)
 	)
-	(label "B"
-		(at 194.31 41.91 0)
-		(fields_autoplaced yes)
-		(effects
-			(font
-				(size 1.27 1.27)
-			)
-			(justify left bottom)
-		)
-	)
-	(label "TB_A"
-		(at 260.35 55.88 0)
+	(label "TB-"
+		(at 193.04 66.04 0)
 		(fields_autoplaced yes)
 		(effects
@@
 		)
 	)
-	(hierarchical_label "B"
+	(hierarchical_label "A-"
 		(shape input)
 		(at 36.83 57.15 180)
@@
 		)
 	)
-	(hierarchical_label "A"
+	(hierarchical_label "A+"
 		(shape input)
 		(at 36.83 52.07 180)
