File: CM4_GPIO.kicad_sch (KiCad schematic)
At the start: 28 parts, among them J1 Conn_01x03, J2 Conn_02x07_Odd_Even, J3 Conn_01x03, J7 Micro_SD_Card_Det, J8 THD-20-R, J9 THD-02-R, U1 TPD4EUSB30, U18 RT9742GGJ5, U2 TPD4EUSB30, U3 MagJack-A70-112-331N126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

Commit message: stuff
Changed lines of the file:
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@@
+		)
+	)
+	(hierarchical_label "TX"
+		(shape output)
+		(at 114.3 82.55 0)
+		(fields_autoplaced yes)
+		(effects
+			(font
+				(size 1.27 1.27)
+			)
+			(justify left)
+		)
+	)
+	(hierarchical_label "RX"
+		(shape output)
+		(at 114.3 87.63 0)
+		(fields_autoplaced yes)
+		(effects
+			(font
+				(size 1.27 1.27)
+			)
+			(justify left)
+		)
+	)
+	(hierarchical_label "Int"
+		(shape output)
+		(at 114.3 80.01 0)
+		(fields_autoplaced yes)
+		(effects
+			(font
+				(size 1.27 1.27)
+			)
+			(justify left)
+		)
+	)
+	(hierarchical_label "Rst"
+		(shape output)
+		(at 114.3 74.93 0)
+		(fields_autoplaced yes)
+		(effects
+			(font
+				(size 1.27 1.27)
+			)
+			(justify left)
 		)
 	)
@@
 		)
 	)
+	(hierarchical_label "Boot"
+		(shape output)
+		(at 114.3 77.47 0)
+		(fields_autoplaced yes)
+		(effects
+			(font
+				(size 1.27 1.27)
+			)
+			(justify left)
+		)
+	)

Commit message: stuff
Connections:
- net GPIO25: no longer Module1.41 (GPIO25)
- net GPIO8: no longer Module1.39 (GPIO8)
- new net Alert: Module1.41 (GPIO25)
- new net Leak: Module1.39 (GPIO8)
Changed lines of the file:
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@@
 		)
 	)
-	(label "GPIO8"
+	(label "Leak"
 		(at 108.966 67.31 180)
 		(fields_autoplaced yes)
@@
 		)
 	)
-	(label "GPIO25"
+	(label "Alert"
 		(at 110.236 69.85 180)
 		(fields_autoplaced yes)
@@
 		)
 	)
+	(hierarchical_label "Leak"
+		(shape output)
+		(at 114.3 67.31 0)
+		(fields_autoplaced yes)
+		(effects
+			(font
+				(size 1.27 1.27)
+			)
+			(justify left)
+		)
+	)
 	(hierarchical_label "TX"
 		(shape output)
@@
 		(fields_autoplaced yes)
 		(effects
+			(font
+				(size 1.27 1.27)
+			)
+			(justify left)
+		)
+	)
+	(hierarchical_label "Alert"
+		(shape output)
+		(at 114.3 69.85 0)
+		(fields_autoplaced yes)
+		(effects

Commit message: stuff
Connections:
- net GPIO12: no longer Module1.31 (GPIO12)
- net GPIO16: no longer Module1.29 (GPIO16)
- new net DE: Module1.31 (GPIO12)
- new net RE: Module1.29 (GPIO16)
Changed lines of the file:
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@@
 		)
 	)
-	(label "GPIO12"
+	(label "DE"
 		(at 110.236 57.15 180)
 		(fields_autoplaced yes)
@@
 		)
 	)
-	(label "GPIO16"
+	(label "RE"
 		(at 110.236 54.61 180)
 		(fields_autoplaced yes)
@@
 		)
 	)
+	(hierarchical_label "RE"
+		(shape output)
+		(at 114.3 54.61 0)
+		(fields_autoplaced yes)
+		(effects
+			(font
+				(size 1.27 1.27)
+			)
+			(justify left)
+		)
+	)
 	(hierarchical_label "Leak"
 		(shape output)
@@
 		)
 	)
+	(hierarchical_label "DE"
+		(shape output)
+		(at 114.3 57.15 0)
+		(fields_autoplaced yes)
+		(effects
+			(font
+				(size 1.27 1.27)
+			)
+			(justify left)
+		)
+	)

Commit message: stuff
Connections:
- net GPIO20: no longer Module1.27 (GPIO20)
- net GPIO21: no longer Module1.25 (GPIO21)
- new net OE_PWM: Module1.25 (GPIO21)
- new net n_reset: Module1.27 (GPIO20)
Changed lines of the file:
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@@
 		)
 	)
-	(label "GPIO20"
+	(label "n_reset"
 		(at 110.236 52.07 180)
 		(fields_autoplaced yes)
@@
 		)
 	)
-	(label "GPIO21"
+	(label "OE_PWM"
 		(at 110.236 49.53 180)
 		(fields_autoplaced yes)
@@
 		)
 	)
+	(hierarchical_label "OE_PWM"
+		(shape output)
+		(at 114.3 49.53 0)
+		(fields_autoplaced yes)
+		(effects
+			(font
+				(size 1.27 1.27)
+			)
+			(justify left)
+		)
+	)
 	(hierarchical_label "TX"
 		(shape output)
@@
 		(fields_autoplaced yes)
 		(effects
+			(font
+				(size 1.27 1.27)
+			)
+			(justify left)
+		)
+	)
+	(hierarchical_label "n_reset"
+		(shape output)
+		(at 114.3 52.07 0)
+		(fields_autoplaced yes)
+		(effects

Commit message: stuff
Connections:
- net GPIO13: no longer Module1.28 (GPIO13)
- net GPIO19: no longer Module1.26 (GPIO19)
- net GPIO26: no longer Module1.24 (GPIO26)
- new net Boot1: Module1.24 (GPIO26)
- new net IMU_Rst1: Module1.28 (GPIO13)
- new net Int1: Module1.26 (GPIO19)
Changed lines of the file:
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@@
 		)
 	)
-	(label "GPIO26"
+	(label "Boot1"
 		(at 32.766 46.99 180)
 		(fields_autoplaced yes)
@@
 		)
 	)
-	(label "GPIO13"
+	(label "IMU_Rst1"
 		(at 32.766 52.07 180)
 		(fields_autoplaced yes)
@@
 		)
 	)
-	(label "GPIO19"
+	(label "Int1"
 		(at 32.766 49.53 180)
 		(fields_autoplaced yes)
@@
 		)
 	)
+	(hierarchical_label "Int1"
+		(shape output)
+		(at 25.4 49.53 180)
+		(fields_autoplaced yes)
+		(effects
+			(font
+				(size 1.27 1.27)
+			)
+			(justify right)
+		)
+	)
 	(hierarchical_label "SCL0"
 		(shape output)
@@
 		(fields_autoplaced yes)
 		(effects
+			(font
+				(size 1.27 1.27)
+			)
+			(justify right)
+		)
+	)
+	(hierarchical_label "Boot1"
+		(shape output)
+		(at 25.4 46.99 180)
+		(fields_autoplaced yes)
+		(effects
+			(font
+				(size 1.27 1.27)
+			)
+			(justify right)
+		)
+	)
+	(hierarchical_label "IMU_Rst1"
+		(shape output)
+		(at 25.4 52.07 180)
+		(fields_autoplaced yes)
+		(effects

Commit message: stuff
Connections:
- net GPIO17: no longer Module1.50 (GPIO17)
- net GPIO27: no longer Module1.48 (GPIO27)
- new net IMU1_PS0: Module1.48 (GPIO27)
- new net IMU_PS0: Module1.50 (GPIO17)
Changed lines of the file:
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@@
-	(wire
-		(pts
-			(xy 25.146 80.01) (xy 39.116 80.01)
-		)
-		(stroke
-			(width 0)
-			(type solid)
-		)
-	)
 	(wire
 		(pts
@@
 	(wire
 		(pts
+			(xy 24.13 77.47) (xy 39.116 77.47)
+		)
+		(stroke
+			(width 0)
+			(type solid)
+		)
+	)
+	(wire
+		(pts
 			(xy 185.42 33.02) (xy 194.31 33.02)
 		)
@@
 	(wire
 		(pts
-			(xy 25.146 77.47) (xy 39.116 77.47)
-		)
-		(stroke
-			(width 0)
-			(type solid)
-		)
-	)
-	(wire
-		(pts
 			(xy 100.076 57.15) (xy 114.046 57.15)
 		)
@@
 		(pts
 			(xy 165.1 59.69) (xy 166.37 59.69)
+		)
+		(stroke
+			(width 0)
+			(type solid)
+		)
+	)
+	(wire
+		(pts
+			(xy 24.13 80.01) (xy 39.116 80.01)
 		)
 		(stroke
@@
 		)
 	)
-	(label "GPIO27"
-		(at 32.766 77.47 180)
-		(fields_autoplaced yes)
-		(effects
-			(font
-				(size 1.27 1.27)
-			)
-			(justify right bottom)
-		)
-	)
 	(label "GLOBAL_EN"
 		(at 90.17 180.34 180)
@@
 	(label "GPIO3"
 		(at 31.496 87.63 180)
-		(fields_autoplaced yes)
-		(effects
-			(font
-				(size 1.27 1.27)
-			)
-			(justify right bottom)
-		)
-	)
-	(label "GPIO17"
-		(at 32.766 80.01 180)
 		(fields_autoplaced yes)
 		(effects
@@
 		)
 	)
+	(hierarchical_label "IMU1_PS0"
+		(shape output)
+		(at 24.13 77.47 180)
+		(fields_autoplaced yes)
+		(effects
+			(font
+				(size 1.27 1.27)
+			)
+			(justify right)
+		)
+	)
 	(hierarchical_label "TX"
 		(shape output)
@@
 		(fields_autoplaced yes)
 		(effects
+			(font
+				(size 1.27 1.27)
+			)
+			(justify right)
+		)
+	)
+	(hierarchical_label "IMU_PS0"
+		(shape output)
+		(at 24.13 80.01 180)
+		(fields_autoplaced yes)
+		(effects

Commit message: stuff
Connections:
- net CAM_GPIO: no longer names the net of Module1.97 (Camera_GPIO)
- net GPIO12: no longer names the net of J8.32 (Pin_32)
- net GPIO13: no longer names the net of J8.33 (Pin_33)
- net GPIO14: no longer names the net of J8.8 (Pin_8)
- net GPIO15: no longer names the net of J8.10 (Pin_10)
- net GPIO16: no longer names the net of J8.36 (Pin_36)
- net GPIO17: no longer names the net of J8.11 (Pin_11)
- net GPIO18: no longer names the net of J8.12 (Pin_12)
- net GPIO19: no longer names the net of J8.35 (Pin_35)
- net GPIO2: no longer names the net of J8.3 (Pin_3)
- net GPIO2: no longer Module1.58 (GPIO2)
- net GPIO20: no longer names the net of J8.38 (Pin_38)
- net GPIO21: no longer names the net of J8.40 (Pin_40)
- net GPIO23: no longer names the net of J8.16 (Pin_16)
- net GPIO24: no longer names the net of J8.18 (Pin_18)
- net GPIO25: no longer names the net of J8.22 (Pin_22)
- net GPIO26: no longer names the net of J8.37 (Pin_37)
- net GPIO27: no longer names the net of J8.13 (Pin_13)
- net GPIO8: no longer names the net of J8.24 (Pin_24)
- new net XRSTJ: Module1.58 (GPIO2)
- no-connect marks 7 -> 24
Changed lines of the file:
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@@
 	)
 	(no_connect
+		(at 140.97 67.31)
+	)
+	(no_connect
+		(at 176.53 67.31)
+	)
+	(no_connect
+		(at 176.53 49.53)
+	)
+	(no_connect
+		(at 140.97 39.37)
+	)
+	(no_connect
 		(at 243.84 156.21)
 	)
 	(no_connect
+		(at 176.53 62.23)
+	)
+	(no_connect
+		(at 176.53 72.39)
+	)
+	(no_connect
+		(at 176.53 41.91)
+	)
+	(no_connect
 		(at 100.076 110.49)
 	)
 	(no_connect
+		(at 140.97 69.85)
+	)
+	(no_connect
+		(at 176.53 31.75)
+	)
+	(no_connect
+		(at 140.97 26.67)
+	)
+	(no_connect
+		(at 140.97 64.77)
+	)
+	(no_connect
 		(at 39.116 97.79)
 	)
 	(no_connect
+		(at 176.53 34.29)
+	)
+	(no_connect
+		(at 176.53 36.83)
+	)
+	(no_connect
+		(at 176.53 52.07)
+	)
+	(no_connect
 		(at 100.076 41.91)
 	)
 	(no_connect
+		(at 176.53 69.85)
+	)
+	(no_connect
+		(at 140.97 36.83)
+	)
+	(no_connect
 		(at 39.116 107.95)
 	)
 	(no_connect
+		(at 176.53 44.45)
+	)
+	(no_connect
 		(at 39.116 105.41)
 	)
@@
 	(wire
 		(pts
-			(xy 25.146 90.17) (xy 39.116 90.17)
-		)
-		(stroke
-			(width 0)
-			(type solid)
-		)
-	)
-	(wire
-		(pts
 			(xy 140.97 64.77) (xy 152.4 64.77)
 		)
@@
 	(wire
 		(pts
-			(xy 100.076 80.01) (xy 114.046 80.01)
+			(xy 24.13 90.17) (xy 39.116 90.17)
+		)
+		(stroke
+			(width 0)
+			(type solid)
+		)
+	)
+	(wire
+		(pts
+			(xy 100.076 80.01) (xy 114.3 80.01)
 		)
 		(stroke
@@
 	(wire
 		(pts
-			(xy 100.076 52.07) (xy 114.046 52.07)
+			(xy 100.076 52.07) (xy 114.3 52.07)
 		)
 		(stroke
@@
 	(wire
 		(pts
-			(xy 100.076 87.63) (xy 114.046 87.63)
+			(xy 100.076 87.63) (xy 114.3 87.63)
 		)
 		(stroke
@@
 	(wire
 		(pts
-			(xy 100.076 67.31) (xy 114.046 67.31)
+			(xy 100.076 67.31) (xy 114.3 67.31)
 		)
 		(stroke
@@
 		)
 	)
-	(wire
-		(pts
-			(xy 100.076 140.97) (xy 116.586 140.97)
-		)
-		(stroke
-			(width 0)
-			(type solid)
-		)
-	)
 	(polyline
 		(pts
@@
 	(wire
 		(pts
-			(xy 100.076 82.55) (xy 114.046 82.55)
+			(xy 100.076 82.55) (xy 114.3 82.55)
 		)
 		(stroke
@@
 	(wire
 		(pts
-			(xy 100.076 69.85) (xy 114.046 69.85)
+			(xy 100.076 69.85) (xy 114.3 69.85)
 		)
 		(stroke
@@
 	(wire
 		(pts
-			(xy 100.076 77.47) (xy 114.046 77.47)
+			(xy 100.076 77.47) (xy 114.3 77.47)
 		)
 		(stroke
@@
 	(wire
 		(pts
-			(xy 100.076 49.53) (xy 114.046 49.53)
+			(xy 100.076 49.53) (xy 114.3 49.53)
 		)
 		(stroke
@@
 	(wire
 		(pts
-			(xy 100.076 74.93) (xy 114.046 74.93)
+			(xy 100.076 74.93) (xy 114.3 74.93)
 		)
 		(stroke
@@
 	(wire
 		(pts
-			(xy 100.076 57.15) (xy 114.046 57.15)
+			(xy 100.076 57.15) (xy 114.3 57.15)
 		)
 		(stroke
@@
 	(wire
 		(pts
-			(xy 100.076 54.61) (xy 114.046 54.61)
+			(xy 100.076 54.61) (xy 114.3 54.61)
 		)
 		(stroke
@@
 		)
 	)
-	(label "GPIO15"
-		(at 175.26 34.29 180)
-		(fields_autoplaced yes)
-		(effects
-			(font
-				(size 1.27 1.27)
-			)
-			(justify right bottom)
-		)
-	)
 	(label "TRD2_N"
 		(at 245.11 46.99 180)
@@
 		)
 	)
-	(label "GPIO12"
-		(at 175.26 62.23 180)
-		(fields_autoplaced yes)
-		(effects
-			(font
-				(size 1.27 1.27)
-			)
-			(justify right bottom)
-		)
-	)
 	(label "SD_DAT0"
 		(at 223.52 130.81 0)
@@
 		)
 	)
-	(label "GPIO18"
-		(at 175.26 36.83 180)
-		(fields_autoplaced yes)
-		(effects
-			(font
-				(size 1.27 1.27)
-			)
-			(justify right bottom)
-		)
-	)
 	(label "nPWR_LED"
 		(at 105.156 138.43 0)
@@
 		)
 	)
-	(label "GPIO14"
-		(at 175.26 31.75 180)
-		(fields_autoplaced yes)
-		(effects
-			(font
-				(size 1.27 1.27)
-			)
-			(justify right bottom)
-		)
-	)
 	(label "GPIO7"
 		(at 173.99 54.61 180)
@@
 		)
 	)
-	(label "GPIO26"
-		(at 148.59 69.85 180)
-		(fields_autoplaced yes)
-		(effects
-			(font
-				(size 1.27 1.27)
-			)
-			(justify right bottom)
-		)
-	)
 	(label "BT_nDis"
 		(at 112.6236 133.35 180)
@@
 		)
 	)
-	(label "GPIO2"
-		(at 147.32 26.67 180)
-		(fields_autoplaced yes)
-		(effects
-			(font
-				(size 1.27 1.27)
-			)
-			(justify right bottom)
-		)
-	)
 	(label "TRD3_N"
 		(at 193.04 33.02 180)
@@
 		)
 	)
-	(label "GPIO13"
-		(at 148.59 64.77 180)
-		(fields_autoplaced yes)
-		(effects
-			(font
-				(size 1.27 1.27)
-			)
-			(justify right bottom)
-		)
-	)
 	(label "GPIO6"
 		(at 31.496 54.61 180)
@@
 		)
 	)
-	(label "GPIO17"
-		(at 148.59 36.83 180)
-		(fields_autoplaced yes)
-		(effects
-			(font
-				(size 1.27 1.27)
-			)
-			(justify right bottom)
-		)
-	)
 	(label "GPIO9"
 		(at 147.32 49.53 180)
@@
 		)
 	)
-	(label "GPIO25"
-		(at 175.26 49.53 180)
-		(fields_autoplaced yes)
-		(effects
-			(font
-				(size 1.27 1.27)
-			)
-			(justify right bottom)
-		)
-	)
-	(label "GPIO21"
-		(at 175.26 72.39 180)
-		(fields_autoplaced yes)
-		(effects
-			(font
-				(size 1.27 1.27)
-			)
-			(justify right bottom)
-		)
-	)
 	(label "AIN1"
 		(at 84.074 170.18 180)
@@
 		)
 	)
-	(label "GPIO19"
-		(at 148.59 67.31 180)
-		(fields_autoplaced yes)
-		(effects
-			(font
-				(size 1.27 1.27)
-			)
-			(justify right bottom)
-		)
-	)
 	(label "TRD0_P"
 		(at 245.11 21.59 180)
@@
 		)
 	)
-	(label "GPIO27"
-		(at 148.59 39.37 180)
-		(fields_autoplaced yes)
-		(effects
-			(font
-				(size 1.27 1.27)
-			)
-			(justify right bottom)
-		)
-	)
 	(label "GPIO11"
 		(at 32.766 64.77 180)
@@
 		)
 	)
-	(label "GPIO20"
-		(at 175.26 69.85 180)
-		(fields_autoplaced yes)
-		(effects
-			(font
-				(size 1.27 1.27)
-			)
-			(justify right bottom)
-		)
-	)
 	(label "GPIO7"
 		(at 108.966 64.77 180)
@@
 		)
 	)
-	(label "GPIO8"
-		(at 173.99 52.07 180)
-		(fields_autoplaced yes)
-		(effects
-			(font
-				(size 1.27 1.27)
-			)
-			(justify right bottom)
-		)
-	)
 	(label "ETH_LEDY"
 		(at 102.87 36.83 0)
@@
 		)
 	)
-	(label "GPIO2"
+	(label "XRSTJ"
 		(at 31.496 90.17 180)
 		(fields_autoplaced yes)
@@
 		)
 	)
-	(label "GPIO23"
-		(at 175.26 41.91 180)
-		(fields_autoplaced yes)
-		(effects
-			(font
-				(size 1.27 1.27)
-			)
-			(justify right bottom)
-		)
-	)
 	(label "SD_CLK"
 		(at 110.236 90.17 180)
@@
 		)
 	)
-	(label "GPIO16"
-		(at 175.26 67.31 180)
-		(fields_autoplaced yes)
-		(effects
-			(font
-				(size 1.27 1.27)
-			)
-			(justify right bottom)
-		)
-	)
 	(label "GPIO10"
 		(at 32.766 72.39 180)
@@
 		)
 	)
-	(label "GPIO24"
-		(at 175.26 44.45 180)
-		(fields_autoplaced yes)
-		(effects
-			(font
-				(size 1.27 1.27)
-			)
-			(justify right bottom)
-		)
-	)
 	(label "ETH_LEDY"
 		(at 227.33 80.01 180)
@@
 		)
 	)
+	(hierarchical_label "XRSTJ"
+		(shape output)
+		(at 24.13 90.17 180)
+		(fields_autoplaced yes)
+		(effects
+			(font
+				(size 1.27 1.27)
+			)
+			(justify right)
+		)
+	)
 	(hierarchical_label "TX"
 		(shape output)
@@
 		(fields_autoplaced yes)
 		(effects
-			(font
-				(size 1.27 1.27)
-			)
-			(justify left)
-		)
-	)
-	(hierarchical_label "CAM_GPIO"
-		(shape output)
-		(at 116.586 140.97 0)
-		(fields_autoplaced yes)
-		(effects

Commit message: stuff
Connections:
- net GPIO22: no longer names the net of J8.15 (Pin_15)
- net GPIO22: no longer Module1.46 (GPIO22)
- new net TB_EN: Module1.46 (GPIO22)
- no-connect marks 24 -> 26
Changed lines of the file:
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@@
 	)
 	(no_connect
+		(at 100.33 140.97)
+	)
+	(no_connect
 		(at 176.53 67.31)
 	)
@@
 	)
 	(no_connect
+		(at 140.97 41.91)
+	)
+	(no_connect
 		(at 140.97 64.77)
 	)
@@
 	(wire
 		(pts
+			(xy 24.13 74.93) (xy 39.116 74.93)
+		)
+		(stroke
+			(width 0)
+			(type solid)
+		)
+	)
+	(wire
+		(pts
 			(xy 151.13 34.29) (xy 151.13 54.61)
 		)
@@
 	(wire
 		(pts
-			(xy 25.146 74.93) (xy 39.116 74.93)
-		)
-		(stroke
-			(width 0)
-			(type solid)
-		)
-	)
-	(wire
-		(pts
 			(xy 114.046 102.87) (xy 100.076 102.87)
 		)
@@
 		)
 	)
-	(label "GPIO22"
+	(label "TB_EN"
 		(at 32.766 74.93 180)
 		(fields_autoplaced yes)
@@
 		)
 	)
-	(label "GPIO22"
-		(at 148.59 41.91 180)
-		(fields_autoplaced yes)
-		(effects
-			(font
-				(size 1.27 1.27)
-			)
-			(justify right bottom)
-		)
-	)
 	(label "ETH_LEDG"
 		(at 102.87 39.37 0)
@@
 		)
 	)
+	(hierarchical_label "TB_EN"
+		(shape output)
+		(at 24.13 74.93 180)
+		(fields_autoplaced yes)
+		(effects
+			(font
+				(size 1.27 1.27)
+			)
+			(justify right)
+		)
+	)
