File: CM4_GPIO.kicad_sch (KiCad schematic)
At the start: 28 parts, among them J1 Conn_01x03, J2 Conn_02x07_Odd_Even, J3 Conn_01x03, J7 Micro_SD_Card_Det, J8 THD-20-R, J9 THD-02-R, U1 TPD4EUSB30, U18 RT9742GGJ5, U2 TPD4EUSB30, U3 MagJack-A70-112-331N126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

Commit message: stuff
Connections:
- net GPIO9: no longer names the net of J8.21 (Pin_21)
- net GPIO9: no longer Module1.40 (GPIO9)
- new net NRST2: Module1.40 (GPIO9)
- no-connect marks 26 -> 27
Changed lines of the file:
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@@
 	)
 	(no_connect
-		(at 100.33 140.97)
+		(at 113.03 140.97)
 	)
 	(no_connect
@@
 	)
 	(no_connect
+		(at 140.97 49.53)
+	)
+	(no_connect
 		(at 176.53 31.75)
 	)
@@
 	(wire
 		(pts
+			(xy 100.076 140.97) (xy 113.03 140.97)
+		)
+		(stroke
+			(width 0)
+			(type default)
+		)
+	)
+	(wire
+		(pts
 			(xy 166.37 39.37) (xy 165.1 39.37)
 		)
@@
 	(wire
 		(pts
-			(xy 25.146 67.31) (xy 39.116 67.31)
+			(xy 39.116 125.73) (xy 39.116 123.19)
 		)
 		(stroke
@@
 	(wire
 		(pts
-			(xy 39.116 125.73) (xy 39.116 123.19)
+			(xy 78.994 177.8) (xy 96.774 177.8)
 		)
 		(stroke
@@
 	(wire
 		(pts
-			(xy 78.994 177.8) (xy 96.774 177.8)
+			(xy 237.49 41.91) (xy 246.38 41.91)
 		)
 		(stroke
@@
 	(wire
 		(pts
-			(xy 237.49 41.91) (xy 246.38 41.91)
+			(xy 183.388 143.002) (xy 183.388 137.922)
 		)
 		(stroke
@@
 	(wire
 		(pts
-			(xy 183.388 143.002) (xy 183.388 137.922)
+			(xy 24.13 67.31) (xy 39.116 67.31)
 		)
 		(stroke
@@
 		)
 	)
-	(label "GPIO9"
-		(at 147.32 49.53 180)
-		(fields_autoplaced yes)
-		(effects
-			(font
-				(size 1.27 1.27)
-			)
-			(justify right bottom)
-		)
-	)
 	(label "TRD0_P"
 		(at 227.33 64.77 180)
@@
 		)
 	)
-	(label "GPIO9"
+	(label "NRST2"
 		(at 31.496 67.31 180)
 		(fields_autoplaced yes)
@@
 		)
 	)
+	(hierarchical_label "NRST2"
+		(shape output)
+		(at 24.13 67.31 180)
+		(fields_autoplaced yes)
+		(effects
+			(font
+				(size 1.27 1.27)
+			)
+			(justify right)
+		)
+	)

Commit message: stuff
Connections:
- net +3.3v: no longer D1.2 (A), D2.2 (A), J8.1 (Pin_1), J8.17 (Pin_17), Module1.84 (+3.3v_(Output)), Module1.86 (+3.3v_(Output)), R17.1, R5.1, U3.15 (LEDG_A), U3.17 (LEDY_A), U5.5 (VCC)
- net +5v: no longer Module1.77 (+5v_(Input)), Module1.79 (+5v_(Input)), Module1.81 (+5v_(Input)), Module1.83 (+5v_(Input)), Module1.85 (+5v_(Input)), Module1.87 (+5v_(Input))
- net +1.8v renamed 1.8v
- new net +3.3V: D1.2 (A), D2.2 (A), J8.1 (Pin_1), J8.17 (Pin_17), Module1.84 (+3.3v_(Output)), Module1.86 (+3.3v_(Output)), R17.1, R5.1, U3.15 (LEDG_A), U3.17 (LEDY_A), U5.5 (VCC)
- new net +5V: Module1.77 (+5v_(Input)), Module1.79 (+5v_(Input)), Module1.81 (+5v_(Input)), Module1.83 (+5v_(Input)), Module1.85 (+5v_(Input)), Module1.87 (+5v_(Input))
Other:
- moved on the sheet: D1, U5

Commit message: minor erc fixes
Connections:
- net +3.3v is gone; now on net +3.3V: R29.1, U18.5 (IN)
Changed lines of the file:
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@@
 		)
 	)
-	(label "+3.3v"
+	(label "+3.3V"
 		(at 273.685 148.59 180)
 		(fields_autoplaced yes)
@@
 		(on_board yes)
 		(dnp no)
-		(fields_autoplaced yes)
 		(property "Reference" "#PWR0135"
 			(at 15.24 127 0)

Commit message: stuff
Connections:
- net +5V: now also U9.5 (VCC)
- net +5v: no longer U9.5 (VCC)
- net nEXTRST: no longer names the net of Module1.100 (nEXTRST)
- no-connect marks 27 -> 28
Changed lines of the file:
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@@
 	)
 	(no_connect
+		(at 25.4 143.51)
+	)
+	(no_connect
 		(at 100.076 41.91)
 	)
@@
 	(wire
 		(pts
-			(xy 25.146 143.51) (xy 39.116 143.51)
+			(xy 25.4 143.51) (xy 39.116 143.51)
 		)
 		(stroke
@@
 		)
 	)
-	(label "+5v"
-		(at 16.51 172.72 0)
-		(fields_autoplaced yes)
-		(effects
-			(font
-				(size 2.0066 2.0066)
-			)
-			(justify left bottom)
-		)
-	)
 	(label "SD_DAT0"
 		(at 111.506 97.79 180)
@@
 		)
 	)
-	(hierarchical_label "nEXTRST"
-		(shape output)
-		(at 25.146 143.51 180)
-		(fields_autoplaced yes)
-		(effects
-			(font
-				(size 1.27 1.27)
-			)
-			(justify right)
-		)
-	)
 	(hierarchical_label "Boot1"
 		(shape output)
@@
 					(unit 1)
 				)
+			)
+		)
+	)
+	(symbol
+		(lib_id "power:+5V")
+		(at 13.97 172.72 0)
+		(unit 1)
+		(exclude_from_sim no)
+		(in_bom yes)
+		(on_board yes)
+		(dnp no)
+		(fields_autoplaced yes)
+		(property "Reference" "#PWR0150"
+			(at 13.97 176.53 0)
+			(effects
+				(font
+					(size 1.27 1.27)
+				)
+				(hide yes)
+			)
+		)
+		(property "Value" "+5V"
+			(at 13.97 167.64 0)
+			(effects
+				(font
+					(size 1.27 1.27)
+				)
+			)
+		)
+		(property "Footprint" ""
+			(at 13.97 172.72 0)
+			(effects
+				(font
+					(size 1.27 1.27)
+				)
+				(hide yes)
+			)
+		)
+		(property "Datasheet" ""
+			(at 13.97 172.72 0)
+			(effects
+				(font
+					(size 1.27 1.27)
+				)
+				(hide yes)
+			)
+		)
+		(property "Description" "Power symbol creates a global label with name \"+5V\""
+			(at 13.97 172.72 0)
+			(effects
+				(font
+					(size 1.27 1.27)
+				)
+				(hide yes)
+			)
+		)
+		(pin "1"
+		)
+		(instances
+			(project ""
+				(path "/e63e39d7-6ac0-4ffd-8aa3-1841a4541b55/00000000-0000-0000-0000-00005cff706a"
+					(reference "#PWR0150")
+					(unit 1)
+				)

Commit message: stuff
Changed lines of the file:
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@@
+	)
+	(symbol
+		(lib_id "power:PWR_FLAG")
+		(at 146.05 175.26 0)
+		(unit 1)
+		(exclude_from_sim no)
+		(in_bom yes)
+		(on_board yes)
+		(dnp no)
+		(fields_autoplaced yes)
+		(property "Reference" "#FLG04"
+			(at 146.05 173.355 0)
+			(effects
+				(font
+					(size 1.27 1.27)
+				)
+				(hide yes)
+			)
+		)
+		(property "Value" "PWR_FLAG"
+			(at 146.05 170.18 0)
+			(effects
+				(font
+					(size 1.27 1.27)
+				)
+			)
+		)
+		(property "Footprint" ""
+			(at 146.05 175.26 0)
+			(effects
+				(font
+					(size 1.27 1.27)
+				)
+				(hide yes)
+			)
+		)
+		(property "Datasheet" "~"
+			(at 146.05 175.26 0)
+			(effects
+				(font
+					(size 1.27 1.27)
+				)
+				(hide yes)
+			)
+		)
+		(property "Description" "Special symbol for telling ERC where power comes from"
+			(at 146.05 175.26 0)
+			(effects
+				(font
+					(size 1.27 1.27)
+				)
+				(hide yes)
+			)
+		)
+		(pin "1"
+		)
+		(instances
+			(project ""
+				(path "/e63e39d7-6ac0-4ffd-8aa3-1841a4541b55/00000000-0000-0000-0000-00005cff706a"
+					(reference "#FLG04")
+					(unit 1)
+				)
+			)
+		)
 	)
 	(symbol
@@
 					(unit 1)
 				)
+			)
+		)
+	)
+	(symbol
+		(lib_name "GND_1")
+		(lib_id "power:GND")
+		(at 146.05 175.26 0)
+		(unit 1)
+		(exclude_from_sim no)
+		(in_bom yes)
+		(on_board yes)
+		(dnp no)
+		(fields_autoplaced yes)
+		(property "Reference" "#PWR0154"
+			(at 146.05 181.61 0)
+			(effects
+				(font
+					(size 1.27 1.27)
+				)
+				(hide yes)
+			)
+		)
+		(property "Value" "GND"
+			(at 146.05 180.34 0)
+			(effects
+				(font
+					(size 1.27 1.27)
+				)
+			)
+		)
+		(property "Footprint" ""
+			(at 146.05 175.26 0)
+			(effects
+				(font
+					(size 1.27 1.27)
+				)
+				(hide yes)
+			)
+		)
+		(property "Datasheet" ""
+			(at 146.05 175.26 0)
+			(effects
+				(font
+					(size 1.27 1.27)
+				)
+				(hide yes)
+			)
+		)
+		(property "Description" "Power symbol creates a global label with name \"GND\" , ground"
+			(at 146.05 175.26 0)
+			(effects
+				(font
+					(size 1.27 1.27)
+				)
+				(hide yes)
+			)
+		)
+		(pin "1"
+		)
+		(instances
+			(project ""
+				(path "/e63e39d7-6ac0-4ffd-8aa3-1841a4541b55/00000000-0000-0000-0000-00005cff706a"
+					(reference "#PWR0154")
+					(unit 1)
+				)

Commit message: assigned footprints
Parts:
- C1: footprint Capacitor_SMD:C_0402_1005Metric -> Capacitor_SMD:C_0805_2012Metric
- D1, D2: footprint LED_SMD:LED_0603_1608Metric -> LED_SMD:LED_0805_2012Metric
- R1, R10, R17, R18, R2, R29, R3: footprint Resistor_SMD:R_0402_1005Metric -> Resistor_SMD:R_0805_2012Metric
- R4, R5: footprint Resistor_SMD:R_0805_2012Metric_Pad1.15x1.40mm_HandSolder -> Resistor_SMD:R_0805_2012Metric
Changed lines of the file:
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@@
 			)
 		)
-		(property "Footprint" "Capacitor_SMD:C_0402_1005Metric"
+		(property "Footprint" "Capacitor_SMD:C_0805_2012Metric"
 			(at 229.5652 45.72 0)
 			(effects
@@
 			)
 		)
-		(property "Footprint" "Resistor_SMD:R_0402_1005Metric"
+		(property "Footprint" "Resistor_SMD:R_0805_2012Metric"
 			(at 232.41 73.152 90)
 			(effects
@@
 			)
 		)
-		(property "Footprint" "Resistor_SMD:R_0402_1005Metric"
+		(property "Footprint" "Resistor_SMD:R_0805_2012Metric"
 			(at 232.41 78.232 90)
 			(effects
@@
 			)
 		)
-		(property "Footprint" "LED_SMD:LED_0603_1608Metric"
+		(property "Footprint" "LED_SMD:LED_0805_2012Metric"
 			(at 116.84 25.4 0)
 			(effects
@@
 			)
 		)
-		(property "Footprint" "Resistor_SMD:R_0402_1005Metric"
+		(property "Footprint" "Resistor_SMD:R_0805_2012Metric"
 			(at 115.062 38.1 90)
 			(effects
@@
 			)
 		)
-		(property "Footprint" "LED_SMD:LED_0603_1608Metric"
+		(property "Footprint" "LED_SMD:LED_0805_2012Metric"
 			(at 191.77 125.73 0)
 			(effects
@@
 			)
 		)
-		(property "Footprint" "Resistor_SMD:R_0402_1005Metric"
+		(property "Footprint" "Resistor_SMD:R_0805_2012Metric"
 			(at 189.23 135.382 90)
 			(effects
@@
 			)
 		)
-		(property "Footprint" "Resistor_SMD:R_0805_2012Metric_Pad1.15x1.40mm_HandSolder"
+		(property "Footprint" "Resistor_SMD:R_0805_2012Metric"
 			(at 156.21 93.218 90)
 			(effects
@@
 			)
 		)
-		(property "Footprint" "Resistor_SMD:R_0805_2012Metric_Pad1.15x1.40mm_HandSolder"
+		(property "Footprint" "Resistor_SMD:R_0805_2012Metric"
 			(at 156.21 97.028 90)
 			(effects
@@
 			)
 		)
-		(property "Footprint" "Resistor_SMD:R_0402_1005Metric"
+		(property "Footprint" "Resistor_SMD:R_0805_2012Metric"
 			(at 228.6 137.668 90)
 			(effects
@@
 			)
 		)
-		(property "Footprint" "Resistor_SMD:R_0402_1005Metric"
+		(property "Footprint" "Resistor_SMD:R_0805_2012Metric"
 			(at 271.907 152.4 90)
 			(effects
@@
 			)
 		)
-		(property "Footprint" "Resistor_SMD:R_0402_1005Metric"
+		(property "Footprint" "Resistor_SMD:R_0805_2012Metric"
 			(at 228.6 145.288 90)
 			(effects
