File: CM4_GPIO.kicad_sch (KiCad schematic)
At the start: 28 parts, among them J1 Conn_01x03, J2 Conn_02x07_Odd_Even, J3 Conn_01x03, J7 Micro_SD_Card_Det, J8 THD-20-R, J9 THD-02-R, U1 TPD4EUSB30, U18 RT9742GGJ5, U2 TPD4EUSB30, U3 MagJack-A70-112-331N126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

Commit message: stuff
Connections:
- net GPIO10: no longer Module1.44 (GPIO10)
- net GPIO4: no longer Module1.54 (GPIO4)
- net GPIO5: no longer Module1.34 (GPIO5)
- new net ISO_FLT: Module1.44 (GPIO10)
- new net RX_TB: Module1.34 (GPIO5)
- new net TX_TB: Module1.54 (GPIO4)
Changed lines of the file:
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@@
 	(wire
 		(pts
+			(xy 24.13 46.99) (xy 39.116 46.99)
+		)
+		(stroke
+			(width 0)
+			(type solid)
+		)
+	)
+	(wire
+		(pts
+			(xy 24.13 52.07) (xy 39.116 52.07)
+		)
+		(stroke
+			(width 0)
+			(type solid)
+		)
+	)
+	(wire
+		(pts
 			(xy 100.076 21.59) (xy 113.03 21.59)
 		)
@@
 	(wire
 		(pts
-			(xy 25.146 59.69) (xy 39.116 59.69)
-		)
-		(stroke
-			(width 0)
-			(type solid)
-		)
-	)
-	(wire
-		(pts
 			(xy 100.076 140.97) (xy 113.03 140.97)
 		)
@@
 	(wire
 		(pts
+			(xy 22.86 59.69) (xy 39.116 59.69)
+		)
+		(stroke
+			(width 0)
+			(type solid)
+		)
+	)
+	(wire
+		(pts
 			(xy 100.076 107.95) (xy 101.346 107.95)
 		)
@@
 	(wire
 		(pts
+			(xy 24.13 87.63) (xy 39.116 87.63)
+		)
+		(stroke
+			(width 0)
+			(type solid)
+		)
+	)
+	(wire
+		(pts
 			(xy 100.076 26.67) (xy 101.346 26.67)
 		)
@@
 	(wire
 		(pts
-			(xy 25.146 46.99) (xy 39.116 46.99)
-		)
-		(stroke
-			(width 0)
-			(type solid)
-		)
-	)
-	(wire
-		(pts
 			(xy 25.146 120.65) (xy 39.116 120.65)
 		)
@@
 	(wire
 		(pts
+			(xy 24.13 49.53) (xy 39.116 49.53)
+		)
+		(stroke
+			(width 0)
+			(type solid)
+		)
+	)
+	(wire
+		(pts
 			(xy 114.046 90.17) (xy 100.076 90.17)
 		)
@@
 	(wire
 		(pts
-			(xy 25.146 52.07) (xy 39.116 52.07)
+			(xy 24.13 85.09) (xy 39.116 85.09)
 		)
 		(stroke
@@
 	(wire
 		(pts
-			(xy 25.146 85.09) (xy 39.116 85.09)
-		)
-		(stroke
-			(width 0)
-			(type solid)
-		)
-	)
-	(wire
-		(pts
-			(xy 25.146 49.53) (xy 39.116 49.53)
-		)
-		(stroke
-			(width 0)
-			(type solid)
-		)
-	)
-	(wire
-		(pts
 			(xy 243.84 153.67) (xy 234.95 153.67)
 		)
@@
 	(wire
 		(pts
+			(xy 21.59 72.39) (xy 39.116 72.39)
+		)
+		(stroke
+			(width 0)
+			(type solid)
+		)
+	)
+	(wire
+		(pts
 			(xy 24.13 77.47) (xy 39.116 77.47)
 		)
@@
 	(wire
 		(pts
-			(xy 25.146 87.63) (xy 39.116 87.63)
-		)
-		(stroke
-			(width 0)
-			(type solid)
-		)
-	)
-	(wire
-		(pts
 			(xy 114.046 95.25) (xy 100.076 95.25)
 		)
@@
 	(wire
 		(pts
-			(xy 25.146 72.39) (xy 39.116 72.39)
-		)
-		(stroke
-			(width 0)
-			(type solid)
-		)
-	)
-	(wire
-		(pts
 			(xy 210.82 128.27) (xy 232.41 128.27)
 		)
@@
 	)
 	(label "TRD1_P"
-		(at 30.226 21.59 180)
+		(at 30.48 21.59 180)
 		(fields_autoplaced yes)
 		(effects
@@
 		)
 	)
+	(label "TX_TB"
+		(at 24.13 85.09 0)
+		(fields_autoplaced yes)
+		(effects
+			(font
+				(size 1.27 1.27)
+			)
+			(justify left bottom)
+		)
+	)
 	(label "TRD0_P"
 		(at 245.11 21.59 180)
@@
 		)
 	)
-	(label "GPIO4"
-		(at 31.496 85.09 180)
-		(fields_autoplaced yes)
-		(effects
-			(font
-				(size 1.27 1.27)
-			)
-			(justify right bottom)
-		)
-	)
 	(label "TR2_TAP"
 		(at 221.9198 90.17 180)
@@
 		)
 	)
-	(label "GPIO5"
-		(at 31.496 59.69 180)
-		(fields_autoplaced yes)
-		(effects
-			(font
-				(size 1.27 1.27)
-			)
-			(justify right bottom)
-		)
-	)
 	(label "GPIO10"
 		(at 148.59 46.99 180)
@@
 		)
 	)
+	(label "RX_TB"
+		(at 24.13 59.69 0)
+		(fields_autoplaced yes)
+		(effects
+			(font
+				(size 1.27 1.27)
+			)
+			(justify left bottom)
+		)
+	)
 	(label "TRD3_P"
 		(at 245.11 49.53 180)
@@
 		)
 	)
+	(label "ISO_FLT"
+		(at 21.59 72.39 0)
+		(fields_autoplaced yes)
+		(effects
+			(font
+				(size 1.27 1.27)
+			)
+			(justify left bottom)
+		)
+	)
 	(label "ETH_LEDY"
 		(at 102.87 36.83 0)
@@
 	)
 	(label "GPIO3"
-		(at 31.496 87.63 180)
+		(at 24.13 87.63 180)
 		(fields_autoplaced yes)
 		(effects
@@
 	)
 	(label "XRSTJ"
-		(at 31.496 90.17 180)
+		(at 30.48 90.17 180)
 		(fields_autoplaced yes)
 		(effects
@@
 		)
 	)
-	(label "GPIO10"
-		(at 32.766 72.39 180)
-		(fields_autoplaced yes)
-		(effects
-			(font
-				(size 1.27 1.27)
-			)
-			(justify right bottom)
-		)
-	)
 	(label "OE_PWM"
 		(at 110.236 49.53 180)
@@
 		)
 	)
+	(hierarchical_label "TX_TB"
+		(shape output)
+		(at 24.13 85.09 180)
+		(fields_autoplaced yes)
+		(effects
+			(font
+				(size 1.27 1.27)
+			)
+			(justify right)
+		)
+	)
 	(hierarchical_label "TV_OUT"
 		(shape input)
@@
 	(hierarchical_label "Int1"
 		(shape output)
-		(at 25.4 49.53 180)
+		(at 24.13 49.53 180)
+		(fields_autoplaced yes)
+		(effects
+			(font
+				(size 1.27 1.27)
+			)
+			(justify right)
+		)
+	)
+	(hierarchical_label "RX_TB"
+		(shape output)
+		(at 22.86 59.69 180)
 		(fields_autoplaced yes)
 		(effects
@@
 	(hierarchical_label "Boot1"
 		(shape output)
-		(at 25.4 46.99 180)
+		(at 24.13 46.99 180)
 		(fields_autoplaced yes)
 		(effects
@@
 	(hierarchical_label "IMU_Rst1"
 		(shape output)
-		(at 25.4 52.07 180)
+		(at 24.13 52.07 180)
 		(fields_autoplaced yes)
 		(effects
@@
 		)
 	)
+	(hierarchical_label "ISO_FLT"
+		(shape output)
+		(at 21.59 72.39 180)
+		(fields_autoplaced yes)
+		(effects
+			(font
+				(size 1.27 1.27)
+			)
+			(justify right)
+		)
+	)

Commit message: stuff
Connections:
- net GPIO7: no longer Module1.37 (GPIO7)
- new net Fan: Module1.37 (GPIO7)
Changed lines of the file:
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@@
 	(wire
 		(pts
-			(xy 100.076 64.77) (xy 114.046 64.77)
+			(xy 100.076 64.77) (xy 114.3 64.77)
 		)
 		(stroke
@@
 		)
 	)
-	(label "GPIO7"
-		(at 108.966 64.77 180)
-		(fields_autoplaced yes)
-		(effects
-			(font
-				(size 1.27 1.27)
-			)
-			(justify right bottom)
-		)
-	)
 	(label "SD_DAT1"
 		(at 111.506 102.87 180)
@@
 		(fields_autoplaced yes)
 		(effects
+			(font
+				(size 1.27 1.27)
+			)
+			(justify left)
+		)
+	)
+	(hierarchical_label "Fan"
+		(shape output)
+		(at 114.3 64.77 0)
+		(fields_autoplaced yes)
+		(effects

Commit message: stuff
Parts:
- removed J8: THD-20-R, Connector_PinHeader_2.54mm:PinHeader_2x20_P2.54mm_Vertical, symbol Connector_Generic:Conn_02x20_Odd_Even
- added J34, J35, J36, J37, J38, J39, J40, J41, J42: Conn_01x01, Connector_PinHeader_2.54mm:PinHeader_1x01_P2.54mm_Vertical, symbol Connector_Generic:Conn_01x01
Connections:
- net GPIO10: now also J36.1 (Pin_1)
- net GPIO11: now also J37.1 (Pin_1)
- net GPIO3: now also J34.1 (Pin_1)
- net GPIO4: now also J35.1 (Pin_1)
- net GPIO5: now also J39.1 (Pin_1)
- net GPIO6: now also J40.1 (Pin_1)
- net GPIO7: now also J41.1 (Pin_1)
- net ID_SC: now also J42.1 (Pin_1)
- net ID_SD: now also J38.1 (Pin_1)
- no-connect marks 28 -> 9

Commit message: stuff
Parts:
- removed J41: Conn_01x01, Connector_PinHeader_2.54mm:PinHeader_1x01_P2.54mm_Vertical, symbol Connector_Generic:Conn_01x01
Changed lines of the file:
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@@
 	(wire
 		(pts
-			(xy 146.05 45.72) (xy 152.4 45.72)
-		)
-		(stroke
-			(width 0)
-			(type default)
-		)
-	)
-	(wire
-		(pts
 			(xy 27.94 172.72) (xy 27.94 177.8)
 		)
@@
 		)
 	)
-	(label "GPIO7"
-		(at 146.05 45.72 0)
-		(fields_autoplaced yes)
-		(effects
-			(font
-				(size 1.27 1.27)
-			)
-			(justify left bottom)
-		)
-	)
 	(label "ETH_LEDG"
 		(at 102.87 39.37 0)
@@
 					(unit 1)
 				)
-			)
-		)
-	)
-	(symbol
-		(lib_id "Connector_Generic:Conn_01x01")
-		(at 157.48 45.72 0)
-		(unit 1)
-		(exclude_from_sim no)
-		(in_bom yes)
-		(on_board yes)
-		(dnp no)
-		(fields_autoplaced yes)
-		(property "Reference" "J41"
-			(at 160.02 44.4499 0)
-			(effects
-				(font
-					(size 1.27 1.27)
-				)
-				(justify left)
-			)
-		)
-		(property "Value" "Conn_01x01"
-			(at 160.02 46.9899 0)
-			(effects
-				(font
-					(size 1.27 1.27)
-				)
-				(justify left)
-			)
-		)
-		(property "Footprint" "Connector_PinHeader_2.54mm:PinHeader_1x01_P2.54mm_Vertical"
-			(at 157.48 45.72 0)
-			(effects
-				(font
-					(size 1.27 1.27)
-				)
-				(hide yes)
-			)
-		)
-		(property "Datasheet" "~"
-			(at 157.48 45.72 0)
-			(effects
-				(font
-					(size 1.27 1.27)
-				)
-				(hide yes)
-			)
-		)
-		(property "Description" "Generic connector, single row, 01x01, script generated (kicad-library-utils/schlib/autogen/connector/)"
-			(at 157.48 45.72 0)
-			(effects
-				(font
-					(size 1.27 1.27)
-				)
-				(hide yes)
-			)
-		)
-		(pin "1"
-		)
-		(instances
-			(project "CM4IOv5"
-				(path "/e63e39d7-6ac0-4ffd-8aa3-1841a4541b55/00000000-0000-0000-0000-00005cff706a"
-					(reference "J41")
-					(unit 1)
-				)

Commit message: stuff
Parts:
- TP3, TP5: footprint TestPoint:TestPoint_Pad_2.0x2.0mm -> TestPoint:TestPoint_Plated_Hole_D3.0mm
Changed lines of the file:
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@@
 			)
 		)
-		(property "Footprint" "TestPoint:TestPoint_Pad_2.0x2.0mm"
+		(property "Footprint" "TestPoint:TestPoint_Plated_Hole_D3.0mm"
 			(at 186.0042 125.349 0)
 			(effects
@@
 			)
 		)
-		(property "Footprint" "TestPoint:TestPoint_Pad_2.0x2.0mm"
+		(property "Footprint" "TestPoint:TestPoint_Plated_Hole_D3.0mm"
 			(at 123.19 36.83 0)
 			(effects
