File: PWM_Generatrion.kicad_sch (KiCad schematic)
At the start: 1 part, among them U22 PCA9685PW_118

Commit message: stuff
Parts:
- added J25: IPT1-105-01-L-D, IPT1-105-01-L-D:SAMTEC_IPT1-105-01-L-D, symbol IPT1-105-01-L-D:IPT1-105-01-L-D
Changed lines of the file:
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@@
+	)
+	(symbol
+		(lib_id "IPT1-105-01-L-D:IPT1-105-01-L-D")
+		(at 217.17 71.12 0)
+		(unit 1)
+		(exclude_from_sim no)
+		(in_bom yes)
+		(on_board yes)
+		(dnp no)
+		(fields_autoplaced yes)
+		(property "Reference" "J25"
+			(at 217.17 58.42 0)
+			(effects
+				(font
+					(size 1.27 1.27)
+				)
+			)
+		)
+		(property "Value" "IPT1-105-01-L-D"
+			(at 217.17 60.96 0)
+			(effects
+				(font
+					(size 1.27 1.27)
+				)
+			)
+		)
+		(property "Footprint" "IPT1-105-01-L-D:SAMTEC_IPT1-105-01-L-D"
+			(at 217.17 71.12 0)
+			(effects
+				(font
+					(size 1.27 1.27)
+				)
+				(justify bottom)
+				(hide yes)
+			)
+		)
+		(property "Datasheet" ""
+			(at 217.17 71.12 0)
+			(effects
+				(font
+					(size 1.27 1.27)
+				)
+				(hide yes)
+			)
+		)
+		(property "Description" ""
+			(at 217.17 71.12 0)
+			(effects
+				(font
+					(size 1.27 1.27)
+				)
+				(hide yes)
+			)
+		)
+		(property "PARTREV" "R"
+			(at 217.17 71.12 0)
+			(effects
+				(font
+					(size 1.27 1.27)
+				)
+				(justify bottom)
+				(hide yes)
+			)
+		)
+		(property "STANDARD" "Manufacturer Recommendations"
+			(at 217.17 71.12 0)
+			(effects
+				(font
+					(size 1.27 1.27)
+				)
+				(justify bottom)
+				(hide yes)
+			)
+		)
+		(property "MANUFACTURER" "Samtec"
+			(at 217.17 71.12 0)
+			(effects
+				(font
+					(size 1.27 1.27)
+				)
+				(justify bottom)
+				(hide yes)
+			)
+		)
+		(pin "10"
+		)
+		(pin "07"
+		)
+		(pin "01"
+		)
+		(pin "09"
+		)
+		(pin "04"
+		)
+		(pin "02"
+		)
+		(pin "06"
+		)
+		(pin "08"
+		)
+		(pin "03"
+		)
+		(pin "05"
+		)
+		(instances
+			(project ""
+				(path "/e63e39d7-6ac0-4ffd-8aa3-1841a4541b55/dbf465c7-7de0-4b8a-860d-b014ecfe2e4f"
+					(reference "J25")
+					(unit 1)
+				)
+			)
+		)
 	)
 	(symbol

Commit message: stuff
Changed lines of the file:
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@@
+		)
+	)
+	(label "PWM Generator"
+		(at 132.08 111.76 0)
+		(fields_autoplaced yes)
+		(effects
+			(font
+				(size 1.27 1.27)
+			)
+			(justify left bottom)
 		)
 	)
@@
 		(fields_autoplaced yes)
 		(effects
+			(font
+				(size 1.27 1.27)
+			)
+			(justify left bottom)
+		)
+	)
+	(label "Backplane connector"
+		(at 208.28 82.55 0)
+		(fields_autoplaced yes)
+		(effects

Commit message: stuff
Other:
- note added: "Backplane connector"
- note added: "PWM Generator"
- moved on the sheet: J25, U22

Commit message: stuff
Parts:
- removed J25: IPT1-105-01-L-D, IPT1-105-01-L-D:SAMTEC_IPT1-105-01-L-D, symbol IPT1-105-01-L-D:IPT1-105-01-L-D
- added J13, J14: DF11-10DP-2DSA24, CON10_2X5_UF_DF11_HIR, symbol DF11_10DP_2DSA:DF11-10DP-2DSA24
Connections:
- net 4: now reaches U22.10 (LED4)
- net 4: now also J13.9
- net 5: now reaches U22.11 (LED5)
- net 5: now also J13.10
- net 6: now reaches U22.12 (LED6)
- net 6: now also J14.1
- net 7: now reaches U22.13 (LED7)
- net 7: now also J14.2
- net 8: now reaches U22.15 (LED8)
- net 8: now also J14.3
- net 9: now reaches U22.16 (LED9)
- net 9: now also J14.4
- net 0: now reaches U22.6 (LED0)
- net 0: now also J13.5
- net 1: now reaches U22.7 (LED1)
- net 1: now also J13.6
- net 2: now reaches U22.8 (LED2)
- net 2: now also J13.7
- net 3: now reaches U22.9 (LED3)
- net 3: now also J13.8
- new net 5v: J13.1
- new net A: J13.3
- new net B: J13.4
- new net CS: J14.10
- new net ConRst: J14.6
- new net NISO: J14.7
- new net NOSI: J14.8
- new net SCLK: J14.9
- new net Telemetry: J14.5
- no-connect marks 0 -> 7
Other:
- note added: "Esc Controller Connector"
- note removed: "Backplane connector"

Commit message: stuff
Parts:
- removed J13, J14: DF11-10DP-2DSA24, CON10_2X5_UF_DF11_HIR, symbol DF11_10DP_2DSA:DF11-10DP-2DSA24
- added J13: 302-S101, digikey-footprints:PinHeader_2x5_P2.54mm_Drill1.2mm, symbol dk_Rectangular-Connectors-Headers-Male-Pins:302-S101
Connections:
- net 1: now also J13.1
- net 2: now also J13.3
- net 3: now also J13.5
- net 4: now also J13.7
- net 5: now also J13.9
- net 6: now also J13.2
- net 7: now also J13.4
- net 8: now also J13.6
- net 9: now also J13.8
- no-connect marks 7 -> 8
Other:
- note added: "Backplane Connector"
- note removed: "Esc Controller Connector"

Commit message: stuff
Connections:
- net 0: now also J13.10
- no-connect marks 8 -> 7
Changed lines of the file:
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@@
-	)
-	(no_connect
-		(at 151.13 64.77)
 	)
 	(no_connect
@@
 		(fields_autoplaced yes)
 		(effects
+			(font
+				(size 1.27 1.27)
+			)
+			(justify left bottom)
+		)
+	)
+	(label "0"
+		(at 151.13 64.77 0)
+		(fields_autoplaced yes)
+		(effects

Commit message: stuff
Connections:
- net 3.3v renamed +3.3V
Changed lines of the file:
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@@
-		)
-	)
-	(label "3.3v"
-		(at 36.83 46.99 0)
-		(fields_autoplaced yes)
-		(effects
-			(font
-				(size 1.27 1.27)
-			)
-			(justify left bottom)
-		)
-	)
-	(label "SCL"
-		(at 36.83 54.61 0)
-		(fields_autoplaced yes)
-		(effects
-			(font
-				(size 1.27 1.27)
-			)
-			(justify left bottom)
 		)
 	)
@@
 		)
 	)
-	(label "OE_PWM"
-		(at 36.83 52.07 0)
-		(fields_autoplaced yes)
-		(effects
-			(font
-				(size 1.27 1.27)
-			)
-			(justify left bottom)
-		)
-	)
 	(label "6"
 		(at 151.13 54.61 0)
@@
 	(label "5"
 		(at 86.36 64.77 0)
-		(fields_autoplaced yes)
-		(effects
-			(font
-				(size 1.27 1.27)
-			)
-			(justify left bottom)
-		)
-	)
-	(label "SDA"
-		(at 86.36 46.99 0)
 		(fields_autoplaced yes)
 		(effects
@@
 		)
 	)
-	(hierarchical_label "3.3v"
-		(shape input)
-		(at 36.83 46.99 180)
-		(fields_autoplaced yes)
-		(effects
-			(font
-				(size 1.27 1.27)
-			)
-			(justify right)
-		)
-	)
+	(symbol
+		(lib_id "power:+3.3V")
+		(at 36.83 46.99 0)
+		(unit 1)
+		(exclude_from_sim no)
+		(in_bom yes)
+		(on_board yes)
+		(dnp no)
+		(fields_autoplaced yes)
+		(property "Reference" "#PWR0134"
+			(at 36.83 50.8 0)
+			(effects
+				(font
+					(size 1.27 1.27)
+				)
+				(hide yes)
+			)
+		)
+		(property "Value" "+3.3V"
+			(at 36.83 41.91 0)
+			(effects
+				(font
+					(size 1.27 1.27)
+				)
+			)
+		)
+		(property "Footprint" ""
+			(at 36.83 46.99 0)
+			(effects
+				(font
+					(size 1.27 1.27)
+				)
+				(hide yes)
+			)
+		)
+		(property "Datasheet" ""
+			(at 36.83 46.99 0)
+			(effects
+				(font
+					(size 1.27 1.27)
+				)
+				(hide yes)
+			)
+		)
+		(property "Description" "Power symbol creates a global label with name \"+3.3V\""
+			(at 36.83 46.99 0)
+			(effects
+				(font
+					(size 1.27 1.27)
+				)
+				(hide yes)
+			)
+		)
+		(pin "1"
+		)
+		(instances
+			(project ""
+				(path "/e63e39d7-6ac0-4ffd-8aa3-1841a4541b55/dbf465c7-7de0-4b8a-860d-b014ecfe2e4f"
+					(reference "#PWR0134")
+					(unit 1)
+				)
+			)
+		)
+	)
