File: PWM_Generatrion.kicad_sch (KiCad schematic)
At the start: 2 parts, among them J13 302-S101, U22 PCA9685PW_118

Commit message: assigned footprints
Parts:
- J13: footprint digikey-footprints:PinHeader_2x5_P2.54mm_Drill1.2mm -> 302_S101:CONN10_302-S101_OST
Changed lines of the file:
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@@
 			)
 		)
-		(property "Footprint" "digikey-footprints:PinHeader_2x5_P2.54mm_Drill1.2mm"
+		(property "Footprint" "302_S101:CONN10_302-S101_OST"
 			(at 144.78 54.61 0)
 			(effects

Commit message: stuff
Parts:
- removed J13: 302-S101, 302_S101:CONN10_302-S101_OST, symbol dk_Rectangular-Connectors-Headers-Male-Pins:302-S101
- added J14, J20: DF11-10DP-2DSA24, CON10_2X5_UF_DF11_HIR, symbol DF11_10DP_2DSA:DF11-10DP-2DSA24
Connections:
- net 0: now also J14.5
- net 1: now also J14.6
- net 2: now also J14.7
- net 3: now also J14.8
- net 4: now also J14.9
- net 5: now also J14.10
- net 6: now also J20.1
- net 7: now also J20.2
- net 8: now also J20.3
- net 9: now also J20.4
- no-connect marks 7 -> 17
Other:
- note added: "ESC Controller Connector"
- note removed: "Backplane Connector"

Commit message: stuff
Parts:
- J14, J20: footprint CON10_2X5_UF_DF11_HIR -> DF11_10DP_2DSA_24:CON10_2X5_UF_DF11_HIR
Changed lines of the file:
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@@
 			)
 		)
-		(property "Footprint" "CON10_2X5_UF_DF11_HIR"
+		(property "Footprint" "DF11_10DP_2DSA_24:CON10_2X5_UF_DF11_HIR"
 			(at 133.35 64.77 0)
 			(effects
@@
 			)
 		)
-		(property "Footprint" "CON10_2X5_UF_DF11_HIR"
+		(property "Footprint" "DF11_10DP_2DSA_24:CON10_2X5_UF_DF11_HIR"
 			(at 133.35 35.56 0)
 			(effects

Commit message: stuff
Connections:
- net 0: now also J14.6; no longer J14.5
- net 1: now also J14.5; no longer J14.6
- net 2: now also J14.8; no longer J14.7
- net 3: now also J14.7; no longer J14.8
- net 4: now also J14.10; no longer J14.9
- net 5: now also J14.9; no longer J14.10
- net 6: now also J20.2; no longer J20.1
- net 7: now also J20.1; no longer J20.2
- net 8: now also J20.4; no longer J20.3
- net 9: now also J20.3; no longer J20.4
Changed lines of the file:
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@@
 		)
 	)
-	(label "9"
+	(label "8"
 		(at 123.19 72.39 0)
 		(fields_autoplaced yes)
@@
 		)
 	)
-	(label "2"
+	(label "3"
 		(at 123.19 50.8 0)
 		(fields_autoplaced yes)
@@
 		)
 	)
-	(label "1"
+	(label "0"
 		(at 123.19 48.26 0)
 		(fields_autoplaced yes)
@@
 		)
 	)
-	(label "4"
+	(label "5"
 		(at 123.19 55.88 0)
 		(fields_autoplaced yes)
@@
 		)
 	)
-	(label "7"
+	(label "6"
 		(at 123.19 67.31 0)
 		(fields_autoplaced yes)
@@
 		)
 	)
-	(label "6"
+	(label "7"
 		(at 123.19 64.77 0)
 		(fields_autoplaced yes)
@@
 		)
 	)
-	(label "8"
+	(label "9"
 		(at 123.19 69.85 0)
 		(fields_autoplaced yes)
@@
 		)
 	)
-	(label "3"
+	(label "2"
 		(at 123.19 53.34 0)
 		(fields_autoplaced yes)
@@
 		)
 	)
-	(label "5"
+	(label "4"
 		(at 123.19 58.42 0)
 		(fields_autoplaced yes)
@@
 		)
 	)
-	(label "0"
+	(label "1"
 		(at 123.19 45.72 0)
 		(fields_autoplaced yes)
