File: USBhub.kicad_sch (KiCad schematic)
At the start: 12 parts, among them U10 FE1.1s, U11 24LC02B-I_SN, Y2 ASTX-H12-12.000MHZ-T

Commit message: changes stuff
Parts:
- removed Y2: ASTX-H12-12.000MHZ-T, ASTX-H12-12.000MHZ-T:XTAL_ASTX-H12-12.000MHZ-T, symbol ASTX-H12-12.000MHZ-T:ASTX-H12-12.000MHZ-T
- added C22, C23: 18p, symbol Device:C
- added J10, J4, J5, J6: 482040001, CONN_48204-0001_MOL, symbol 482040001:482040001
- added Y3: ABLS-12.000MHZ-B2-T, ABLS-12.000MHZ-B2-T:XTAL_ABLS-12.000MHZ-B2-T, symbol ABLS-12.000MHZ-B2-T:ABLS-12.000MHZ-B2-T
Connections:
- net GND: now also C22.1, C23.2, J10.4, J4.4, J5.4, J6.4
- net Xin: now reaches U10.3 (XIN)
- net Xin: now also C22.2, Y3.1
- net at U10.10 (DM1): now also J4.2
- net at U10.11 (DP1): now also J4.3
- net Xout: now reaches U10.2 (XOUT)
- net Xout: now also C23.1, Y3.2
- net at U10.25 (PWRJ): now also J10.1, J4.1, J5.1, J6.1
- net at U10.4 (DM4): now also J10.2
- net at U10.5 (DP4): now also J10.3
- net at U10.6 (DM3): now also J6.2
- net at U10.7 (DP3): now also J6.3
- net at U10.8 (DM2): now also J5.2
- net at U10.9 (DP2): now also J5.3
Other:
- note added: "Clock"

Commit message: stuff
Connections:
- net +3.3V renamed 3.3v
- net +5V renamed 5v
Changed lines of the file:
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@@
+		)
+	)
+	(hierarchical_label "5v"
+		(shape input)
+		(at 177.8 64.77 90)
+		(fields_autoplaced yes)
+		(effects
+			(font
+				(size 1.27 1.27)
+			)
+			(justify left)
+		)
+	)
+	(hierarchical_label "3.3v"
+		(shape input)
+		(at 266.7 82.55 90)
+		(fields_autoplaced yes)
+		(effects
+			(font
+				(size 1.27 1.27)
+			)
+			(justify left)
+		)
+	)
+	(hierarchical_label "3.3v"
+		(shape input)
+		(at 185.42 64.77 90)
+		(fields_autoplaced yes)
+		(effects
+			(font
+				(size 1.27 1.27)
+			)
+			(justify left)
+		)
+	)
+	(hierarchical_label "USB2_N"
+		(shape bidirectional)
+		(at 154.94 83.82 180)
+		(fields_autoplaced yes)
+		(effects
+			(font
+				(size 1.27 1.27)
+			)
+			(justify right)
+		)
+	)
+	(hierarchical_label "USB2_P"
+		(shape bidirectional)
+		(at 154.94 81.28 180)
+		(fields_autoplaced yes)
+		(effects
+			(font
+				(size 1.27 1.27)
+			)
+			(justify right)
 		)
 	)
@@
 	)
 	(symbol
-		(lib_id "power:+3.3V")
-		(at 266.7 82.55 0)
-		(unit 1)
-		(exclude_from_sim no)
-		(in_bom yes)
-		(on_board yes)
-		(dnp no)
-		(fields_autoplaced yes)
-		(property "Reference" "#PWR044"
-			(at 266.7 86.36 0)
-			(effects
-				(font
-					(size 1.27 1.27)
-				)
-				(hide yes)
-			)
-		)
-		(property "Value" "+3.3V"
-			(at 266.7 77.47 0)
-			(effects
-				(font
-					(size 1.27 1.27)
-				)
-			)
-		)
-		(property "Footprint" ""
-			(at 266.7 82.55 0)
-			(effects
-				(font
-					(size 1.27 1.27)
-				)
-				(hide yes)
-			)
-		)
-		(property "Datasheet" ""
-			(at 266.7 82.55 0)
-			(effects
-				(font
-					(size 1.27 1.27)
-				)
-				(hide yes)
-			)
-		)
-		(property "Description" "Power symbol creates a global label with name \"+3.3V\""
-			(at 266.7 82.55 0)
-			(effects
-				(font
-					(size 1.27 1.27)
-				)
-				(hide yes)
-			)
-		)
-		(pin "1"
-		)
-		(instances
-			(project ""
-				(path "/e63e39d7-6ac0-4ffd-8aa3-1841a4541b55/6cbc9825-ddcf-4552-a506-0d903a9900c6"
-					(reference "#PWR044")
-					(unit 1)
-				)
-			)
-		)
-	)
-	(symbol
 		(lib_id "Device:R")
 		(at 209.55 114.3 270)
@@
 	)
 	(symbol
-		(lib_id "power:+5V")
-		(at 177.8 64.77 0)
-		(unit 1)
-		(exclude_from_sim no)
-		(in_bom yes)
-		(on_board yes)
-		(dnp no)
-		(fields_autoplaced yes)
-		(property "Reference" "#PWR036"
-			(at 177.8 68.58 0)
-			(effects
-				(font
-					(size 1.27 1.27)
-				)
-				(hide yes)
-			)
-		)
-		(property "Value" "+5V"
-			(at 177.8 59.69 0)
-			(effects
-				(font
-					(size 1.27 1.27)
-				)
-			)
-		)
-		(property "Footprint" ""
-			(at 177.8 64.77 0)
-			(effects
-				(font
-					(size 1.27 1.27)
-				)
-				(hide yes)
-			)
-		)
-		(property "Datasheet" ""
-			(at 177.8 64.77 0)
-			(effects
-				(font
-					(size 1.27 1.27)
-				)
-				(hide yes)
-			)
-		)
-		(property "Description" "Power symbol creates a global label with name \"+5V\""
-			(at 177.8 64.77 0)
-			(effects
-				(font
-					(size 1.27 1.27)
-				)
-				(hide yes)
-			)
-		)
-		(pin "1"
-		)
-		(instances
-			(project ""
-				(path "/e63e39d7-6ac0-4ffd-8aa3-1841a4541b55/6cbc9825-ddcf-4552-a506-0d903a9900c6"
-					(reference "#PWR036")
-					(unit 1)
-				)
-			)
-		)
-	)
-	(symbol
 		(lib_id "Device:C")
 		(at 196.85 57.15 0)
@@
 					(unit 1)
 				)
-			)
-		)
-	)
-	(symbol
-		(lib_id "power:+3.3V")
-		(at 185.42 64.77 0)
-		(unit 1)
-		(exclude_from_sim no)
-		(in_bom yes)
-		(on_board yes)
-		(dnp no)
-		(fields_autoplaced yes)
-		(property "Reference" "#PWR037"
-			(at 185.42 68.58 0)
-			(effects
-				(font
-					(size 1.27 1.27)
-				)
-				(hide yes)
-			)
-		)
-		(property "Value" "+3.3V"
-			(at 185.42 59.69 0)
-			(effects
-				(font
-					(size 1.27 1.27)
-				)
-			)
-		)
-		(property "Footprint" ""
-			(at 185.42 64.77 0)
-			(effects
-				(font
-					(size 1.27 1.27)
-				)
-				(hide yes)
-			)
-		)
-		(property "Datasheet" ""
-			(at 185.42 64.77 0)
-			(effects
-				(font
-					(size 1.27 1.27)
-				)
-				(hide yes)
-			)
-		)
-		(property "Description" "Power symbol creates a global label with name \"+3.3V\""
-			(at 185.42 64.77 0)
-			(effects
-				(font
-					(size 1.27 1.27)
-				)
-				(hide yes)
-			)
-		)
-		(pin "1"
-		)
-		(instances
-			(project ""
-				(path "/e63e39d7-6ac0-4ffd-8aa3-1841a4541b55/6cbc9825-ddcf-4552-a506-0d903a9900c6"
-					(reference "#PWR037")
-					(unit 1)
-				)

Commit message: stuff
Connections:
- net 3.3v: no longer U10.13 (VD33)
- net 5v: now also U10.18 (VBUSM)
- net at J10.1, J4.1, J5.1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: now also U10.21 (VD33_O); no longer U10.25 (PWRJ)
Changed lines of the file:
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@@
+	)
+	(junction
+		(at 213.36 138.43)
+		(diameter 0)
+		(color 0 0 0 0)
+	)
+	(junction
+		(at 134.62 67.31)
+		(diameter 0)
+		(color 0 0 0 0)
+	)
+	(junction
+		(at 226.06 125.73)
+		(diameter 0)
+		(color 0 0 0 0)
+	)
+	(junction
+		(at 200.66 157.48)
+		(diameter 0)
+		(color 0 0 0 0)
+	)
+	(junction
+		(at 203.2 54.61)
+		(diameter 0)
+		(color 0 0 0 0)
+	)
+	(junction
+		(at 224.79 125.73)
+		(diameter 0)
+		(color 0 0 0 0)
+	)
+	(junction
+		(at 242.57 125.73)
+		(diameter 0)
+		(color 0 0 0 0)
+	)
+	(junction
+		(at 200.66 138.43)
+		(diameter 0)
+		(color 0 0 0 0)
+	)
+	(junction
+		(at 200.66 153.67)
+		(diameter 0)
+		(color 0 0 0 0)
+	)
+	(junction
+		(at 232.41 62.23)
+		(diameter 0)
+		(color 0 0 0 0)
+	)
+	(junction
+		(at 143.51 58.42)
+		(diameter 0)
+		(color 0 0 0 0)
+	)
+	(junction
+		(at 127 55.88)
+		(diameter 0)
+		(color 0 0 0 0)
+	)
+	(junction
+		(at 200.66 142.24)
+		(diameter 0)
+		(color 0 0 0 0)
+	)
+	(junction
+		(at 232.41 77.47)
+		(diameter 0)
+		(color 0 0 0 0)
+	)
+	(junction
+		(at 177.8 68.58)
+		(diameter 0)
+		(color 0 0 0 0)
+	)
+	(junction
+		(at 232.41 45.72)
+		(diameter 0)
+		(color 0 0 0 0)
 	)
 	(junction
@@
 		(color 0 0 0 0)
 	)
-	(junction
-		(at 213.36 138.43)
-		(diameter 0)
-		(color 0 0 0 0)
-	)
-	(junction
-		(at 134.62 67.31)
-		(diameter 0)
-		(color 0 0 0 0)
-	)
-	(junction
-		(at 226.06 125.73)
-		(diameter 0)
-		(color 0 0 0 0)
-	)
-	(junction
-		(at 200.66 157.48)
-		(diameter 0)
-		(color 0 0 0 0)
-	)
-	(junction
-		(at 203.2 54.61)
-		(diameter 0)
-		(color 0 0 0 0)
-	)
-	(junction
-		(at 224.79 125.73)
-		(diameter 0)
-		(color 0 0 0 0)
-	)
-	(junction
-		(at 242.57 125.73)
-		(diameter 0)
-		(color 0 0 0 0)
-	)
-	(junction
-		(at 200.66 138.43)
-		(diameter 0)
-		(color 0 0 0 0)
-	)
-	(junction
-		(at 200.66 153.67)
-		(diameter 0)
-		(color 0 0 0 0)
-	)
-	(junction
-		(at 232.41 62.23)
-		(diameter 0)
-		(color 0 0 0 0)
-	)
-	(junction
-		(at 143.51 58.42)
-		(diameter 0)
-		(color 0 0 0 0)
-	)
-	(junction
-		(at 127 55.88)
-		(diameter 0)
-		(color 0 0 0 0)
-	)
-	(junction
-		(at 200.66 142.24)
-		(diameter 0)
-		(color 0 0 0 0)
-	)
-	(junction
-		(at 232.41 77.47)
-		(diameter 0)
-		(color 0 0 0 0)
-	)
-	(junction
-		(at 232.41 45.72)
-		(diameter 0)
-		(color 0 0 0 0)
-	)
 	(wire
 		(pts
@@
 	(wire
 		(pts
+			(xy 161.29 68.58) (xy 177.8 68.58)
+		)
+		(stroke
+			(width 0)
+			(type default)
+		)
+	)
+	(wire
+		(pts
 			(xy 187.96 64.77) (xy 196.85 64.77)
 		)
@@
 	(wire
 		(pts
+			(xy 161.29 76.2) (xy 161.29 68.58)
+		)
+		(stroke
+			(width 0)
+			(type default)
+		)
+	)
+	(wire
+		(pts
 			(xy 127 67.31) (xy 134.62 67.31)
 		)
@@
 	(wire
 		(pts
+			(xy 177.8 68.58) (xy 177.8 71.12)
+		)
+		(stroke
+			(width 0)
+			(type default)
+		)
+	)
+	(wire
+		(pts
 			(xy 127 55.88) (xy 127 53.34)
 		)
@@
 	(wire
 		(pts
-			(xy 177.8 64.77) (xy 177.8 71.12)
+			(xy 177.8 64.77) (xy 177.8 68.58)
 		)
 		(stroke
@@
 	(wire
 		(pts
-			(xy 200.66 121.92) (xy 203.2 121.92)
+			(xy 165.1 76.2) (xy 161.29 76.2)
 		)
 		(stroke
@@
 	(wire
 		(pts
-			(xy 185.42 64.77) (xy 185.42 71.12)
-		)
-		(stroke
-			(width 0)
-			(type default)
-		)
-	)
-	(wire
-		(pts
-			(xy 203.2 69.85) (xy 203.2 121.92)
+			(xy 182.88 69.85) (xy 182.88 71.12)
+		)
+		(stroke
+			(width 0)
+			(type default)
+		)
+	)
+	(wire
+		(pts
+			(xy 203.2 69.85) (xy 182.88 69.85)
 		)
 		(stroke
@@
 		(fields_autoplaced yes)
 		(effects
-			(font
-				(size 1.27 1.27)
-			)
-			(justify left)
-		)
-	)
-	(hierarchical_label "3.3v"
-		(shape input)
-		(at 185.42 64.77 90)
-		(fields_autoplaced yes)
-		(effects

Commit message: stuff
Parts:
- added C8: 0.1u, symbol Device:C
- added R6: 2.7k, symbol Device:R
Connections:
- net 5v: now also C8.1
- net GND: now also C8.2, R6.2
- net at U10.14 (REXT): now also R6.1
- no-connect marks 0 -> 4
Other:
- note added: "connect OVCJ, BUSJ with a LED indicator Connect XRSTJ with a testpoint/headerpin (or connect to pi for debugging purpose)"

Commit message: stuff
Parts:
- removed C50: .1u, symbol Device:C
- added D4, D9: LED, symbol Device:LED
- added R19, R7: 1k, symbol Device:R
Connections:
- net 5v: now also J10.1, J4.1, J5.1, J6.1
- net GND: now also R19.1, R7.1
- net DRV: now reaches D3.1 (K), D5.2 (A), D6.1 (K), D7.2 (A), D8.2 (A), U10.22 (DRV)
- net DM1: now reaches J4.2, U10.10 (DM1)
- net DP1: now reaches J4.3, U10.11 (DP1)
- net LED1/EESCL: now reaches R34.1, U10.23 (LED1/EESCL), U11.6 (SCL)
- net LED2: now reaches R33.2, U10.24 (LED2)
- net DM2: now reaches J5.2, U10.8 (DM2)
- net DP2: now reaches J5.3, U10.9 (DP2)
- net DM4: now reaches J10.2, U10.4 (DM4)
- net DP4: now reaches J10.3, U10.5 (DP4)
- net EESDA: now reaches U10.27 (TESTJ/EESDA), U11.5 (SDA)
- net DM3: now reaches J6.2, U10.6 (DM3)
- net DP3: now reaches J6.3, U10.7 (DP3)
- net XRSTJ: now reaches U10.17 (~{XRSTJ})
- net BUSJ: now reaches U10.19 (BUSJ)
- net BUSJ: now also D4.2 (A)
- net OVCJ: now reaches U10.26 (OVCJ)
- net OVCJ: now also D9.2 (A)
- new net: D9.1 (K), R19.2
- new net: D4.1 (K), R7.2
- now unconnected: U10.21 (VD33_O)
- no-connect marks 4 -> 6
Other:
- note added: "Activity Leds"
- note added: "Bus Power"
- note added: "EEPROM"
- note added: "Overcurrent"
- note added: "USB 2.0 Hub"
- note added: "USB 2.0 Type A"
- note removed: "connect OVCJ, BUSJ with a LED indicator Connect XRSTJ with a testpoint/headerpin (or connect to pi for debugging purpose)"
- moved on the sheet: C22, C23, C8, D3, D5, D6, D7, D8, J10, J4, J5, J6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

Commit message: stuff
Connections:
- net 3.3v renamed +3.3V
- net 5v renamed +5V

Commit message: stuff
Changed lines of the file:
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@@
 	(wire
 		(pts
-			(xy 33.02 33.02) (xy 33.02 34.29)
-		)
-		(stroke
-			(width 0)
-			(type default)
-		)
-	)
-	(wire
-		(pts
 			(xy 31.75 48.26) (xy 36.83 48.26)
 		)
@@
 	(symbol
 		(lib_id "power:GND")
-		(at 33.02 34.29 0)
+		(at 33.02 33.02 0)
 		(unit 1)
 		(exclude_from_sim no)
@@
 		(dnp no)
 		(property "Reference" "#PWR01"
-			(at 33.02 40.64 0)
+			(at 33.02 39.37 0)
 			(effects
 				(font
@@
 		)
 		(property "Value" "GND"
-			(at 35.306 34.798 0)
+			(at 35.306 33.528 0)
 			(effects
 				(font
@@
 		)
 		(property "Footprint" ""
-			(at 33.02 34.29 0)
+			(at 33.02 33.02 0)
 			(effects
 				(font
@@
 		)
 		(property "Datasheet" ""
-			(at 33.02 34.29 0)
+			(at 33.02 33.02 0)
 			(effects
 				(font
@@
 		)
 		(property "Description" "Power symbol creates a global label with name \"GND\" , ground"
-			(at 33.02 34.29 0)
+			(at 33.02 33.02 0)
 			(effects
 				(font
