File: USBhub.kicad_sch (KiCad schematic)
At the start: 23 parts, among them J10 482040001, J4 482040001, J5 482040001, J6 482040001, U10 FE1.1s, U11 24LC02B-I_SN, Y3 ABLS-12.000MHZ-B2-T

Commit message: assigned footprints
Parts:
- C22, C23, C8: footprint (none) -> Capacitor_SMD:C_0805_2012Metric
- D3, D4, D5, D6, D7, D8, D9: footprint (none) -> LED_SMD:LED_0805_2012Metric
- J10, J4, J5, J6: footprint CONN_48204-0001_MOL -> USBA-Port:CONN_48204-0001_MOL
- R19, R33, R34, R35, R6, R7: footprint (none) -> Resistor_SMD:R_0805_2012Metric
Changed lines of the file:
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@@
 			)
 		)
-		(property "Footprint" ""
+		(property "Footprint" "LED_SMD:LED_0805_2012Metric"
 			(at 34.29 138.43 0)
 			(effects
@@
 			)
 		)
-		(property "Footprint" ""
+		(property "Footprint" "Resistor_SMD:R_0805_2012Metric"
 			(at 29.972 83.82 90)
 			(effects
@@
 			)
 		)
-		(property "Footprint" "CONN_48204-0001_MOL"
+		(property "Footprint" "USBA-Port:CONN_48204-0001_MOL"
 			(at 135.89 34.29 0)
 			(effects
@@
 			)
 		)
-		(property "Footprint" ""
+		(property "Footprint" "LED_SMD:LED_0805_2012Metric"
 			(at 34.29 153.67 0)
 			(effects
@@
 			)
 		)
-		(property "Footprint" ""
+		(property "Footprint" "LED_SMD:LED_0805_2012Metric"
 			(at 34.29 157.48 0)
 			(effects
@@
 			)
 		)
-		(property "Footprint" ""
+		(property "Footprint" "Resistor_SMD:R_0805_2012Metric"
 			(at 49.53 136.652 90)
 			(effects
@@
 			)
 		)
-		(property "Footprint" ""
+		(property "Footprint" "Resistor_SMD:R_0805_2012Metric"
 			(at 49.53 155.448 90)
 			(effects
@@
 			)
 		)
-		(property "Footprint" ""
+		(property "Footprint" "Resistor_SMD:R_0805_2012Metric"
 			(at 60.96 159.512 90)
 			(effects
@@
 			)
 		)
-		(property "Footprint" "CONN_48204-0001_MOL"
+		(property "Footprint" "USBA-Port:CONN_48204-0001_MOL"
 			(at 135.89 49.53 0)
 			(effects
@@
 			)
 		)
-		(property "Footprint" ""
+		(property "Footprint" "Capacitor_SMD:C_0805_2012Metric"
 			(at 33.9852 33.02 0)
 			(effects
@@
 			)
 		)
-		(property "Footprint" "CONN_48204-0001_MOL"
+		(property "Footprint" "USBA-Port:CONN_48204-0001_MOL"
 			(at 135.89 81.28 0)
 			(effects
@@
 			)
 		)
-		(property "Footprint" ""
+		(property "Footprint" "LED_SMD:LED_0805_2012Metric"
 			(at 50.8 161.29 0)
 			(effects
@@
 			)
 		)
-		(property "Footprint" ""
+		(property "Footprint" "Resistor_SMD:R_0805_2012Metric"
 			(at 41.91 126.238 90)
 			(effects
@@
 			)
 		)
-		(property "Footprint" ""
+		(property "Footprint" "Capacitor_SMD:C_0805_2012Metric"
 			(at 95.5548 137.16 0)
 			(effects
@@
 			)
 		)
-		(property "Footprint" ""
+		(property "Footprint" "LED_SMD:LED_0805_2012Metric"
 			(at 34.29 142.24 0)
 			(effects
@@
 			)
 		)
-		(property "Footprint" "CONN_48204-0001_MOL"
+		(property "Footprint" "USBA-Port:CONN_48204-0001_MOL"
 			(at 135.89 66.04 0)
 			(effects
@@
 			)
 		)
-		(property "Footprint" ""
+		(property "Footprint" "Capacitor_SMD:C_0805_2012Metric"
 			(at 113.9952 144.78 0)
 			(effects
@@
 			)
 		)
-		(property "Footprint" ""
+		(property "Footprint" "LED_SMD:LED_0805_2012Metric"
 			(at 52.07 124.46 0)
 			(effects
@@
 			)
 		)
-		(property "Footprint" ""
+		(property "Footprint" "Resistor_SMD:R_0805_2012Metric"
 			(at 41.91 117.348 90)
 			(effects
@@
 			)
 		)
-		(property "Footprint" ""
+		(property "Footprint" "LED_SMD:LED_0805_2012Metric"
 			(at 52.07 115.57 0)
 			(effects

Commit message: stuff
Parts:
- U11: footprint 24LC02B-I_SN:SOIC127P600X175-8N -> 24LC02B_I_SN:SOIC127P600X175-8N
- Y3: footprint ABLS-12.000MHZ-B2-T:XTAL_ABLS-12.000MHZ-B2-T -> ABLS_12_000MHZ_B2_T:XTAL_ABLS-12.000MHZ-B2-T
Changed lines of the file:
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@@
 			)
 		)
-		(property "Footprint" "ABLS-12.000MHZ-B2-T:XTAL_ABLS-12.000MHZ-B2-T"
+		(property "Footprint" "ABLS_12_000MHZ_B2_T:XTAL_ABLS-12.000MHZ-B2-T"
 			(at 104.14 130.81 0)
 			(effects
@@
 			)
 		)
-		(property "Footprint" "24LC02B-I_SN:SOIC127P600X175-8N"
+		(property "Footprint" "24LC02B_I_SN:SOIC127P600X175-8N"
 			(at 210.82 62.23 0)
 			(effects

Commit message: stuff
Other:
- note added: "Do I need 1k pull up?"
Changed lines of the file:
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@@
+		)
+	)
+	(text "Do I need 1k pull up?\n"
+		(exclude_from_sim no)
+		(at 186.182 72.136 0)
+		(effects
+			(font
+				(size 1.27 1.27)
+			)
 		)
 	)

Commit message: STUFF
Connections:
- net DM1 renamed D1-
- net DM2 renamed D2-
- net DM3 renamed D3-
- net DM4 renamed D4-
- net DP1 renamed D1+
- net DP2 renamed D2+
- net DP3 renamed D3+
- net DP4 renamed D4+
Changed lines of the file:
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@@
 		)
 	)
-	(label "DP1"
+	(label "D1+"
 		(at 124.46 39.37 0)
 		(fields_autoplaced yes)
@@
 		)
 	)
-	(label "DP3"
+	(label "D3+"
 		(at 74.93 48.26 0)
 		(fields_autoplaced yes)
@@
 		)
 	)
-	(label "DM3"
+	(label "D3-"
 		(at 74.93 50.8 0)
 		(fields_autoplaced yes)
@@
 		)
 	)
-	(label "DP1"
+	(label "D1+"
 		(at 74.93 33.02 0)
 		(fields_autoplaced yes)
@@
 		)
 	)
-	(label "DP4"
+	(label "D4+"
 		(at 124.46 86.36 0)
 		(fields_autoplaced yes)
@@
 		)
 	)
-	(label "DM4"
+	(label "D4-"
 		(at 124.46 83.82 0)
 		(fields_autoplaced yes)
@@
 		)
 	)
-	(label "DP2"
+	(label "D2+"
 		(at 124.46 54.61 0)
 		(fields_autoplaced yes)
@@
 		)
 	)
-	(label "DM1"
+	(label "D1-"
 		(at 74.93 35.56 0)
 		(fields_autoplaced yes)
@@
 		)
 	)
-	(label "DM1"
+	(label "D1-"
 		(at 124.46 36.83 0)
 		(fields_autoplaced yes)
@@
 		)
 	)
-	(label "DM2"
+	(label "D2-"
 		(at 124.46 52.07 0)
 		(fields_autoplaced yes)
@@
 		)
 	)
-	(label "DP4"
+	(label "D4+"
 		(at 74.93 55.88 0)
 		(fields_autoplaced yes)
@@
 		)
 	)
-	(label "DM4"
+	(label "D4-"
 		(at 74.93 58.42 0)
 		(fields_autoplaced yes)
@@
 		)
 	)
-	(label "DP2"
+	(label "D2+"
 		(at 74.93 40.64 0)
 		(fields_autoplaced yes)
@@
 		)
 	)
-	(label "DM2"
+	(label "D2-"
 		(at 74.93 43.18 0)
 		(fields_autoplaced yes)
@@
 		)
 	)
-	(label "DM3"
+	(label "D3-"
 		(at 124.46 68.58 0)
 		(fields_autoplaced yes)
@@
 		)
 	)
-	(label "DP3"
+	(label "D3+"
 		(at 124.46 71.12 0)
 		(fields_autoplaced yes)
