File: CM4_HighSpeed.kicad_sch (KiCad schematic)
At the start: 11 parts, among them J15 Conn_01x22_Female, J16 Conn_01x22_Female, J4 Conn_01x22_Female, J5 Conn_01x22_Female, J6 THD-02-R, U12 RT9742SNGV

Commit message: board
Parts:
- removed C12, C13: 100n, Capacitor_SMD:C_0402_1005Metric, symbol Device:C
- removed J15, J16, J4, J5: Conn_01x22_Female, CM4IO:Hirose_FH12-22S-0.5SH_1x22-1MP_P0.50mm_Horizontal, symbol Connector:Conn_01x22_Female
- removed J6: THD-02-R, Connector_PinHeader_2.54mm:PinHeader_2x02_P2.54mm_Vertical, symbol Connector_Generic:Conn_02x02_Odd_Even
- removed R6, R7: 2.2K 1%, Resistor_SMD:R_0402_1005Metric, symbol Device:R
- removed U12: RT9742SNGV, Package_TO_SOT_SMD:SOT-23, symbol CM4IO:RT9742SNGV
Connections:
- no-connect marks 16 -> 2
Other:
- note removed: "Camera Connectors"
- note removed: "Display Connectors"
- note removed: "Jumpers to be fitted if Camera0 or Display0 are used."

Commit message: stuff
Parts:
- added C80, C81: 100n, Capacitor_SMD:C_0402_1005Metric, symbol Device:C
- added J26: 690-019-298-412, CM4IO:EDAC 690-019-298-412, symbol CM4IO:HDMI_A_1.4
- added U25: RT9742SNGV, Package_TO_SOT_SMD:SOT-23, symbol CM4IO:RT9742SNGV
Connections:
- net GND: now also C80.2, C81.2, J26.11 (CKS), J26.17 (GND), J26.2 (D2S), J26.5 (D1S), J26.8 (D0S), J26.SH1 (SH), J26.SH2 (SH), J26.SH3 (SH), J26.SH4 (SH), U25.3 (GND)
- net HDMI0_CEC: now also J26.13 (CEC)
- net HDMI0_CK_N: now also J26.12 (CK-)
- net HDMI0_CK_P: now also J26.10 (CK+)
- net HDMI0_D0_N: now also J26.9 (D0-)
- net HDMI0_D0_P: now also J26.7 (D0+)
- net HDMI0_D1_N: now also J26.6 (D1-)
- net HDMI0_D1_P: now also J26.4 (D1+)
- net HDMI0_D2_N: now also J26.3 (D2-)
- net HDMI0_D2_P: now also J26.1 (D2+)
- net HDMI0_HOTPLUG: now also J26.19 (HPD/HEAC-)
- net HDMI0_SCL: now also J26.15 (SCL)
- net HDMI0_SDA: now also J26.16 (SDA)
- new net +5v: C80.1, U25.1 (IN)
- new net HDMI_5v: C81.1, J26.18 (+5V), U25.2 (OUT)
- no-connect marks 2 -> 3

Commit message: stuff
Connections:
- net PCIE_CLK_N: no longer names the net of Module1.112 (PCIe_CLK_N)
- net PCIE_CLK_P: no longer names the net of Module1.110 (PCIe_CLK_P)
- net PCIE_CLK_nREQ: no longer names the net of Module1.102 (PCIe_CLK_nREQ)
- net PCIE_RX_N: no longer names the net of Module1.118 (PCIe_RX_N)
- net PCIE_RX_P: no longer names the net of Module1.116 (PCIe_RX_P)
- net PCIE_TX_N: no longer names the net of Module1.124 (PCIe_TX_N)
- net PCIE_TX_P: no longer names the net of Module1.122 (PCIe_TX_P)
Changed lines of the file:
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@@
-		)
-	)
-	(hierarchical_label "PCIE_RX_P"
-		(shape input)
-		(at 35.56 44.45 180)
-		(fields_autoplaced yes)
-		(effects
-			(font
-				(size 1.27 1.27)
-			)
-			(justify right)
 		)
 	)
@@
 		)
 	)
-	(hierarchical_label "PCIE_CLK_N"
-		(shape output)
-		(at 35.56 39.37 180)
-		(fields_autoplaced yes)
-		(effects
-			(font
-				(size 1.27 1.27)
-			)
-			(justify right)
-		)
-	)
 	(hierarchical_label "PCIE_nRST"
 		(shape output)
@@
 			)
 			(justify left)
-		)
-	)
-	(hierarchical_label "PCIE_RX_N"
-		(shape input)
-		(at 35.56 46.99 180)
-		(fields_autoplaced yes)
-		(effects
-			(font
-				(size 1.27 1.27)
-			)
-			(justify right)
-		)
-	)
-	(hierarchical_label "PCIE_CLK_nREQ"
-		(shape input)
-		(at 35.56 26.67 180)
-		(fields_autoplaced yes)
-		(effects
-			(font
-				(size 1.27 1.27)
-			)
-			(justify right)
 		)
 	)
@@
 		)
 	)
-	(hierarchical_label "PCIE_TX_N"
-		(shape output)
-		(at 35.56 54.61 180)
-		(fields_autoplaced yes)
-		(effects
-			(font
-				(size 1.27 1.27)
-			)
-			(justify right)
-		)
-	)
-	(hierarchical_label "PCIE_TX_P"
-		(shape output)
-		(at 35.56 52.07 180)
-		(fields_autoplaced yes)
-		(effects
-			(font
-				(size 1.27 1.27)
-			)
-			(justify right)
-		)
-	)
 	(hierarchical_label "USB2_N"
 		(shape bidirectional)
@@
 		)
 	)
-	(hierarchical_label "PCIE_CLK_P"
-		(shape output)
-		(at 35.56 36.83 180)
-		(fields_autoplaced yes)
-		(effects
-			(font
-				(size 1.27 1.27)
-			)
-			(justify right)
-		)
-	)

Commit message: stuff
Parts:
- added J12: THD-02-R, Connector_PinHeader_2.54mm:PinHeader_2x02_P2.54mm_Vertical, symbol Connector_Generic:Conn_02x02_Odd_Even
- added R21, R22: 2.2K 1%, Resistor_SMD:R_0402_1005Metric, symbol Device:R
Connections:
- net PCIE_nRST: no longer names the net of Module1.109 (PCIe_nRST)
- net USBOTG_ID: no longer names the net of Module1.101 (USB_OTG_ID)
- new net GPIO_VREF: R21.1, R22.1
- new net ID_SC: J12.1 (Pin_1)
- new net ID_SD: J12.3 (Pin_3)
- new net SCL1: J12.2 (Pin_2), R22.2
- new net SDA1: J12.4 (Pin_4), R21.2
- no-connect marks 3 -> 56
Other:
- note added: "Jumpers to be fitted if Camera0 or Display0 are used."

Commit message: stuff
Connections:
- net HDMI_5v renamed +5VL
Changed lines of the file:
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@@
-		)
-	)
-	(label "HDMI_5v"
-		(at 102.87 180.34 180)
-		(fields_autoplaced yes)
-		(effects
-			(font
-				(size 1.27 1.27)
-			)
-			(justify right bottom)
 		)
 	)
@@
 	(label "HDMI0_CK_N"
 		(at 228.6 49.53 0)
-		(fields_autoplaced yes)
-		(effects
-			(font
-				(size 1.27 1.27)
-			)
-			(justify left bottom)
-		)
-	)
-	(label "HDMI_5v"
-		(at 247.65 21.59 0)
 		(fields_autoplaced yes)
 		(effects
@@
 	)
 	(symbol
+		(lib_id "power:+5VL")
+		(at 104.14 180.34 0)
+		(unit 1)
+		(exclude_from_sim no)
+		(in_bom yes)
+		(on_board yes)
+		(dnp no)
+		(fields_autoplaced yes)
+		(property "Reference" "#PWR022"
+			(at 104.14 184.15 0)
+			(effects
+				(font
+					(size 1.27 1.27)
+				)
+				(hide yes)
+			)
+		)
+		(property "Value" "+5VL"
+			(at 104.14 175.26 0)
+			(effects
+				(font
+					(size 1.27 1.27)
+				)
+			)
+		)
+		(property "Footprint" ""
+			(at 104.14 180.34 0)
+			(effects
+				(font
+					(size 1.27 1.27)
+				)
+				(hide yes)
+			)
+		)
+		(property "Datasheet" ""
+			(at 104.14 180.34 0)
+			(effects
+				(font
+					(size 1.27 1.27)
+				)
+				(hide yes)
+			)
+		)
+		(property "Description" "Power symbol creates a global label with name \"+5VL\""
+			(at 104.14 180.34 0)
+			(effects
+				(font
+					(size 1.27 1.27)
+				)
+				(hide yes)
+			)
+		)
+		(pin "1"
+		)
+		(instances
+			(project ""
+				(path "/e63e39d7-6ac0-4ffd-8aa3-1841a4541b55/00000000-0000-0000-0000-00005cff70b1"
+					(reference "#PWR022")
+					(unit 1)
+				)
+			)
+		)
+	)
+	(symbol
 		(lib_id "power:GND")
 		(at 60.96 187.96 0)
@@
 					(unit 1)
 				)
+			)
+		)
+	)
+	(symbol
+		(lib_id "power:+5VL")
+		(at 246.38 21.59 0)
+		(unit 1)
+		(exclude_from_sim no)
+		(in_bom yes)
+		(on_board yes)
+		(dnp no)
+		(fields_autoplaced yes)
+		(property "Reference" "#PWR029"
+			(at 246.38 25.4 0)
+			(effects
+				(font
+					(size 1.27 1.27)
+				)
+				(hide yes)
+			)
+		)
+		(property "Value" "+5VL"
+			(at 246.38 16.51 0)
+			(effects
+				(font
+					(size 1.27 1.27)
+				)
+			)
+		)
+		(property "Footprint" ""
+			(at 246.38 21.59 0)
+			(effects
+				(font
+					(size 1.27 1.27)
+				)
+				(hide yes)
+			)
+		)
+		(property "Datasheet" ""
+			(at 246.38 21.59 0)
+			(effects
+				(font
+					(size 1.27 1.27)
+				)
+				(hide yes)
+			)
+		)
+		(property "Description" "Power symbol creates a global label with name \"+5VL\""
+			(at 246.38 21.59 0)
+			(effects
+				(font
+					(size 1.27 1.27)
+				)
+				(hide yes)
+			)
+		)
+		(pin "1"
+		)
+		(instances
+			(project "CM4IOv5"
+				(path "/e63e39d7-6ac0-4ffd-8aa3-1841a4541b55/00000000-0000-0000-0000-00005cff70b1"
+					(reference "#PWR029")
+					(unit 1)
+				)

Commit message: stuff
Connections:
- net +5v renamed +5V
Other:
- note added: "5vl: The power for the HDMI"
Changed lines of the file:
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@@
 	)
 	(junction
+		(at 181.61 142.113)
+		(diameter 0)
+		(color 0 0 0 0)
+	)
+	(junction
 		(at 39.37 110.49)
 		(diameter 1.016)
@@
 	)
 	(junction
+		(at 189.23 142.113)
+		(diameter 0)
+		(color 0 0 0 0)
+	)
+	(junction
 		(at 105.41 148.59)
 		(diameter 1.016)
@@
 	)
 	(junction
-		(at 39.37 118.11)
-		(diameter 1.016)
+		(at 181.61 140.97)
+		(diameter 0)
 		(color 0 0 0 0)
 	)
 	(junction
-		(at 250.19 80.01)
+		(at 39.37 118.11)
 		(diameter 1.016)
 		(color 0 0 0 0)
 	)
 	(junction
-		(at 105.41 102.87)
+		(at 250.19 80.01)
 		(diameter 1.016)
 		(color 0 0 0 0)
 	)
 	(junction
-		(at 181.61 140.589)
+		(at 105.41 102.87)
 		(diameter 1.016)
 		(color 0 0 0 0)
@@
 	(wire
 		(pts
+			(xy 189.23 142.113) (xy 189.23 142.24)
+		)
+		(stroke
+			(width 0)
+			(type default)
+		)
+	)
+	(wire
+		(pts
 			(xy 39.37 80.01) (xy 39.37 87.63)
 		)
@@
 	(wire
 		(pts
-			(xy 189.23 140.589) (xy 189.23 142.113)
-		)
-		(stroke
-			(width 0)
-			(type solid)
-		)
-	)
-	(wire
-		(pts
 			(xy 189.23 149.733) (xy 189.23 154.94)
 		)
@@
 	(wire
 		(pts
+			(xy 168.91 139.7) (xy 168.91 140.97)
+		)
+		(stroke
+			(width 0)
+			(type default)
+		)
+	)
+	(wire
+		(pts
 			(xy 35.56 54.61) (xy 41.91 54.61)
 		)
@@
 	(wire
 		(pts
-			(xy 181.61 140.589) (xy 189.23 140.589)
-		)
-		(stroke
-			(width 0)
-			(type solid)
-		)
-	)
-	(wire
-		(pts
 			(xy 105.41 57.15) (xy 105.41 49.53)
 		)
@@
 	(wire
 		(pts
-			(xy 171.958 140.589) (xy 181.61 140.589)
-		)
-		(stroke
-			(width 0)
-			(type solid)
-		)
-	)
-	(wire
-		(pts
-			(xy 181.61 140.589) (xy 181.61 142.113)
+			(xy 60.96 180.34) (xy 72.39 180.34)
 		)
 		(stroke
@@
 	(wire
 		(pts
-			(xy 60.96 180.34) (xy 72.39 180.34)
+			(xy 41.91 135.89) (xy 25.4 135.89)
 		)
 		(stroke
@@
 	(wire
 		(pts
-			(xy 41.91 135.89) (xy 25.4 135.89)
+			(xy 181.61 140.97) (xy 181.61 142.113)
 		)
 		(stroke
 			(width 0)
-			(type solid)
+			(type default)
 		)
 	)
@@
 	(wire
 		(pts
+			(xy 181.61 142.113) (xy 181.61 142.24)
+		)
+		(stroke
+			(width 0)
+			(type default)
+		)
+	)
+	(wire
+		(pts
 			(xy 105.41 34.29) (xy 102.87 34.29)
 		)
@@
 	(wire
 		(pts
+			(xy 168.91 140.97) (xy 181.61 140.97)
+		)
+		(stroke
+			(width 0)
+			(type default)
+		)
+	)
+	(wire
+		(pts
 			(xy 35.56 26.67) (xy 41.91 26.67)
 		)
@@
 	(wire
 		(pts
+			(xy 181.61 140.97) (xy 189.23 140.97)
+		)
+		(stroke
+			(width 0)
+			(type default)
+		)
+	)
+	(wire
+		(pts
 			(xy 39.37 72.39) (xy 39.37 80.01)
 		)
@@
 	(wire
 		(pts
+			(xy 189.23 140.97) (xy 189.23 142.113)
+		)
+		(stroke
+			(width 0)
+			(type default)
+		)
+	)
+	(wire
+		(pts
 			(xy 102.87 105.41) (xy 119.38 105.41)
 		)
@@
 		)
 	)
+	(text "5vl: The power for the HDMI\n"
+		(exclude_from_sim no)
+		(at 120.904 179.832 0)
+		(effects
+			(font
+				(size 1.27 1.27)
+			)
+		)
+	)
 	(label "HDMI0_CK_P"
 		(at 36.83 135.89 180)
@@
 		)
 	)
-	(label "GPIO_VREF"
-		(at 171.958 140.589 0)
-		(fields_autoplaced yes)
-		(effects
-			(font
-				(size 1.27 1.27)
-			)
-			(justify left bottom)
-		)
-	)
 	(label "HDMI0_HOTPLUG"
 		(at 106.68 92.71 0)
@@
 		)
 	)
-	(hierarchical_label "GPIO_VREF"
-		(shape input)
-		(at 171.958 140.589 180)
-		(fields_autoplaced yes)
-		(effects
-			(font
-				(size 1.27 1.27)
-			)
-			(justify right)
-		)
-	)
 	(hierarchical_label "ID_SC"
 		(shape input)
@@
 		)
 	)
-	(hierarchical_label "+5v"
-		(shape input)
-		(at 55.88 180.34 180)
-		(fields_autoplaced yes)
-		(effects
-			(font
-				(size 1.27 1.27)
-			)
-			(justify right)
-		)
-	)
 	(hierarchical_label "USB2_P"
 		(shape bidirectional)
@@
 	)
 	(symbol
+		(lib_id "power:VD")
+		(at 168.91 139.7 0)
+		(unit 1)
+		(exclude_from_sim no)
+		(in_bom yes)
+		(on_board yes)
+		(dnp no)
+		(property "Reference" "#PWR0148"
+			(at 168.91 143.51 0)
+			(effects
+				(font
+					(size 1.27 1.27)
+				)
+				(hide yes)
+			)
+		)
+		(property "Value" "GPIO_VREF"
+			(at 175.26 138.684 0)
+			(effects
+				(font
+					(size 1.27 1.27)
+				)
+			)
+		)
+		(property "Footprint" ""
+			(at 168.91 139.7 0)
+			(effects
+				(font
+					(size 1.27 1.27)
+				)
+				(hide yes)
+			)
+		)
+		(property "Datasheet" ""
+			(at 168.91 139.7 0)
+			(effects
+				(font
+					(size 1.27 1.27)
+				)
+				(hide yes)
+			)
+		)
+		(property "Description" "Power symbol creates a global label with name \"VD\""
+			(at 168.91 139.7 0)
+			(effects
+				(font
+					(size 1.27 1.27)
+				)
+				(hide yes)
+			)
+		)
+		(pin "1"
+		)
+		(instances
+			(project "CM4IOv5"
+				(path "/e63e39d7-6ac0-4ffd-8aa3-1841a4541b55/00000000-0000-0000-0000-00005cff70b1"
+					(reference "#PWR0148")
+					(unit 1)
+				)
+			)
+		)
+	)
+	(symbol
 		(lib_id "Device:R")
 		(at 189.23 145.923 0)
@@
 					(unit 1)
 				)
+			)
+		)
+	)
+	(symbol
+		(lib_id "power:+5V")
+		(at 55.88 180.34 0)
+		(unit 1)
+		(exclude_from_sim no)
+		(in_bom yes)
+		(on_board yes)
+		(dnp no)
+		(fields_autoplaced yes)
+		(property "Reference" "#PWR094"
+			(at 55.88 184.15 0)
+			(effects
+				(font
+					(size 1.27 1.27)
+				)
+				(hide yes)
+			)
+		)
+		(property "Value" "+5V"
+			(at 55.88 175.26 0)
+			(effects
+				(font
+					(size 1.27 1.27)
+				)
+			)
+		)
+		(property "Footprint" ""
+			(at 55.88 180.34 0)
+			(effects
+				(font
+					(size 1.27 1.27)
+				)
+				(hide yes)
+			)
+		)
+		(property "Datasheet" ""
+			(at 55.88 180.34 0)
+			(effects
+				(font
+					(size 1.27 1.27)
+				)
+				(hide yes)
+			)
+		)
+		(property "Description" "Power symbol creates a global label with name \"+5V\""
+			(at 55.88 180.34 0)
+			(effects
+				(font
+					(size 1.27 1.27)
+				)
+				(hide yes)
+			)
+		)
+		(pin "1"
+		)
+		(instances
+			(project ""
+				(path "/e63e39d7-6ac0-4ffd-8aa3-1841a4541b55/00000000-0000-0000-0000-00005cff70b1"
+					(reference "#PWR094")
+					(unit 1)
+				)

Commit message: assigned footprints
Parts:
- C80, C81: footprint Capacitor_SMD:C_0402_1005Metric -> Capacitor_SMD:C_0805_2012Metric
- R21, R22: footprint Resistor_SMD:R_0402_1005Metric -> Resistor_SMD:R_0805_2012Metric
Changed lines of the file:
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@@
 			)
 		)
-		(property "Footprint" "Capacitor_SMD:C_0402_1005Metric"
+		(property "Footprint" "Capacitor_SMD:C_0805_2012Metric"
 			(at 61.9252 187.96 0)
 			(effects
@@
 			)
 		)
-		(property "Footprint" "Resistor_SMD:R_0402_1005Metric"
+		(property "Footprint" "Resistor_SMD:R_0805_2012Metric"
 			(at 187.452 145.923 90)
 			(effects
@@
 			)
 		)
-		(property "Footprint" "Resistor_SMD:R_0402_1005Metric"
+		(property "Footprint" "Resistor_SMD:R_0805_2012Metric"
 			(at 179.832 145.923 90)
 			(effects
@@
 			)
 		)
-		(property "Footprint" "Capacitor_SMD:C_0402_1005Metric"
+		(property "Footprint" "Capacitor_SMD:C_0805_2012Metric"
 			(at 94.9452 187.96 0)
 			(effects
