File: Connectors.kicad_sch (KiCad schematic)
At the start: 5 parts

Commit message: stuff
Parts:
- added TP15, TP16: TestPoint, symbol Connector:TestPoint
Connections:
- new net A: TP15.1
- new net B: TP16.1
Changed lines of the file:
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@@
+	(wire
+		(pts
+			(xy 44.45 63.5) (xy 50.8 63.5)
+		)
+		(stroke
+			(width 0)
+			(type default)
+		)
+	)
 	(wire
 		(pts
@@
 	(wire
 		(pts
-			(xy 44.45 44.45) (xy 50.8 44.45)
+			(xy 44.45 69.85) (xy 50.8 69.85)
 		)
 		(stroke
@@
 		)
 	)
+	(wire
+		(pts
+			(xy 44.45 44.45) (xy 50.8 44.45)
+		)
+		(stroke
+			(width 0)
+			(type default)
+		)
+	)
 	(label "SCL"
 		(at 44.45 50.8 0)
@@
 		)
 	)
+	(label "A"
+		(at 46.99 63.5 0)
+		(fields_autoplaced yes)
+		(effects
+			(font
+				(size 1.27 1.27)
+			)
+			(justify left bottom)
+		)
+	)
 	(label "LEAK"
 		(at 44.45 57.15 0)
@@
 			)
 			(justify left bottom)
+		)
+	)
+	(label "B"
+		(at 44.45 69.85 0)
+		(fields_autoplaced yes)
+		(effects
+			(font
+				(size 1.27 1.27)
+			)
+			(justify left bottom)
+		)
+	)
+	(hierarchical_label "A"
+		(shape input)
+		(at 44.45 63.5 180)
+		(fields_autoplaced yes)
+		(effects
+			(font
+				(size 1.27 1.27)
+			)
+			(justify right)
 		)
 	)
@@
 		)
 	)
+	(hierarchical_label "B"
+		(shape input)
+		(at 44.45 69.85 180)
+		(fields_autoplaced yes)
+		(effects
+			(font
+				(size 1.27 1.27)
+			)
+			(justify right)
+		)
+	)
 	(hierarchical_label "LEAK"
 		(shape input)
@@
 			)
 			(justify right)
+		)
+	)
+	(symbol
+		(lib_id "Connector:TestPoint")
+		(at 50.8 69.85 270)
+		(unit 1)
+		(exclude_from_sim no)
+		(in_bom yes)
+		(on_board yes)
+		(dnp no)
+		(fields_autoplaced yes)
+		(property "Reference" "TP16"
+			(at 55.88 68.5799 90)
+			(effects
+				(font
+					(size 1.27 1.27)
+				)
+				(justify left)
+			)
+		)
+		(property "Value" "TestPoint"
+			(at 55.88 71.1199 90)
+			(effects
+				(font
+					(size 1.27 1.27)
+				)
+				(justify left)
+			)
+		)
+		(property "Footprint" ""
+			(at 50.8 74.93 0)
+			(effects
+				(font
+					(size 1.27 1.27)
+				)
+				(hide yes)
+			)
+		)
+		(property "Datasheet" "~"
+			(at 50.8 74.93 0)
+			(effects
+				(font
+					(size 1.27 1.27)
+				)
+				(hide yes)
+			)
+		)
+		(property "Description" "test point"
+			(at 50.8 69.85 0)
+			(effects
+				(font
+					(size 1.27 1.27)
+				)
+				(hide yes)
+			)
+		)
+		(pin "1"
+		)
+		(instances
+			(project ""
+				(path "/e63e39d7-6ac0-4ffd-8aa3-1841a4541b55/75579089-7949-4303-bf9d-35e30a6c418a"
+					(reference "TP16")
+					(unit 1)
+				)
+			)
 		)
 	)
@@
 					(unit 1)
 				)
+			)
+		)
+	)
+	(symbol
+		(lib_id "Connector:TestPoint")
+		(at 50.8 63.5 270)
+		(unit 1)
+		(exclude_from_sim no)
+		(in_bom yes)
+		(on_board yes)
+		(dnp no)
+		(fields_autoplaced yes)
+		(property "Reference" "TP15"
+			(at 55.88 62.2299 90)
+			(effects
+				(font
+					(size 1.27 1.27)
+				)
+				(justify left)
+			)
+		)
+		(property "Value" "TestPoint"
+			(at 55.88 64.7699 90)
+			(effects
+				(font
+					(size 1.27 1.27)
+				)
+				(justify left)
+			)
+		)
+		(property "Footprint" ""
+			(at 50.8 68.58 0)
+			(effects
+				(font
+					(size 1.27 1.27)
+				)
+				(hide yes)
+			)
+		)
+		(property "Datasheet" "~"
+			(at 50.8 68.58 0)
+			(effects
+				(font
+					(size 1.27 1.27)
+				)
+				(hide yes)
+			)
+		)
+		(property "Description" "test point"
+			(at 50.8 63.5 0)
+			(effects
+				(font
+					(size 1.27 1.27)
+				)
+				(hide yes)
+			)
+		)
+		(pin "1"
+		)
+		(instances
+			(project ""
+				(path "/e63e39d7-6ac0-4ffd-8aa3-1841a4541b55/75579089-7949-4303-bf9d-35e30a6c418a"
+					(reference "TP15")
+					(unit 1)
+				)

Commit message: stuff
Connections:
- net LEAK renamed Leak
Changed lines of the file:
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@@
 		)
 	)
-	(hierarchical_label "LEAK"
+	(hierarchical_label "Leak"
 		(shape input)
 		(at 44.45 57.15 180)

Commit message: stuff
Changed lines of the file:
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@@
-		)
-	)
-	(label "LEAK"
-		(at 44.45 57.15 0)
-		(fields_autoplaced yes)
-		(effects
-			(font
-				(size 1.27 1.27)
-			)
-			(justify left bottom)
 		)
 	)

Commit message: assigned footprints
Parts:
- TP10, TP11, TP12, TP13, TP14, TP15, TP16: footprint (none) -> TestPoint:TestPoint_Pad_2.0x2.0mm
Changed lines of the file:
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@@
 			)
 		)
-		(property "Footprint" ""
+		(property "Footprint" "TestPoint:TestPoint_Pad_2.0x2.0mm"
 			(at 50.8 74.93 0)
 			(effects
@@
 			)
 		)
-		(property "Footprint" ""
+		(property "Footprint" "TestPoint:TestPoint_Pad_2.0x2.0mm"
 			(at 50.8 49.53 0)
 			(effects
@@
 			)
 		)
-		(property "Footprint" ""
+		(property "Footprint" "TestPoint:TestPoint_Pad_2.0x2.0mm"
 			(at 50.8 43.18 0)
 			(effects
@@
 			)
 		)
-		(property "Footprint" ""
+		(property "Footprint" "TestPoint:TestPoint_Pad_2.0x2.0mm"
 			(at 50.8 55.88 0)
 			(effects
@@
 			)
 		)
-		(property "Footprint" ""
+		(property "Footprint" "TestPoint:TestPoint_Pad_2.0x2.0mm"
 			(at 50.8 36.83 0)
 			(effects
@@
 			)
 		)
-		(property "Footprint" ""
+		(property "Footprint" "TestPoint:TestPoint_Pad_2.0x2.0mm"
 			(at 50.8 62.23 0)
 			(effects
@@
 			)
 		)
-		(property "Footprint" ""
+		(property "Footprint" "TestPoint:TestPoint_Pad_2.0x2.0mm"
 			(at 50.8 68.58 0)
 			(effects

Commit message: stuff
Parts:
- removed TP10, TP11, TP12, TP13, TP14, TP15, TP16: TestPoint, TestPoint:TestPoint_Pad_2.0x2.0mm, symbol Connector:TestPoint
- added J13, J21, J24: Conn_01x02, Connector_PinHeader_2.54mm:PinHeader_1x02_P2.54mm_Vertical, symbol Connector_Generic:Conn_01x02
- added J25: Conn_01x01, Connector_PinHeader_2.54mm:PinHeader_1x01_P2.54mm_Vertical, symbol Connector_Generic:Conn_01x01
Connections:
- net A: now also J24.1 (Pin_1)
- net B: now also J24.2 (Pin_2)
- net Leak: now also J25.1 (Pin_1)
- net RX: now also J13.2 (Pin_2)
- net SCL: now also J21.2 (Pin_2)
- net SDA: now also J21.1 (Pin_1)
- net TX: now also J13.1 (Pin_1)

Commit message: stuff
Parts:
- added J27, J28: DF13-4P-1.25DSA25, DF13_4P_1_25DSA_25:CONN4_DF13-4P_HIR, symbol DF13_4P_1_25DSA_25:DF13-4P-1.25DSA25
- added J29, J31: BM04B-GHS-TBT, BM04B_GHS_TBT:CONN_BM04B-GHS-TBT_JST, symbol BM04B_GHS_TBT:BM04B-GHS-TBT
- added J30, J32: Conn_01x02, Connector_PinHeader_2.54mm:PinHeader_1x02_P2.54mm_Vertical, symbol Connector_Generic:Conn_01x02
Connections:
- net SCL: now also J27.2, J28.2, J29.3, J31.3
- net SDA: now also J27.3, J28.3, J29.4, J31.4
- new net +3.3V: J27.1, J28.1, J29.2, J30.1 (Pin_1), J31.2
- new net +5V: J32.1 (Pin_1)
- new net GND: J27.4, J28.4, J29.1, J30.2 (Pin_2), J31.1, J32.2 (Pin_2)
Other:
- note added: "Depth Sensor Connectors"
- note added: "I2C Connectors"
- note added: "Power Breakouts"
- note added: "Signal Breakouts"
- moved on the sheet: J13, J21, J24, J25

Commit message: stuff
Parts:
- added J33: B3B-XH-A, B3B_XH_A:CONN_B3B-XH-A_JST, symbol B3B_XH_A:B3B-XH-A
Connections:
- net +5V: now also J33.2
- net GND: now also J33.1
- new net Fan: J33.3
Other:
- note added: "Fan Header"

Commit message: stuff
Parts:
- added J8: BM04B-GHS-TBT, BM04B_GHS_TBT:CONN_BM04B-GHS-TBT_JST, symbol BM04B_GHS_TBT:BM04B-GHS-TBT
Connections:
- net +3.3V: now also J8.2
- net GND: now also J8.1
- net SCL: now also J8.3
- net SDA: now also J8.4
