File: Connectors.kicad_sch (KiCad schematic)
At the start: 12 parts, among them J13 Conn_01x02, J21 Conn_01x02, J24 Conn_01x02, J25 Conn_01x01, J27 DF13-4P-1.25DSA25, J28 DF13-4P-1.25DSA25, J29 BM04B-GHS-TBT, J30 Conn_01x02, J31 BM04B-GHS-TBT, J32 Conn_01x02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

Commit message: STUFF
Connections:
- net A renamed A+
- net B renamed A-
Changed lines of the file:
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@@
+	(wire
+		(pts
+			(xy 34.29 81.28) (xy 40.64 81.28)
+		)
+		(stroke
+			(width 0)
+			(type default)
+		)
+	)
 	(wire
 		(pts
@@
 		(pts
 			(xy 113.03 39.37) (xy 127 39.37)
-		)
-		(stroke
-			(width 0)
-			(type default)
-		)
-	)
-	(wire
-		(pts
-			(xy 34.29 81.28) (xy 40.64 81.28)
 		)
 		(stroke
@@
 		)
 	)
-	(label "A"
+	(label "A+"
 		(at 34.29 78.74 0)
 		(fields_autoplaced yes)
@@
 		)
 	)
-	(label "B"
-		(at 34.29 81.28 0)
-		(fields_autoplaced yes)
-		(effects
-			(font
-				(size 1.27 1.27)
-			)
-			(justify left bottom)
-		)
-	)
-	(hierarchical_label "A"
+	(hierarchical_label "A+"
 		(shape input)
 		(at 34.29 78.74 180)
@@
 		)
 	)
-	(hierarchical_label "B"
+	(hierarchical_label "A-"
 		(shape input)
 		(at 34.29 81.28 180)
