File: CM4IOv5.kicad_pcb (KiCad board)
At the start: 2 copper layers, 9.3 x 6.9 mm, 167 parts, among them J1 Conn_01x03, J10 482040001, J11 430450212, J12 THD-02-R, J13 302-S101, J15 430450612, J16 SM02B-GHS-TB, J17 SM02B-GHS-TB, J18 SM02B-GHS-TB, J19 SM02B-GHS-TB, J2 Conn_02x07_Odd_Even, J22 430450212, J23 UJC-HP-L-G-5-MSMT-TR, J26 690-019-298-412, J3 Conn_01x03, J4 482040001, J5 482040001, J6 482040001, J7 Micro_SD_Card_Det, J8 THD-20-R, J9 THD-02-R, Q2 2N7002, SW1 1301.9314.24, T1 DA2304-ALD, U1 TPD4EUSB30, U10 FE1.1s, U11 24LC02B-I_SN, U12 TPS2117DRLR, U14 INA260AIPW, U15 BME280, U16 BNO085, U17 BME280, U18 RT9742GGJ5, U2 TPD4EUSB30, U20 AZ1117IH-3.3TRG1, U22 PCA9685PW_118, U25 RT9742SNGV, U3 MagJack-A70-112-331N126, U4 LP2985A-50DBVR, U5 74LVC1G07SE-7, U6 ISO3086TDW, U7 BNO085, U8 MAX485CSA_T, U9 74LVC1G07SE-7, Y3 ABLS-12.000MHZ-B2-T

Commit message: stuff
Parts:
- added C10: 10n, Capacitor_SMD:C_0805_2012Metric, F.Cu at (10.3, -65.4)
- added C11: 1u, Capacitor_SMD:C_0805_2012Metric, F.Cu at (10.3, -62.4)
- added C19: 10u, Capacitor_SMD:C_0805_2012Metric, F.Cu at (14.8, -68.4)
- added C21: .1u, Capacitor_SMD:C_0805_2012Metric, F.Cu at (14.8, -65.4)
- added C24: 10u, Capacitor_SMD:C_0805_2012Metric, F.Cu at (14.8, -62.4)
- added C25: 10n, Capacitor_SMD:C_0805_2012Metric, F.Cu at (19.2, -68.4)
- added C26: 1u, Capacitor_SMD:C_0805_2012Metric, F.Cu at (19.2, -65.4)
- added C27: 10u, Capacitor_SMD:C_0805_2012Metric, F.Cu at (19.2, -62.4)
- added C9: .1u, Capacitor_SMD:C_0805_2012Metric, F.Cu at (10.3, -68.4)
- added FB1: FerriteBead, CM4IO:L_Bourns_SRN6045TA, F.Cu at (4.08, -80.5)
- added FB2: FerriteBead, CM4IO:L_Bourns_SRN6045TA, F.Cu at (4.08, -73.0)
- added FB3: FerriteBead, CM4IO:L_Bourns_SRN6045TA, F.Cu at (4.08, -65.4)
- added FB4: FerriteBead, CM4IO:L_Bourns_SRN6045TA, F.Cu at (4.08, -57.9)
- added FB6: FerriteBead, CM4IO:L_Bourns_SRN6045TA, F.Cu at (4.08, -50.3)
- added J13: Conn_01x02, Connector_PinHeader_2.54mm:PinHeader_1x02_P2.54mm_Vertical, F.Cu at (26.2, -65.2)
- added J14: DF11-10DP-2DSA24, DF11_10DP_2DSA_24:CON10_2X5_UF_DF11_HIR, F.Cu at (34.7, -79.9)
- added J20: DF11-10DP-2DSA24, DF11_10DP_2DSA_24:CON10_2X5_UF_DF11_HIR, F.Cu at (34.7, -72.6)
- added J21: Conn_01x02, Connector_PinHeader_2.54mm:PinHeader_1x02_P2.54mm_Vertical, F.Cu at (30.8, -65.2)
- added J24: Conn_01x02, Connector_PinHeader_2.54mm:PinHeader_1x02_P2.54mm_Vertical, F.Cu at (35.5, -65.2)
- added J25: Conn_01x01, Connector_PinHeader_2.54mm:PinHeader_1x01_P2.54mm_Vertical, F.Cu at (26.2, -58.0)
- added R46: 5k, Resistor_SMD:R_0805_2012Metric, F.Cu at (10.3, -59.4)
- added R49: 120, Resistor_SMD:R_0805_2012Metric, F.Cu at (10.3, -56.4)
- added U6: ISOW1432BDFMR, ISOW1432BDFMR:SOIC127P1030X355-20N, F.Cu at (15.4, -77.1)
Connections:
- Module1 pad 34: /CM4_GPIO ( Ethernet, GPIO, SDCARD)/GPIO5 -> /CM4_GPIO ( Ethernet, GPIO, SDCARD)/RX_TB
- Module1 pad 44: /CM4_GPIO ( Ethernet, GPIO, SDCARD)/GPIO10 -> /ISO_FLT
- Module1 pad 54: /CM4_GPIO ( Ethernet, GPIO, SDCARD)/GPIO4 -> /CM4_GPIO ( Ethernet, GPIO, SDCARD)/TX_TB
- R44 pad 2: +5V -> VCC2
- R45 pad 2: GND -> GND2

Commit message: stuff
Parts:
- added J27: DF13-4P-1.25DSA25, DF13_4P_1_25DSA_25:CONN4_DF13-4P_HIR, F.Cu at (21.3, -31.5)
- added J28: DF13-4P-1.25DSA25, DF13_4P_1_25DSA_25:CONN4_DF13-4P_HIR, F.Cu at (21.3, -25.3)
- added J29: BM04B-GHS-TBT, BM04B_GHS_TBT:CONN_BM04B-GHS-TBT_JST, F.Cu at (11.9, -29.5)
- added J30: Conn_01x02, Connector_PinHeader_2.54mm:PinHeader_1x02_P2.54mm_Vertical, F.Cu at (20.2, -19.8)
- added J31: BM04B-GHS-TBT, BM04B_GHS_TBT:CONN_BM04B-GHS-TBT_JST, F.Cu at (11.9, -20.9)
- added J32: Conn_01x02, Connector_PinHeader_2.54mm:PinHeader_1x02_P2.54mm_Vertical, F.Cu at (24.9, -19.8)
Other:
- board size 9.3 x 6.9 mm -> 85 x 56 mm

Commit message: stuff
Parts:
- added J33: B3B-XH-A, B3B_XH_A:CONN_B3B-XH-A_JST, F.Cu at (18.5, -4.00)
- moved Module1 341.9 mm to (168.8, 116.6), turned to 90 degrees
Connections:
- Module1 pad 37: /CM4_GPIO ( Ethernet, GPIO, SDCARD)/GPIO7 -> /Fan

Commit message: stuff
Parts:
- moved J10 273.0 mm to (152.5, 71.2)
- moved J6 270.3 mm to (139.5, 71.2)
- moved J5 267.6 mm to (126.5, 71.2)
- moved J4 265.8 mm to (114.5, 71.2)
- moved J13 28.8 mm to (5.84, -100.0)
- moved Module1 25.5 mm to (152.5, 97.0), turned to 180 degrees
Other:
- board size 85 x 56 mm -> 56 x 85 mm

Commit message: stuff
Parts:
- removed the J13 at (5.84, -100.0)
- removed J8: THD-20-R, Connector_PinHeader_2.54mm:PinHeader_2x20_P2.54mm_Vertical
- added J34: Conn_01x01, Connector_PinHeader_2.54mm:PinHeader_1x01_P2.54mm_Vertical, F.Cu at (-23.6, -15.4)
- added J35: Conn_01x01, Connector_PinHeader_2.54mm:PinHeader_1x01_P2.54mm_Vertical, F.Cu at (-16.6, -9.29)
- added J36: Conn_01x01, Connector_PinHeader_2.54mm:PinHeader_1x01_P2.54mm_Vertical, F.Cu at (-16.6, -4.63)
- added J37: Conn_01x01, Connector_PinHeader_2.54mm:PinHeader_1x01_P2.54mm_Vertical, F.Cu at (-12.0, -13.9)
- added J38: Conn_01x01, Connector_PinHeader_2.54mm:PinHeader_1x01_P2.54mm_Vertical, F.Cu at (-12.0, -9.29)
- added J39: Conn_01x01, Connector_PinHeader_2.54mm:PinHeader_1x01_P2.54mm_Vertical, F.Cu at (-12.0, -4.63)
- added J40: Conn_01x01, Connector_PinHeader_2.54mm:PinHeader_1x01_P2.54mm_Vertical, F.Cu at (-7.34, -13.9)
- added J41: Conn_01x01, Connector_PinHeader_2.54mm:PinHeader_1x01_P2.54mm_Vertical, F.Cu at (-7.34, -9.29)
- added J42: Conn_01x01, Connector_PinHeader_2.54mm:PinHeader_1x01_P2.54mm_Vertical, F.Cu at (-7.34, -4.63)
- added REF**: MountingHole_2.7mm_M2.5_ISO14580, MountingHole:MountingHole_2.7mm_M2.5_ISO14580, F.Cu at (151.5, 65.0)
- added REF**: MountingHole_2.7mm_M2.5_ISO14580, MountingHole:MountingHole_2.7mm_M2.5_ISO14580, F.Cu at (200.5, 65.0)
- added REF**: MountingHole_2.7mm_M2.5_ISO14580, MountingHole:MountingHole_2.7mm_M2.5_ISO14580, F.Cu at (151.5, 123.0)
- added REF**: MountingHole_2.7mm_M2.5_ISO14580, MountingHole:MountingHole_2.7mm_M2.5_ISO14580, F.Cu at (200.5, 123.0)
- J15: footprint RS485-Header:CON_430450212_MOL -> 430450612:CON_430450612_MOL
- moved U3 324.0 mm to (191.9, 110.3), turned to -90 degrees
- moved U10 309.0 mm to (150.8, 138.0), turned to 90 degrees
- moved Y3 305.2 mm to (150.6, 129.2)
- moved J11 303.2 mm to (190.7, 91.2), turned to 90 degrees
- moved J26 300.0 mm to (164.6, 65.1)
- moved J22 287.8 mm to (190.7, 79.9), turned to 90 degrees
- moved J2 286.5 mm to (111.3, 126.8)
- moved J15 284.9 mm to (191.0, 129.2)
- moved J23 271.3 mm to (189.2, 138.5), turned to 180 degrees
- moved SW1 268.6 mm to (186.0, 67.8)
- moved J7 242.8 mm to (135.2, 69.4)
- moved J14 236.8 mm to (200.4, 89.2), turned to 90 degrees
- moved J20 221.4 mm to (200.2, 74.4), turned to 90 degrees
- moved U6 128.0 mm to (84.2, 30.8)
- moved U14 105.8 mm to (28.4, 85.8)
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Other:
- board size 56 x 85 mm -> 107.5 x 85 mm

Commit message: stuff
Parts:
- removed the REF** at (151.5, 65.0)
- removed the REF** at (200.5, 65.0)
- removed the REF** at (151.5, 123.0)
- removed the REF** at (200.5, 123.0)
- removed T1: DA2304-ALD, DA2304-ALD:XFMR_DA2304-ALD
- removed TP10, TP11, TP12, TP13, TP14, TP15, TP16: TestPoint, TestPoint:TestPoint_Pad_2.0x2.0mm
- removed the U6 at (11.8, 28.8)
- added J8: BM04B-GHS-TBT, BM04B_GHS_TBT:CONN_BM04B-GHS-TBT_JST, F.Cu at (222.2, 140.8)
- added REF**: MountingHole_2.7mm_M2.5_ISO14580, MountingHole:MountingHole_2.7mm_M2.5_ISO14580, F.Cu at (254.4, 63.0)
- added REF**: MountingHole_2.7mm_M2.5_ISO14580, MountingHole:MountingHole_2.7mm_M2.5_ISO14580, F.Cu at (205.4, 63.0)
- added REF**: MountingHole_2.7mm_M2.5_ISO14580, MountingHole:MountingHole_2.7mm_M2.5_ISO14580, F.Cu at (-73.3, 167.2)
- added REF**: MountingHole_2.7mm_M2.5_ISO14580, MountingHole:MountingHole_2.7mm_M2.5_ISO14580, F.Cu at (-73.3, 109.2)
- added REF**: MountingHole_2.7mm_M2.5_ISO14580, MountingHole:MountingHole_2.7mm_M2.5_ISO14580, F.Cu at (-24.3, 109.2)
- added REF**: MountingHole_2.7mm_M2.5_ISO14580, MountingHole:MountingHole_2.7mm_M2.5_ISO14580, F.Cu at (254.4, 121.0)
- added REF**: MountingHole_2.7mm_M2.5_ISO14580, MountingHole:MountingHole_2.7mm_M2.5_ISO14580, F.Cu at (205.4, 121.0)
- added REF**: MountingHole_2.7mm_M2.5_ISO14580, MountingHole:MountingHole_2.7mm_M2.5_ISO14580, F.Cu at (-24.3, 167.2)
- JP1, JP10, JP2, JP3, JP4, JP7, JP8, JP9: footprint Jumper:SolderJumper-3_P1.3mm_Open_RoundedPad1.0x1.5mm -> Jumper:SolderJumper-2_P1.3mm_Open_RoundedPad1.0x1.5mm
- Module1: moved to B.Cu
- moved J34 306.2 mm to (249.0, 124.0), turned to 90 degrees
- moved J36 293.3 mm to (249.0, 119.8)
- moved J40 288.2 mm to (254.8, 106.0)
- moved J41 288.2 mm to (254.8, 110.6)
- moved J42 288.2 mm to (254.8, 115.2)
- moved J37 255.2 mm to (191.8, 139.8), turned to 90 degrees
- moved J38 249.0 mm to (187.5, 139.8), turned to 180 degrees
- moved J35 242.2 mm to (174.2, 139.8), turned to 90 degrees
- moved J3 239.8 mm to (249.8, 94.7)
- moved J1 239.7 mm to (249.8, 83.7)
- moved J39 239.2 mm to (178.8, 139.8), turned to 90 degrees
- moved TP2 234.0 mm to (255.5, 79.5)
- moved TP4 233.8 mm to (255.4, 83.2)
- moved TP3 231.4 mm to (255.5, 68.5)
- moved TP5 231.2 mm to (255.5, 72.0)
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Routing:
- net Net-(U6-VIO): track 0.00 -> 17.6 mm
- net +3.3V: track 0.00 -> 16.7 mm
- net Net-(U6-VISOOUT): track 0.00 -> 16.0 mm
- net Net-(U6-GND2): track 0.00 -> 15.6 mm
- net /RS485/TB_A: track 0.00 -> 14.3 mm
- net Net-(U6-GND1): track 0.00 -> 11.9 mm
- net Net-(U6-VDD): track 0.00 -> 10.7 mm
- net /ISO_FLT: track 0.00 -> 8.13 mm
- net /Sensors/SA0: track 0.00 -> 7.85 mm
- net GND: track 0.00 -> 7.85 mm
- net GND2: track 0.00 -> 7.49 mm
- net /USBhub/LED1/EESCL: track 0.00 -> 7.37 mm
- net VCC2: track 0.00 -> 7.22 mm
- net +5V: track 0.00 -> 7.13 mm
- net /Sensors/SA0_1: track 0.00 -> 6.90 mm
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Other:
- board size 107.5 x 85 mm -> 334.7 x 131.2 mm

Commit message: stuff
Parts:
- C10, C11, C19, C21, C24, C25, C26, C27, C9, FB1, FB2, FB3, FB4, FB6, R46, R49, U6: moved to B.Cu
- Module1: moved to F.Cu
- moved U22 279.9 mm to (222.2, 135.2)
- moved R25 221.4 mm to (233.0, 112.0), turned to 0 degrees
- moved R24 219.6 mm to (240.7, 113.5), turned to 0 degrees
- moved Q2 218.2 mm to (236.8, 111.0), turned to 90 degrees
- moved D18 217.7 mm to (245.0, 113.5), turned to 180 degrees
- moved R26 217.2 mm to (233.8, 109.1), turned to -90 degrees
- moved R23 216.2 mm to (240.8, 111.0), turned to 0 degrees
- moved C7 209.3 mm to (82.5, 104.4)
- moved U8 209.3 mm to (76.0, 106.4)
- moved U9 180.7 mm to (183.8, 74.7)
- moved U4 163.8 mm to (167.0, -21.8)
- moved R38 162.7 mm to (188.8, 67.2), turned to 90 degrees
- moved R16 155.4 mm to (180.2, 71.5), turned to -90 degrees
- moved R15 153.4 mm to (177.8, 71.5), turned to -90 degrees
- moved D11 153.4 mm to (188.8, 63.2), turned to -90 degrees
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Connections:
- J14 pad 10: /PWM_Generatrion/5 -> /PWM_Generatrion/4
- J14 pad 5: /PWM_Generatrion/0 -> /PWM_Generatrion/1
- J14 pad 6: /PWM_Generatrion/1 -> /PWM_Generatrion/0
- J14 pad 7: /PWM_Generatrion/2 -> /PWM_Generatrion/3
- J14 pad 8: /PWM_Generatrion/3 -> /PWM_Generatrion/2
- J14 pad 9: /PWM_Generatrion/4 -> /PWM_Generatrion/5
- J20 pad 1: /PWM_Generatrion/6 -> /PWM_Generatrion/7
- J20 pad 2: /PWM_Generatrion/7 -> /PWM_Generatrion/6
- J20 pad 3: /PWM_Generatrion/8 -> /PWM_Generatrion/9
- J20 pad 4: /PWM_Generatrion/9 -> /PWM_Generatrion/8
Routing:
- net +3.3V: track 16.7 -> 148.9 mm, vias 0 -> 7
- net /SDA: track 0.00 -> 117.3 mm, vias 0 -> 6
- net /SCL: track 0.00 -> 112.4 mm, vias 0 -> 9
- net +5V: track 7.13 -> 101.9 mm, vias 0 -> 5
- net /Sensors/Probe: track 0.00 -> 49.3 mm
- net /CM4_GPIO ( Ethernet, GPIO, SDCARD)/RUN_PG: track 0.00 -> 40.9 mm
- net /CM4_GPIO ( Ethernet, GPIO, SDCARD)/SYNC_OUT: track 0.00 -> 26.9 mm, vias 0 -> 1
- net /Fan: track 0.00 -> 24.8 mm, vias 0 -> 2
- net /CM4_GPIO ( Ethernet, GPIO, SDCARD)/GLOBAL_EN: track 0.00 -> 23.7 mm, vias 0 -> 2
- net /CM4_GPIO ( Ethernet, GPIO, SDCARD)/AIN0: track 0.00 -> 21.6 mm
- net /PWM_Generatrion/6: track 0.00 -> 21.0 mm
- net /CM4_GPIO ( Ethernet, GPIO, SDCARD)/nRPIBOOT: track 0.00 -> 18.9 mm
- net /CM4_GPIO ( Ethernet, GPIO, SDCARD)/AIN1: track 0.00 -> 18.6 mm, vias 0 -> 2
- net /CM4_GPIO ( Ethernet, GPIO, SDCARD)/EEPROM_nWP: track 0.00 -> 17.9 mm
- net /PWM_Generatrion/7: track 0.00 -> 17.0 mm
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Other:
- outline, holes or cut-outs redrawn

Commit message: stuff
Parts:
- removed J41: Conn_01x01, Connector_PinHeader_2.54mm:PinHeader_1x01_P2.54mm_Vertical
- moved R18 159.4 mm to (167.5, 63.2), turned to 180 degrees
- moved R17 154.8 mm to (161.0, 63.2)
- moved SW1 63.4 mm to (189.5, 124.0)
- moved J7 62.8 mm to (162.1, 72.4)
- moved J25 30.1 mm to (245.2, 109.5)
- moved J11 10.3 mm to (164.4, 89.0)
- moved J22 9.03 mm to (160.6, 99.5)
- moved J24 6.76 mm to (163.5, 108.0)
- moved U9 2.91 mm to (184.0, 71.8)
- moved J21 0.81 mm to (249.2, 123.5), turned to 0 degrees
Routing:
- net /OE_PWM: track 0.00 -> 86.8 mm, vias 0 -> 2
- net /CM4_GPIO ( Ethernet, GPIO, SDCARD)/SD_DAT0: track 0.00 -> 44.6 mm, vias 0 -> 2
- net /CM4_GPIO ( Ethernet, GPIO, SDCARD)/SD_DAT1: track 0.00 -> 43.6 mm, vias 0 -> 2
- net /SDA: track 117.3 -> 148.0 mm
- net /SCL: track 112.4 -> 141.4 mm
- net /Leak: track 5.94 -> 12.6 mm
- net +5V: track 101.9 -> 105.2 mm
- net Net-(J2-Pin_13): track 7.12 -> 4.65 mm
- net Net-(J7-DET_B): track 0.00 -> 2.46 mm
- net Net-(J7-DET_A): track 0.00 -> 2.29 mm
- net /CM4_GPIO ( Ethernet, GPIO, SDCARD)/RUN_PG: track 40.9 -> 39.8 mm
- net +3.3V: track 148.9 -> 149.2 mm, vias 7 -> 9
