File: CM4IOv5.kicad_pcb (KiCad board)
At the start: 2 copper layers, 334.7 x 131.2 mm, 203 parts, among them J1 Conn_01x03, J10 482040001, J11 430450212, J12 THD-02-R, J13 Conn_01x02, J14 DF11-10DP-2DSA24, J15 430450612, J16 SM02B-GHS-TB, J17 SM02B-GHS-TB, J18 SM02B-GHS-TB, J19 SM02B-GHS-TB, J2 Conn_02x07_Odd_Even, J20 DF11-10DP-2DSA24, J21 Conn_01x02, J22 430450212, J23 UJC-HP-L-G-5-MSMT-TR, J24 Conn_01x02, J25 Conn_01x01, J26 690-019-298-412, J27 DF13-4P-1.25DSA25, J28 DF13-4P-1.25DSA25, J29 BM04B-GHS-TBT, J3 Conn_01x03, J30 Conn_01x02, J31 BM04B-GHS-TBT, J32 Conn_01x02, J33 B3B-XH-A, J34 Conn_01x01, J35 Conn_01x01, J36 Conn_01x01, J37 Conn_01x01, J38 Conn_01x01, J39 Conn_01x01, J4 482040001, J40 Conn_01x01, J42 Conn_01x01, J5 482040001, J6 482040001, J7 Micro_SD_Card_Det, J8 BM04B-GHS-TBT, J9 THD-02-R, Q2 2N7002, SW1 1301.9314.24, U1 TPD4EUSB30, U10 FE1.1s, U11 24LC02B-I_SN, U12 TPS2117DRLR, U14 INA260AIPW, U15 BME280, U16 BNO085, U17 BME280, U18 RT9742GGJ5, U2 TPD4EUSB30, U20 AZ1117IH-3.3TRG1, U22 PCA9685PW_118, U25 RT9742SNGV, U3 MagJack-A70-112-331N126, U4 LP2985A-50DBVR, U5 74LVC1G07SE-7, U6 ISOW1432BDFMR, U7 BNO085, U8 MAX485CSA_T, U9 74LVC1G07SE-7, Y3 ABLS-12.000MHZ-B2-T

Commit message: stuff
Parts:
- moved J40 34.0 mm to (251.2, 139.8)
- moved C10 30.9 mm to (199.0, 14.2)
- moved C11 30.9 mm to (201.2, 14.2)
- moved C19 30.9 mm to (203.7, 14.2)
- moved C21 30.9 mm to (182.2, 9.54)
- moved C24 30.9 mm to (179.5, 9.54)
- moved C25 30.9 mm to (176.5, 13.8)
- moved C26 30.9 mm to (179.5, 13.8)
- moved C27 30.9 mm to (182.5, 13.8)
- moved C9 30.9 mm to (200.0, 4.24)
- moved FB1 30.9 mm to (208.7, 13.3)
- moved FB2 30.9 mm to (203.7, 20.8)
- moved FB3 30.9 mm to (171.2, 9.71)
- moved FB4 30.9 mm to (171.2, 17.3)
- moved FB6 30.9 mm to (207.7, 3.29)
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
Commit message: stuff
Parts:
- removed the C10 at (-71.5, -23.0)
- removed the C10 at (199.0, 14.2)
- removed the C11 at (-71.5, -20.0)
- removed the C11 at (201.2, 14.2)
- removed the C19 at (-71.5, -17.0)
- removed the C19 at (203.7, 14.2)
- removed the C21 at (-71.5, -11.0)
- removed the C21 at (182.2, 9.54)
- removed the C9 at (-71.5, -26.0)
- removed the C9 at (200.0, 4.24)
- removed D12, D17: MBR0520LT, Diode_SMD:D_SOD-123
- removed the REF** at (254.4, 63.0)
- removed the REF** at (205.4, 63.0)
- removed the REF** at (-73.3, 167.2)
- removed the REF** at (-73.3, 109.2)
- removed the REF** at (-24.3, 109.2)
- removed the REF** at (254.4, 121.0)
- removed the REF** at (205.4, 121.0)
- removed the REF** at (-24.3, 167.2)
- added C10: 10n, Capacitor_SMD:C_0805_2012Metric, B.Cu at (135.1, 141.7)
- added C11: 1u, Capacitor_SMD:C_0805_2012Metric, B.Cu at (138.5, 141.6)
- added C19: 10u, Capacitor_SMD:C_0805_2012Metric, B.Cu at (141.8, 141.6)
- added C21: .1u, Capacitor_SMD:C_0805_2012Metric, B.Cu at (117.4, 135.7)
- added C9: .1u, Capacitor_SMD:C_0805_2012Metric, B.Cu at (135.5, 128.7)
- added REF**: MountingHole_2.7mm_M2.5_ISO14580, MountingHole:MountingHole_2.7mm_M2.5_ISO14580, F.Cu at (150.7, 72.6)
- added REF**: MountingHole_2.7mm_M2.5_ISO14580, MountingHole:MountingHole_2.7mm_M2.5_ISO14580, F.Cu at (200.0, 130.0)
- added REF**: MountingHole_2.7mm_M2.5_ISO14580, MountingHole:MountingHole_2.7mm_M2.5_ISO14580, F.Cu at (199.7, 72.6)
- added REF**: MountingHole_2.7mm_M2.5_ISO14580, MountingHole:MountingHole_2.7mm_M2.5_ISO14580, F.Cu at (151.0, 130.0)
- C13, C14, C15, C16, C17, C18, C20, C22, C23, C3, C4, C6, C8, D10, D18, D4, D8, D9, J23, JP10, JP7, JP8, JP9, Q2, R11, R12, R13, R14, R15, R16, R19, R20, R23, R24, R25, R26, R27, R28, R33, R34, R35, R36, R37, R47, R48, R6, R7, R9, U10, U11, U12, U14, U15, U16, U17, U20, U4, U7, Y3: moved to B.Cu
- TP2, TP3, TP4, TP5, TP6, TP7, TP8, TP9: footprint TestPoint:TestPoint_Pad_2.0x2.0mm -> TestPoint:TestPoint_Plated_Hole_D3.0mm
- moved J35 397.5 mm to (-131.2, 47.1), turned to 0 degrees
- moved J34 396.2 mm to (-131.2, 42.4), turned to 0 degrees
- moved J36 390.7 mm to (-126.5, 42.4)
- moved J39 387.4 mm to (-121.9, 47.1), turned to 0 degrees
- moved TP5 387.0 mm to (-131.5, 75.4)
- moved TP3 387.0 mm to (-131.5, 71.3)
- moved J37 384.0 mm to (-126.5, 47.1), turned to 0 degrees
- moved J38 381.5 mm to (-121.9, 42.4), turned to 0 degrees
- moved J40 381.1 mm to (-117.2, 42.4)
- moved J42 378.2 mm to (-117.2, 47.1)
- moved J3 366.8 mm to (-119.3, 60.6)
- moved J2 336.2 mm to (-131.2, 51.7), turned to 0 degrees
- moved J1 322.5 mm to (-124.0, 60.6), turned to 0 degrees
- moved U9 301.0 mm to (-117.0, 73.9)
- moved R18 282.9 mm to (-115.3, 53.8), turned to 0 degrees
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Routing:
- net /SDA: track 148.0 -> 0.00 mm, vias 6 -> 0
- net /SCL: track 141.4 -> 0.00 mm, vias 9 -> 0
- net +3.3V: track 149.2 -> 12.2 mm, vias 9 -> 0
- net +5V: track 105.2 -> 2.88 mm, vias 5 -> 0
- net /OE_PWM: track 86.8 -> 0.00 mm, vias 2 -> 0
- net /CM4_GPIO ( Ethernet, GPIO, SDCARD)/SD_DAT0: track 44.6 -> 0.00 mm, vias 2 -> 0
- net /CM4_GPIO ( Ethernet, GPIO, SDCARD)/SD_DAT1: track 43.6 -> 0.00 mm, vias 2 -> 0
- net /CM4_GPIO ( Ethernet, GPIO, SDCARD)/RUN_PG: track 39.8 -> 0.00 mm
- net Mux_PWR_Out: track 0.00 -> 34.9 mm, vias 0 -> 2
- net /CM4_GPIO ( Ethernet, GPIO, SDCARD)/SYNC_OUT: track 26.9 -> 0.00 mm, vias 1 -> 0
- net /Fan: track 24.8 -> 0.00 mm, vias 2 -> 0
- net /USBhub/LED2: track 0.00 -> 24.2 mm
- net /CM4_GPIO ( Ethernet, GPIO, SDCARD)/GLOBAL_EN: track 23.7 -> 0.00 mm, vias 2 -> 0
- net /CM4_GPIO ( Ethernet, GPIO, SDCARD)/AIN0: track 21.6 -> 0.00 mm
- net /Sensors/Probe: track 49.3 -> 29.2 mm
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Other:
- board size 334.7 x 131.2 mm -> 122.8 x 85 mm
- board text added: "Top"

Commit message: stuff
Parts:
- C10, C11, C13, C14, C15, C16, C17, C18, C19, C20, C21, C22, C23, C24, C25, C26, C27, C3, C4, C6, C8, C9, D10, D18, D4, D8, D9, FB1, FB2, FB3, FB4, FB6, J23, JP10, JP7, JP8, JP9, Q2, R11, R12, R13, R14, R15, R16, R19, R20, R23, R24, R25, R26, R27, R28, R33, R34, R35, R36, R37, R46, R47, R48, R49, R6, R7, R9, U10, U11, U12, U14, U15, U16, U17, U20, U4, U6, U7, Y3: moved to F.Cu
- moved FB4 401.4 mm to (163.3, -250.7), turned to 0 degrees
- moved FB3 401.1 mm to (162.2, -263.1)
- moved C27 400.9 mm to (161.2, -256.9)
- moved C26 400.1 mm to (157.8, -256.9)
- moved C20 400.0 mm to (157.2, -267.1)
- moved C21 400.0 mm to (157.0, -262.3)
- moved U4 399.8 mm to (156.1, -271.9)
- moved C24 399.6 mm to (155.0, -262.3)
- moved R49 399.6 mm to (154.9, -267.0)
- moved C25 399.6 mm to (154.9, -256.9)
- moved FB2 398.6 mm to (126.1, -255.2), turned to 0 degrees
- moved U6 398.5 mm to (147.5, -262.6), turned to 0 degrees
- moved FB6 398.1 mm to (132.6, -269.4), turned to 0 degrees
- moved C19 398.1 mm to (132.6, -256.3)
- moved FB1 398.1 mm to (132.6, -262.1)
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Routing:
- net GND: track 0.00 -> 69.1 mm
- net /SDA: track 0.00 -> 57.0 mm
- net /SCL: track 0.00 -> 55.2 mm, vias 0 -> 4
- net /CM4_GPIO ( Ethernet, GPIO, SDCARD)/SD_CMD: track 0.00 -> 49.1 mm, vias 0 -> 2
- net /CM4_GPIO ( Ethernet, GPIO, SDCARD)/IMU_Rst1: track 0.00 -> 36.0 mm, vias 0 -> 2
- net /CM4_GPIO ( Ethernet, GPIO, SDCARD)/Int1: track 0.00 -> 35.8 mm
- net /CM4_GPIO ( Ethernet, GPIO, SDCARD)/SD_DAT1: track 0.00 -> 34.4 mm, vias 0 -> 2
- net /CM4_GPIO ( Ethernet, GPIO, SDCARD)/SD_DAT0: track 0.00 -> 33.9 mm, vias 0 -> 2
- net /CM4_GPIO ( Ethernet, GPIO, SDCARD)/SD_CLK: track 0.00 -> 32.8 mm, vias 0 -> 2
- net /CM4_GPIO ( Ethernet, GPIO, SDCARD)/Boot1: track 2.92 -> 34.9 mm
- net /CM4_GPIO ( Ethernet, GPIO, SDCARD)/SD_DAT3: track 0.00 -> 28.8 mm, vias 0 -> 2
- net /CM4_GPIO ( Ethernet, GPIO, SDCARD)/SD_DAT2: track 0.00 -> 26.3 mm
- net /RE: track 0.00 -> 24.7 mm, vias 0 -> 2
- net /Int: track 0.00 -> 24.4 mm, vias 0 -> 2
- net /DE: track 0.00 -> 23.3 mm, vias 0 -> 2
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Other:
- outline, holes or cut-outs redrawn
- copper layers 2 -> 4

Commit message: stuff
Parts:
- moved J13 320.3 mm to (-6.02, -145.7)
- moved J24 320.3 mm to (3.28, -145.7)
- moved J25 320.3 mm to (5.86, -130.1)
- moved J30 320.3 mm to (10.2, -144.7)
- moved J32 320.3 mm to (14.9, -144.7)
- moved J33 320.3 mm to (11.8, -135.6)
- moved R30 297.1 mm to (5.42, -169.3)
- moved R31 297.1 mm to (10.3, -166.5)
- moved R32 297.1 mm to (10.5, -169.7)
- moved R39 297.1 mm to (5.42, -166.3)
- moved R44 297.1 mm to (5.42, -163.4)
- moved R45 297.1 mm to (5.42, -160.4)
- moved J11 242.0 mm to (-34.8, -193.7)
- moved J22 242.0 mm to (-22.4, -192.5)
- moved U3 216.7 mm to (108.8, -252.4), turned to -90 degrees
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Routing:
- net /CM4_GPIO ( Ethernet, GPIO, SDCARD)/GLOBAL_EN: track 1.50 -> 39.7 mm, vias 0 -> 2
- net /Leak: track 5.55 -> 16.8 mm, vias 0 -> 2
- net /CM4_HighSpeed/HDMI0_SDA: track 1.22 -> 11.3 mm
- net Net-(U6-GND2): track 15.0 -> 19.4 mm
- net /CM4_HighSpeed/HDMI0_SCL: track 1.50 -> 5.76 mm
- net +3.3V: track 26.2 -> 28.7 mm
- net Net-(J7-DET_B): track 0.00 -> 2.21 mm
- net Net-(J7-DET_A): track 0.00 -> 2.13 mm
- net Net-(D18-A): track 1.84 -> 3.87 mm
- net /CM4_HighSpeed/HDMI0_D2_P: track 1.50 -> 0.00 mm
- net /CM4_HighSpeed/HDMI0_D0_P: track 1.50 -> 2.65 mm
- net /CM4_HighSpeed/HDMI0_D2_N: track 1.50 -> 2.60 mm
- net /CM4_HighSpeed/HDMI0_D1_P: track 1.50 -> 2.55 mm
- net /CM4_HighSpeed/HDMI0_D1_N: track 1.50 -> 2.45 mm

Commit message: stuff
Parts:
- moved J34 416.8 mm to (-133.3, 147.6)
- moved J35 416.8 mm to (-133.3, 152.3)
- moved J36 416.8 mm to (-128.7, 147.6)
- moved J37 416.8 mm to (-128.7, 152.3)
- moved J38 416.8 mm to (-124.0, 147.6)
- moved J39 416.8 mm to (-124.0, 152.3)
- moved J40 416.8 mm to (-119.4, 147.6)
- moved J42 416.8 mm to (-119.4, 152.3)
- moved C1 414.5 mm to (-31.3, 204.3)
- moved D2 414.5 mm to (-31.3, 201.3)
- moved D3 405.3 mm to (-76.6, 66.6)
- moved D5 405.3 mm to (-76.3, 98.2)
- moved D6 405.3 mm to (-76.7, 87.3)
- moved D7 405.3 mm to (-76.7, 77.0)
- moved J10 405.3 mm to (-73.7, 104.2)
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Routing:
- net /OE_PWM: track 1.50 -> 55.8 mm, vias 0 -> 4
- net 5v_Ext_Stack: track 14.6 -> 55.6 mm, vias 0 -> 2
- net 1.8v: track 2.64 -> 41.7 mm, vias 0 -> 2
- net /SCL: track 55.2 -> 93.6 mm, vias 4 -> 6
- net /CM4_GPIO ( Ethernet, GPIO, SDCARD)/RUN_PG: track 1.32 -> 36.3 mm, vias 0 -> 2
- net /SDA: track 57.0 -> 91.2 mm, vias 0 -> 2
- net /CM4_GPIO ( Ethernet, GPIO, SDCARD)/nPWR_LED: track 1.50 -> 30.3 mm, vias 0 -> 2
- net /CM4_GPIO ( Ethernet, GPIO, SDCARD)/SD_PWR_ON: track 1.50 -> 30.1 mm
- net /CM4_HighSpeed/HDMI0_HOTPLUG: track 1.22 -> 23.0 mm, vias 0 -> 2
- net Mux_PWR_Out: track 36.1 -> 57.3 mm, vias 2 -> 4
- net Regulator_PWR_Out: track 17.0 -> 38.0 mm
- net USBC_PWR_In: track 24.3 -> 43.8 mm, vias 0 -> 2
- net +5VL: track 0.00 -> 11.7 mm
- net GND2: track 15.6 -> 26.8 mm
- net /CM4_GPIO ( Ethernet, GPIO, SDCARD)/SD_PWR: track 1.80 -> 12.1 mm, vias 0 -> 2
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
Commit message: stuff
Parts:
- moved TP8 269.0 mm to (121.5, 63.8)
- moved TP9 267.3 mm to (121.5, 70.8)
- moved TP4 266.4 mm to (120.9, 83.8)
- moved TP7 259.5 mm to (120.9, 90.4)
- moved TP2 254.5 mm to (121.0, 104.0)
- moved TP6 254.2 mm to (121.1, 97.3)
- moved TP3 233.4 mm to (121.2, 77.3)
- moved TP5 222.8 mm to (120.8, 110.5)
- moved J15 158.3 mm to (125.6, 129.3)
- moved R8 2.44 mm to (143.3, 123.7)
- moved R1 1.11 mm to (169.2, 96.0)
- moved C12 1.00 mm to (132.0, 91.6)
Routing:
- net /NRST2: track 1.32 -> 132.7 mm, vias 0 -> 4
- net Net-(D1-K): track 2.66 -> 74.6 mm
- net /n_reset: track 1.50 -> 72.4 mm, vias 0 -> 2
- net 5v_Ext_Stack: track 55.6 -> 107.0 mm
- net /A: track 2.28 -> 45.9 mm
- net /Alert: track 1.50 -> 38.1 mm, vias 0 -> 2
- net /B: track 3.21 -> 38.7 mm
- net USBC_PWR_In: track 43.8 -> 63.7 mm
- net Mux_PWR_Out: track 57.3 -> 61.2 mm
- net Net-(Module1A-PI_nLED_Activity): track 1.50 -> 4.19 mm
- net +5V: track 14.1 -> 16.7 mm
- net /CM4_GPIO ( Ethernet, GPIO, SDCARD)/GLOBAL_EN: track 39.7 -> 37.2 mm
- net Net-(C2-Pad2): track 5.67 -> 8.04 mm

Commit message: stuff
Parts:
- removed J35, J36, J39: Conn_01x01, Connector_PinHeader_2.54mm:PinHeader_1x01_P2.54mm_Vertical
- moved J22 357.1 mm to (242.8, 151.3)
- moved J34 350.9 mm to (206.9, 61.9), turned to 180 degrees
- moved J29 343.8 mm to (241.4, 69.5)
- moved J8 343.8 mm to (241.4, 58.8)
- moved J31 343.8 mm to (241.4, 80.8)
- moved J37 343.1 mm to (202.3, 61.8), turned to 180 degrees
- moved J38 332.9 mm to (197.7, 61.9), turned to 180 degrees
- moved J12 329.0 mm to (228.0, 131.4), turned to -90 degrees
- moved J9 325.7 mm to (209.2, 30.7)
- moved J40 323.9 mm to (193.0, 61.9), turned to 180 degrees
- moved J11 320.1 mm to (168.2, 58.3)
- moved J30 312.4 mm to (164.9, 42.4), turned to 90 degrees
- moved D5 311.9 mm to (235.0, 117.5)
- moved D3 311.9 mm to (234.7, 85.8)
- moved D6 311.9 mm to (234.6, 106.5)
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Routing:
- net /CM4_GPIO ( Ethernet, GPIO, SDCARD)/ID_SD: track 1.32 -> 143.0 mm, vias 0 -> 2
- net +5V: track 16.7 -> 156.6 mm, vias 0 -> 10
- net /SDA: track 91.2 -> 214.8 mm, vias 2 -> 3
- net /SCL: track 93.6 -> 212.5 mm, vias 6 -> 13
- net /CM4_GPIO ( Ethernet, GPIO, SDCARD)/nRPIBOOT: track 1.50 -> 101.4 mm, vias 0 -> 1
- net /CM4_GPIO ( Ethernet, GPIO, SDCARD)/GLOBAL_EN: track 37.2 -> 117.9 mm, vias 2 -> 3
- net Net-(J2-Pin_13): track 0.00 -> 75.6 mm, vias 0 -> 1
- net /CM4_GPIO ( Ethernet, GPIO, SDCARD)/GPIO3: track 1.32 -> 69.6 mm, vias 0 -> 2
- net /CM4_GPIO ( Ethernet, GPIO, SDCARD)/GPIO11: track 1.32 -> 62.2 mm, vias 0 -> 2
- net /CM4_GPIO ( Ethernet, GPIO, SDCARD)/AIN1: track 1.32 -> 62.0 mm, vias 0 -> 3
- net /CM4_GPIO ( Ethernet, GPIO, SDCARD)/AIN0: track 1.32 -> 58.8 mm, vias 0 -> 3
- net /CM4_GPIO ( Ethernet, GPIO, SDCARD)/TV_OUT: track 1.22 -> 55.8 mm, vias 0 -> 1
- net /CM4_GPIO ( Ethernet, GPIO, SDCARD)/EEPROM_nWP: track 1.32 -> 54.9 mm, vias 0 -> 3
- net /CM4_GPIO ( Ethernet, GPIO, SDCARD)/GPIO6: track 1.32 -> 52.1 mm, vias 0 -> 2
- net /CM4_GPIO ( Ethernet, GPIO, SDCARD)/WL_nDis: track 1.50 -> 51.3 mm, vias 0 -> 1
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Other:
- board size 122.8 x 85 mm -> 130.2 x 91.5 mm

Commit message: STUFF
Parts:
- moved J22 125.0 mm to (118.3, 141.3), turned to 180 degrees
- moved J1 118.2 mm to (189.7, 148.0)
- moved U3 65.1 mm to (127.6, 37.3), turned to 90 degrees
- moved J24 42.5 mm to (125.7, 144.2), turned to 180 degrees
- moved J27 29.4 mm to (114.7, 125.3)
- moved J28 29.4 mm to (114.7, 134.0)
- moved R7 23.4 mm to (218.3, 77.2), turned to 90 degrees
- moved R19 21.8 mm to (226.5, 77.5), turned to 90 degrees
- moved Y3 21.4 mm to (226.4, 56.5), turned to 0 degrees
- moved R35 20.7 mm to (222.4, 77.2), turned to 90 degrees
- moved R33 20.4 mm to (224.4, 77.1), turned to 90 degrees
- moved R6 18.8 mm to (214.7, 65.0), turned to -90 degrees
- moved C23 16.9 mm to (230.2, 61.4), turned to 180 degrees
- moved D4 16.8 mm to (218.3, 73.2), turned to 90 degrees
- moved J13 15.3 mm to (99.0, 96.4)
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Connections:
- net /A renamed /A+
- net /B renamed /A-
- net /RS485/TB_A renamed /RS485/TB+
- net /RS485/TB_B renamed /RS485/TB-
- net /USBhub/DM1 renamed /USBhub/D1-
- net /USBhub/DM2 renamed /USBhub/D2-
- net /USBhub/DM3 renamed /USBhub/D3-
- net /USBhub/DM4 renamed /USBhub/D4-
- net /USBhub/DP1 renamed /USBhub/D1+
- net /USBhub/DP2 renamed /USBhub/D2+
- net /USBhub/DP3 renamed /USBhub/D3+
- net /USBhub/DP4 renamed /USBhub/D4+
Routing:
- net /CM4_GPIO ( Ethernet, GPIO, SDCARD)/ID_SC: track 34.1 -> 191.4 mm, vias 2 -> 3
- net /SCL: track 212.5 -> 283.3 mm
- net /SDA: track 214.8 -> 284.3 mm, vias 3 -> 7
- net /USBhub/DRV: track 3.15 -> 67.3 mm, vias 0 -> 6
- net Net-(D3-A): track 0.00 -> 52.1 mm
- net /CM4_GPIO ( Ethernet, GPIO, SDCARD)/GLOBAL_EN: track 117.9 -> 167.9 mm
- net /CM4_HighSpeed/HDMI0_CEC: track 1.22 -> 37.4 mm, vias 0 -> 4
- net /CM4_HighSpeed/HDMI0_D2_P: track 0.00 -> 31.4 mm
- net /CM4_HighSpeed/HDMI0_D2_N: track 2.60 -> 31.3 mm
- net /CM4_HighSpeed/HDMI0_D1_P: track 2.55 -> 28.9 mm
- net /CM4_HighSpeed/HDMI0_D1_N: track 2.45 -> 28.2 mm
- net /CM4_HighSpeed/HDMI0_D0_N: track 1.50 -> 25.2 mm
- net /A-: track 40.3 -> 63.9 mm
- net /CM4_HighSpeed/HDMI0_D0_P: track 2.65 -> 25.9 mm
- net /RS485/TB-: track 11.4 -> 34.0 mm, vias 0 -> 1
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Other:
- board size 130.2 x 91.5 mm -> 135.2 x 97.6 mm
